File: KiCad/uranus-fpga-board/fpga.kicad_sch (KiCad schematic)
At the start: 2 parts, among them U1 XC7K325T-3FFG900E

Commit message: New entry and schematic
Parts:
- removed R13: 100 Ohm, symbol Device:R_Small
- added C46, C47, C48: 330 μF, symbol Device:C
- added C49, C50: 100 μF, symbol Device:C
- added C51, C52, C53, C55: 4.7 μF, symbol Device:C_Small
- added C54: C_Small, symbol Device:C_Small
- added C56, C57, C58, C59, C60, C61, C62, C63, C64, C65, C66, C67: 47 μF, symbol Device:C
- U1: footprint FFG900XC7K325T_AMD -> XC7K325T-3FFG900E:FFG900XC7K325T_AMD
Connections:
- net +1V05_GTX is gone; now on net GND: U1.B7 (MGTAVCC), U1.D7 (MGTAVCC), U1.F7 (MGTAVCC), U1.H7 (MGTAVCC), U1.K7 (MGTAVCC), U1.M7 (MGTAVCC), U1.P7 (MGTAVCC)
- net +1V8_GTX is gone; now on net GND: U1.B3 (MGTAVTT), U1.C5 (MGTAVTT), U1.D3 (MGTAVTT), U1.E5 (MGTAVTT), U1.F3 (MGTAVTT), U1.G5 (MGTAVTT), U1.H3 (MGTAVTT), U1.J5 (MGTAVTT), U1.K3 (MGTAVTT), U1.L5 (MGTAVTT), U1.M3 (MGTAVTT), U1.N5 (MGTAVTT), U1.P3 (MGTAVTT), U1.R5 (MGTAVTT), U1.T3 (MGTAVTT), U1.T7 (MGTVCCAUX), U1.U5 (MGTAVTT), U1.V3 (MGTAVTT), U1.V7 (MGTVCCAUX), U1.W5 (MGTAVTT), U1.W7 (MGTAVTTRCAL_115)
- net +1V0: now also C46.1, C47.1, C48.1, C49.1, C50.1, C51.1, C52.1, C53.1, C54.1, C55.1
- net +1V5: now also U1.AA19 (VCCO_32), U1.AA9 (VCCO_33), U1.AB16 (VCCO_32), U1.AC13 (VCCO_33), U1.AC3 (VCCO_34), U1.AD10 (VCCO_33), U1.AE17 (VCCO_32), U1.AE7 (VCCO_34), U1.AF14 (VCCO_32), U1.AF4 (VCCO_34), U1.AG1 (VCCO_34), U1.AG11 (VCCO_33), U1.AH18 (VCCO_32), U1.AH8 (VCCO_34), U1.AJ15 (VCCO_32), U1.AJ5 (VCCO_34), U1.AK12 (VCCO_33), U1.AK2 (VCCO_34), U1.Y12 (VCCO_33), C60.1, C63.1, C64.1
- net +1V8: now also C56.1, C57.1, C58.1, C59.1, C61.1, C62.1
- net +2V5: now also U1.A19 (VCCO_17), U1.B16 (VCCO_17), U1.D20 (VCCO_17), U1.E17 (VCCO_17), U1.G21 (VCCO_17), U1.H18 (VCCO_17), U1.L19 (VCCO_17), C65.1, C66.1
- net +3V3: now also U1.AB6 (VCCO_0), U1.T9 (VCCO_0), C67.1
- net GND: now also C46.2, C47.2, C48.2, C49.2, C50.2, C51.2, C52.2, C53.2, C54.2, C55.2, C56.2, C57.2, C58.2, C59.2, C60.2, C61.2, C62.2, C63.2, C64.2, C65.2, C66.2, C67.2
- net DATA15_N: now reaches U1.C11 (IO_L18N_T2_18)
- net DATA15_P: now reaches U1.D11 (IO_L18P_T2_18)
- net DATA14_N: now reaches U1.E11 (IO_L16N_T2_18)
- net DATA14_P: now reaches U1.F11 (IO_L16P_T2_18)
- net DATA31_N: now reaches U1.F17 (IO_L18N_T2_17)
- net DATA30_N: now reaches U1.F18 (IO_L16N_T2_17)
- net DATA31_P: now reaches U1.G17 (IO_L18P_T2_17)
- net DATA30_P: now reaches U1.G18 (IO_L16P_T2_17)
- net DATA22_N: now reaches U1.C21 (IO_L8N_T1_17)
- net DATA24_N: now reaches U1.C22 (IO_L10N_T1_17)
- net DATA22_P: now reaches U1.D21 (IO_L8P_T1_17)
- net DATA24_P: now reaches U1.D22 (IO_L10P_T1_17)
- net DATA23_N: now reaches U1.F22 (IO_L9N_T1_DQS_17)
- net DATA5_N: now reaches U1.G15 (IO_L7N_T1_18)
- net DATA23_P: now reaches U1.G22 (IO_L9P_T1_DQS_17)
- net DATA8_P: now reaches U1.H11 (IO_L10P_T1_18)
- net DATA8_N: now reaches U1.H12 (IO_L10N_T1_18)
- net DATA5_P: now reaches U1.H15 (IO_L7P_T1_18)
- net DATA7_N: now reaches U1.H16 (IO_L9N_T1_DQS_18)
- net DATA21_P: now reaches U1.H21 (IO_L7P_T1_17)
- net DATA21_N: now reaches U1.H22 (IO_L7N_T1_17)
- net DATA6_P: now reaches U1.J11 (IO_L8P_T1_18)
- net DATA6_N: now reaches U1.J12 (IO_L8N_T1_18)
- net DATA7_P: now reaches U1.J16 (IO_L9P_T1_DQS_18)
- net DATA13_N: now reaches U1.B12 (IO_L15N_T2_DQS_18)
- net DATA13_P: now reaches U1.C12 (IO_L15P_T2_DQS_18)
- net DATA29_N: now reaches U1.C16 (IO_L15N_T2_DQS_17)
- net DATA11_P: now reaches U1.D12 (IO_L13P_T2_MRCC_18)
- net DATA11_N: now reaches U1.D13 (IO_L13N_T2_MRCC_18)
- net DATA29_P: now reaches U1.D16 (IO_L15P_T2_DQS_17)
- net DATA27_P: now reaches U1.D17 (IO_L13P_T2_MRCC_17)
- net DATA27_N: now reaches U1.D18 (IO_L13N_T2_MRCC_17)
- net DATA28_N: now reaches U1.D19 (IO_L14N_T2_SRCC_17)
- net DATA12_N: now reaches U1.E13 (IO_L14N_T2_SRCC_18)
- net DATA28_P: now reaches U1.E19 (IO_L14P_T2_SRCC_17)
- net DATA26_N: now reaches U1.E20 (IO_L12N_T1_MRCC_17)
- net DATA25_N: now reaches U1.E21 (IO_L11N_T1_SRCC_17)
- net DATA12_P: now reaches U1.F12 (IO_L14P_T2_SRCC_18)
- net DATA10_N: now reaches U1.F13 (IO_L12N_T1_MRCC_18)
- net DATA26_P: now reaches U1.F20 (IO_L12P_T1_MRCC_17)
- net DATA9_N: now reaches U1.F21 (IO_L11P_T1_SRCC_17)
- net DATA9_N: now also U1.G14 (IO_L11N_T1_SRCC_18)
- net DATA10_P: now reaches U1.G13 (IO_L12P_T1_MRCC_18)
- net DATA9_P: now reaches U1.H14 (IO_L11P_T1_SRCC_18)
- net DATA17_N: now reaches U1.G20 (IO_L2N_T0_17)
- net DATA18_N: now reaches U1.H17 (IO_L3N_T0_DQS_17)
- net DATA19_N: now reaches U1.H19 (IO_L4N_T0_17)
- net DATA17_P: now reaches U1.H20 (IO_L2P_T0_17)
- net DATA3_N: now reaches U1.J13 (IO_L4N_T0_18)
- net DATA4_N: now reaches U1.J14 (IO_L5N_T0_18)
- net DATA18_P: now reaches U1.J17 (IO_L3P_T0_DQS_17)
- net DATA16_N: now reaches U1.J18 (IO_L1N_T0_17)
- net DATA19_P: now reaches U1.J19 (IO_L4P_T0_17)
- net DATA3_P: now reaches U1.K13 (IO_L4P_T0_18)
- net DATA4_P: now reaches U1.K14 (IO_L5P_T0_18)
- net DATA1_N: now reaches U1.K15 (IO_L2N_T0_18)
- net DATA0_N: now reaches U1.K16 (IO_L1N_T0_18)
- net DATA16_P: now reaches U1.K18 (IO_L1P_T0_17)
- net DATA2_P: now reaches U1.L12 (IO_L3P_T0_DQS_18)
- net DATA2_N: now reaches U1.L13 (IO_L3N_T0_DQS_18)
- net DATA1_P: now reaches U1.L15 (IO_L2P_T0_18)
- net DATA0_P: now reaches U1.L16 (IO_L1P_T0_18)
- net DATA20_P: now reaches U1.L17 (IO_L5P_T0_17)
- net DATA20_N: now reaches U1.L18 (IO_L5N_T0_17)
Other:
- note added: "100 μF"
- note added: "330 μF"
- note added: "4.7 μF"
- note added: "47 μF"
- note added: "VCCAUX"
- note added: "VCCAUX_IO"
- note added: "VCCBRAM"
- note added: "VCCINT"
- note added: "VCCO_0"
- note added: "VCCO_17"
- note added: "VCCO_18"
- note added: "VCCO_32"
- note added: "VCCO_33"
- note added: "VCCO_34"
- note removed: "0.1%"
- moved on the sheet: U1A, U1B, U1C, U1D, U1E, U1F, U1G, U1H, U1I, U1J, U1K

Commit message: New journal entry
Changed lines of the file:
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@@
+	)
+	(symbol
+		(lib_id "power:+1V0")
+		(at 34.29 311.15 0)
+		(unit 1)
+		(body_style 1)
+		(exclude_from_sim no)
+		(in_bom yes)
+		(on_board yes)
+		(in_pos_files yes)
+		(dnp no)
+		(fields_autoplaced yes)
+		(property "Reference" "#PWR094"
+			(at 34.29 314.96 0)
+			(hide yes)
+			(show_name no)
+			(do_not_autoplace no)
+			(effects
+				(font
+					(size 1.27 1.27)
+				)
+			)
+		)
+		(property "Value" "+12V0"
+			(at 34.29 306.07 0)
+			(show_name no)
+			(do_not_autoplace no)
+			(effects
+				(font
+					(size 1.27 1.27)
+				)
+			)
+		)
+		(property "Footprint" "Package_DFN_QFN:Renesas_UQFN-16_2x2mm_P0.4mm"
+			(at 34.29 311.15 0)
+			(hide yes)
+			(show_name no)
+			(do_not_autoplace no)
+			(effects
+				(font
+					(size 1.27 1.27)
+				)
+			)
+		)
+		(property "Datasheet" ""
+			(at 34.29 311.15 0)
+			(hide yes)
+			(show_name no)
+			(do_not_autoplace no)
+			(effects
+				(font
+					(size 1.27 1.27)
+				)
+			)
+		)
+		(property "Description" "Power symbol creates a global label with name \"+1V0\""
+			(at 34.29 311.15 0)
+			(hide yes)
+			(show_name no)
+			(do_not_autoplace no)
+			(effects
+				(font
+					(size 1.27 1.27)
+				)
+			)
+		)
+		(pin "1"
+		)
+		(instances
+			(project "uranus-fpga-board"
+				(path "/11d4e4d4-71ba-48aa-ae73-e6b6dc32b11b/9b31d439-c2fe-44d5-bcd7-596f029a918d"
+					(reference "#PWR094")
+					(unit 1)
+				)
+			)
+		)
 	)
 	(symbol

Commit message: New journal entry, progress on schematic and PCB
Connections:
- net +2V5: now also U1.A29 (VCCO_16), U1.B26 (VCCO_16), U1.C23 (VCCO_16), U1.D30 (VCCO_16), U1.E27 (VCCO_16), U1.F24 (VCCO_16), U1.H28 (VCCO_16)
- net LA30_N: now reaches U1.A11 (IO_L17P_T2_18)
- net LA30_P: now reaches U1.A12 (IO_L17N_T2_18)
- net LA25_N: now reaches U1.A16 (IO_L20P_T3_17)
- net LA25_P: now reaches U1.A17 (IO_L20N_T3_17)
- net LA03_N: now reaches U1.A30 (IO_L17N_T2_16)
- net LA21_P: now reaches U1.B17 (IO_L17N_T2_17)
- net LA20_P: now reaches U1.B20 (IO_L19N_T3_VREF_17)
- net LA03_P: now reaches U1.B30 (IO_L17P_T2_16)
- net LA21_N: now reaches U1.C17 (IO_L17P_T2_17)
- net LA20_N: now reaches U1.C20 (IO_L19P_T3_17)
- net LA02_P: now reaches U1.C30 (IO_L16N_T2_16)
- net LA02_N: now reaches U1.D29 (IO_L16P_T2_16)
- net LA07_N: now reaches U1.A27 (IO_L7N_T1_16)
- net LA08_N: now reaches U1.A28 (IO_L9N_T1_DQS_16)
- net LA12_N: now reaches U1.B24 (IO_L8N_T1_16)
- net LA07_P: now reaches U1.B27 (IO_L7P_T1_16)
- net LA08_P: now reaches U1.B28 (IO_L9P_T1_DQS_16)
- net LA12_P: now reaches U1.C24 (IO_L8P_T1_16)
- net LA04_N: now reaches U1.B29 (IO_L15N_T2_DQS_16)
- net LA00_CC_N: now reaches U1.C27 (IO_L13N_T2_MRCC_16)
- net LA04_P: now reaches U1.C29 (IO_L15P_T2_DQS_16)
- net LA00_CC_P: now reaches U1.D27 (IO_L13P_T2_MRCC_16)
- net LA11_N: now reaches U1.A23 (IO_L1N_T0_16)
- net LA11_P: now reaches U1.B23 (IO_L1P_T0_16)
- net LA31_P: now reaches U1.A13 (IO_L22N_T3_18)
- net LA29_P: now reaches U1.A15 (IO_L24N_T3_18)
- net LA22_P: now reaches U1.A18 (IO_L22N_T3_17)
- net LA15_N: now reaches U1.A20 (IO_L21P_T3_DQS_17)
- net LA15_P: now reaches U1.A21 (IO_L21N_T3_DQS_17)
- net LA16_N: now reaches U1.A22 (IO_L23N_T3_17)
- net LA31_N: now reaches U1.B13 (IO_L22P_T3_18)
- net LA29_N: now reaches U1.B14 (IO_L24P_T3_18)
- net LA24_P: now reaches U1.B15 (IO_L23N_T3_18)
- net LA22_N: now reaches U1.B18 (IO_L22P_T3_17)
- net LA19_P: now reaches U1.B19 (IO_L24N_T3_17)
- net LA16_P: now reaches U1.B22 (IO_L23P_T3_17)
- net LA28_P: now reaches U1.C14 (IO_L21N_T3_DQS_18)
- net LA24_N: now reaches U1.C15 (IO_L23P_T3_18)
- net LA19_N: now reaches U1.C19 (IO_L24P_T3_17)
- net LA28_N: now reaches U1.D14 (IO_L21P_T3_DQS_18)
- net DATA0_N: no longer names the net of U1.K16 (IO_L1N_T0_18)
- net DATA0_P: no longer names the net of U1.L16 (IO_L1P_T0_18)
- net DATA10_N: no longer names the net of U1.F13 (IO_L12N_T1_MRCC_18)
- net DATA10_P: no longer names the net of U1.G13 (IO_L12P_T1_MRCC_18)
- net DATA11_N: no longer names the net of U1.D13 (IO_L13N_T2_MRCC_18)
- net DATA11_P: no longer names the net of U1.D12 (IO_L13P_T2_MRCC_18)
- net DATA12_N: no longer names the net of U1.E13 (IO_L14N_T2_SRCC_18)
- net DATA12_P: no longer names the net of U1.F12 (IO_L14P_T2_SRCC_18)
- net DATA13_N renamed LA33_P
- net DATA13_P renamed LA33_N
- net DATA14_N: no longer names the net of U1.E11 (IO_L16N_T2_18)
- net DATA14_P: no longer names the net of U1.F11 (IO_L16P_T2_18)
- net DATA15_N renamed LA32_P
- net DATA15_P renamed LA32_N
- net DATA16_N: no longer names the net of U1.J18 (IO_L1N_T0_17)
- net DATA16_P: no longer names the net of U1.K18 (IO_L1P_T0_17)
- net DATA17_N: no longer names the net of U1.G20 (IO_L2N_T0_17)
- net DATA17_P: no longer names the net of U1.H20 (IO_L2P_T0_17)
- net DATA18_N: no longer names the net of U1.H17 (IO_L3N_T0_DQS_17)
- net DATA18_P: no longer names the net of U1.J17 (IO_L3P_T0_DQS_17)
- net DATA19_N: no longer names the net of U1.H19 (IO_L4N_T0_17)
- net DATA19_P: no longer names the net of U1.J19 (IO_L4P_T0_17)
- net DATA1_N: no longer names the net of U1.K15 (IO_L2N_T0_18)
- net DATA1_P: no longer names the net of U1.L15 (IO_L2P_T0_18)
- net DATA20_N: no longer names the net of U1.L18 (IO_L5N_T0_17)
- net DATA20_P: no longer names the net of U1.L17 (IO_L5P_T0_17)
- net DATA21_N: no longer names the net of U1.H22 (IO_L7N_T1_17)
- net DATA21_P: no longer names the net of U1.H21 (IO_L7P_T1_17)
- net DATA22_N: no longer names the net of U1.C21 (IO_L8N_T1_17)
- net DATA22_P: no longer names the net of U1.D21 (IO_L8P_T1_17)
- net DATA23_N: no longer names the net of U1.F22 (IO_L9N_T1_DQS_17)
- net DATA23_P: no longer names the net of U1.G22 (IO_L9P_T1_DQS_17)
- net DATA24_N: no longer names the net of U1.C22 (IO_L10N_T1_17)
- net DATA24_P: no longer names the net of U1.D22 (IO_L10P_T1_17)
- net DATA25_N: no longer names the net of U1.E21 (IO_L11N_T1_SRCC_17)
- net DATA26_N: no longer names the net of U1.E20 (IO_L12N_T1_MRCC_17)
- net DATA26_P: no longer names the net of U1.F20 (IO_L12P_T1_MRCC_17)
- net DATA27_N renamed LA18_CC_N
- net DATA27_P renamed LA18_CC_P
- net DATA28_N: no longer names the net of U1.D19 (IO_L14N_T2_SRCC_17)
- net DATA28_P: no longer names the net of U1.E19 (IO_L14P_T2_SRCC_17)
- net DATA29_N: no longer names the net of U1.C16 (IO_L15N_T2_DQS_17)
- net DATA29_P: no longer names the net of U1.D16 (IO_L15P_T2_DQS_17)
- net DATA2_N: no longer names the net of U1.L13 (IO_L3N_T0_DQS_18)
- net DATA2_P: no longer names the net of U1.L12 (IO_L3P_T0_DQS_18)
- net DATA30_N: no longer names the net of U1.F18 (IO_L16N_T2_17)
- net DATA30_P: no longer names the net of U1.G18 (IO_L16P_T2_17)
- net DATA31_N: no longer names the net of U1.F17 (IO_L18N_T2_17)
- net DATA31_P: no longer names the net of U1.G17 (IO_L18P_T2_17)
- net DATA3_N: no longer names the net of U1.J13 (IO_L4N_T0_18)
- net DATA3_P: no longer names the net of U1.K13 (IO_L4P_T0_18)
- net DATA4_N: no longer names the net of U1.J14 (IO_L5N_T0_18)
- net DATA4_P: no longer names the net of U1.K14 (IO_L5P_T0_18)
- net DATA5_N: no longer names the net of U1.G15 (IO_L7N_T1_18)
- net DATA5_P: no longer names the net of U1.H15 (IO_L7P_T1_18)
- net DATA6_N: no longer names the net of U1.J12 (IO_L8N_T1_18)
- net DATA6_P: no longer names the net of U1.J11 (IO_L8P_T1_18)
- net DATA7_N: no longer names the net of U1.H16 (IO_L9N_T1_DQS_18)
- net DATA7_P: no longer names the net of U1.J16 (IO_L9P_T1_DQS_18)
- net DATA8_N: no longer names the net of U1.H12 (IO_L10N_T1_18)
- net DATA8_P: no longer names the net of U1.H11 (IO_L10P_T1_18)
- net DATA9_N: no longer names the net of U1.F21 (IO_L11P_T1_SRCC_17)
- net DATA9_N: no longer U1.G14 (IO_L11N_T1_SRCC_18)
- net DATA9_P: no longer names the net of U1.H14 (IO_L11P_T1_SRCC_18)
Other:
- note added: "VCCO_16"
- note removed: "VCCO_18"
- moved on the sheet: U1G
