File: KiCad/uranus-fpga-board/fpga.kicad_sch (KiCad schematic)
At the start: 23 parts, among them U1 XC7K325T-3FFG900E

Commit message: New journal, moved BOMS into a new directory
Parts:
- renumbered C46 to C1, C52 to C10, C53 to C11, C54 to C12, C55 to C13, C59 to C14, C61 to C15, C62 to C16, C65 to C17, C66 to C18, C67 to C19, C47 to C2, C60 to C20, C63 to C21, C64 to C22, C48 to C3, C56 to C4, C57 to C5, C58 to C6, C49 to C7, C50 to C8, C51 to C9
Connections:
- net +2V5: no longer U1.A19 (VCCO_17), U1.B16 (VCCO_17), U1.C13 (VCCO_18), U1.D10 (VCCO_18), U1.D20 (VCCO_17), U1.E17 (VCCO_17), U1.E27 (VCCO_16), U1.F14 (VCCO_18), U1.F24 (VCCO_16), U1.G11 (VCCO_18), U1.G21 (VCCO_17), U1.H18 (VCCO_17), U1.H28 (VCCO_16), U1.J15 (VCCO_18), U1.K12 (VCCO_18), U1.L19 (VCCO_17)
- net FMC_LA26_N: now reaches U1.E11 (IO_L16N_T2_18)
- net FMC_LA27_N: now reaches U1.E14 (IO_L20P_T3_18)
- net FMC_LA27_P: now reaches U1.E15 (IO_L20N_T3_18)
- net FMC_LA23_P: now reaches U1.E16 (IO_L19N_T3_VREF_18)
- net FMC_LA01_N: now reaches U1.E29 (IO_L18P_T2_16)
- net FMC_LA01_P: now reaches U1.E30 (IO_L18N_T2_16)
- net FMC_LA26_P: now reaches U1.F11 (IO_L16P_T2_18)
- net FMC_LA23_N: now reaches U1.F15 (IO_L19P_T3_18)
- net FMC_DP0_C2M_N: now reaches U1.B1 (MGTXTXN2_118)
- net FMC_DP0_C2M_P: now reaches U1.B2 (MGTXTXP2_118)
- net FMC_MGTREFCLK0_N: now reaches U1.C7 (MGTREFCLK0N_118)
- net FMC_MGTREFCLK0_P: now reaches U1.C8 (MGTREFCLK0P_118)
- net FMC_LA10_N: now reaches U1.C21 (IO_L8N_T1_17)
- net FMC_LA09_N: now reaches U1.C22 (IO_L10N_T1_17)
- net FMC_LA10_P: now reaches U1.D21 (IO_L8P_T1_17)
- net FMC_LA09_P: now reaches U1.D22 (IO_L10P_T1_17)
- net FMC_LA14_N: now reaches U1.C16 (IO_L15N_T2_DQS_17)
- net FMC_LA17_CC_P: now reaches U1.D12 (IO_L13P_T2_MRCC_18)
- net FMC_LA17_CC_N: now reaches U1.D13 (IO_L13N_T2_MRCC_18)
- net FMC_LA14_P: now reaches U1.D16 (IO_L15P_T2_DQS_17)
- net FMC_LA13_N: now reaches U1.D19 (IO_L14N_T2_SRCC_17)
- net FMC_LA13_P: now reaches U1.E19 (IO_L14P_T2_SRCC_17)
- net FMC_LA05_N: now reaches U1.D23 (IO_L2N_T0_16)
- net FMC_LA06_N: now reaches U1.D24 (IO_L4N_T0_16)
- net FMC_LA05_P: now reaches U1.E23 (IO_L2P_T0_16)
- net FMC_LA06_P: now reaches U1.E24 (IO_L4P_T0_16)
- net FMC_DP0_M2C_N: now reaches U1.B5 (MGTXRXN2_118)
- net FMC_DP0_M2C_P: now reaches U1.B6 (MGTXRXP2_118)
- net A0 renamed DDR_A0
- net A1 renamed DDR_A1
- net A10 renamed DDR_A10
- net A11 renamed DDR_A11
- net A12 renamed DDR_A12
- net A2 renamed DDR_A2
- net A3 renamed DDR_A3
- net A4 renamed DDR_A4
- net A5 renamed DDR_A5
- net A6 renamed DDR_A6
- net A7 renamed DDR_A7
- net A8 renamed DDR_A8
- net A9 renamed DDR_A9
- net BA0 renamed DDR_BA0
- net BA1 renamed DDR_BA1
- net BA2 renamed DDR_BA2
- net CAS_N renamed DDR_CAS_N
- net CKE renamed DDR_CKE
- net CK_N renamed DDR_CK_N
- net CK_P renamed DDR_CK_P
- net CLK_N renamed DDR_CLK_N
- net CLK_P renamed DDR_CLK_P
- net CS_N renamed DDR_CS_N
- net DM0 renamed DDR_DM0
- net DM1 renamed DDR_DM1
- net DM2 renamed DDR_DM2
- net DM3 renamed DDR_DM3
- net DM4 renamed DDR_DM4
- net DM5 renamed DDR_DM5
- net DM6 renamed DDR_DM6
- net DM7 renamed DDR_DM7
- net DQ00 renamed DDR_DQ00
- net DQ01 renamed DDR_DQ01
- net DQ02 renamed DDR_DQ02
- net DQ03 renamed DDR_DQ03
- net DQ04 renamed DDR_DQ04
- net DQ05 renamed DDR_DQ05
- net DQ06 renamed DDR_DQ06
- net DQ07 renamed DDR_DQ07
- net DQ08 renamed DDR_DQ08
- net DQ09 renamed DDR_DQ09
- net DQ10 renamed DDR_DQ10
- net DQ11 renamed DDR_DQ11
- net DQ12 renamed DDR_DQ12
- net DQ13 renamed DDR_DQ13
- net DQ14 renamed DDR_DQ14
- net DQ15 renamed DDR_DQ15
- net DQ16 renamed DDR_DQ16
- net DQ17 renamed DDR_DQ17
- net DQ18 renamed DDR_DQ18
- net DQ19 renamed DDR_DQ19
- net DQ20 renamed DDR_DQ20
- net DQ21 renamed DDR_DQ21
- net DQ22 renamed DDR_DQ22
- net DQ23 renamed DDR_DQ23
- net DQ24 renamed DDR_DQ24
- net DQ25 renamed DDR_DQ25
- net DQ26 renamed DDR_DQ26
- net DQ27 renamed DDR_DQ27
- net DQ28 renamed DDR_DQ28
- net DQ29 renamed DDR_DQ29
- net DQ30 renamed DDR_DQ30
- net DQ31 renamed DDR_DQ31
- net DQ32 renamed DDR_DQ32
- net DQ33 renamed DDR_DQ33
- net DQ34 renamed DDR_DQ34
- net DQ35 renamed DDR_DQ35
- net DQ36 renamed DDR_DQ36
- net DQ37 renamed DDR_DQ37
- net DQ38 renamed DDR_DQ38
- net DQ39 renamed DDR_DQ39
- net DQ40 renamed DDR_DQ40
- net DQ41 renamed DDR_DQ41
- net DQ42 renamed DDR_DQ42
- net DQ43 renamed DDR_DQ43
- net DQ44 renamed DDR_DQ44
- net DQ45 renamed DDR_DQ45
- net DQ46 renamed DDR_DQ46
- net DQ47 renamed DDR_DQ47
- net DQ48 renamed DDR_DQ48
- net DQ49 renamed DDR_DQ49
- net DQ50 renamed DDR_DQ50
- net DQ51 renamed DDR_DQ51
- net DQ52 renamed DDR_DQ52
- net DQ53 renamed DDR_DQ53
- net DQ54 renamed DDR_DQ54
- net DQ55 renamed DDR_DQ55
- net DQ56 renamed DDR_DQ56
- net DQ57 renamed DDR_DQ57
- net DQ58 renamed DDR_DQ58
- net DQ59 renamed DDR_DQ59
- net DQ60 renamed DDR_DQ60
- net DQ61 renamed DDR_DQ61
- net DQ62 renamed DDR_DQ62
- net DQ63 renamed DDR_DQ63
- net DQS_N0 renamed DDR_DQS_N0
- net DQS_N1 renamed DDR_DQS_N1
- net DQS_N2 renamed DDR_DQS_N2
- net DQS_N3 renamed DDR_DQS_N3
- net DQS_N4 renamed DDR_DQS_N4
- net DQS_N5 renamed DDR_DQS_N5
- net DQS_N6 renamed DDR_DQS_N6
- net DQS_N7 renamed DDR_DQS_N7
- net DQS_P0 renamed DDR_DQS_P0
- net DQS_P1 renamed DDR_DQS_P1
- net DQS_P2 renamed DDR_DQS_P2
- net DQS_P3 renamed DDR_DQS_P3
- net DQS_P4 renamed DDR_DQS_P4
- net DQS_P5 renamed DDR_DQS_P5
- net DQS_P6 renamed DDR_DQS_P6
- net DQS_P7 renamed DDR_DQS_P7
- net LA00_CC_N renamed FMC_LA00_CC_N
- net LA00_CC_P renamed FMC_LA00_CC_P
- net LA02_N renamed FMC_LA02_N
- net LA02_P renamed FMC_LA02_P
- net LA03_N renamed FMC_LA03_N
- net LA03_P renamed FMC_LA03_P
- net LA04_N renamed FMC_LA04_N
- net LA04_P renamed FMC_LA04_P
- net LA07_N renamed FMC_LA07_N
- net LA07_P renamed FMC_LA07_P
- net LA08_N renamed FMC_LA08_N
- net LA08_P renamed FMC_LA08_P
- net LA11_N renamed FMC_LA11_N
- net LA11_P renamed FMC_LA11_P
- net LA12_N renamed FMC_LA12_N
- net LA12_P renamed FMC_LA12_P
- net LA15_N renamed FMC_LA15_N
- net LA15_P renamed FMC_LA15_P
- net LA16_N renamed FMC_LA16_N
- net LA16_P renamed FMC_LA16_P
- net LA18_CC_N renamed FMC_LA18_CC_N
- net LA18_CC_P renamed FMC_LA18_CC_P
- net LA19_N renamed FMC_LA19_N
- net LA19_P renamed FMC_LA19_P
- net LA20_N renamed FMC_LA20_N
- net LA20_P renamed FMC_LA20_P
- net LA21_N renamed FMC_LA21_N
- net LA21_P renamed FMC_LA21_P
- net LA22_N renamed FMC_LA22_N
- net LA22_P renamed FMC_LA22_P
- net LA24_N renamed FMC_LA24_N
- net LA24_P renamed FMC_LA24_P
- net LA25_N renamed FMC_LA25_N
- net LA25_P renamed FMC_LA25_P
- net LA28_N renamed FMC_LA28_N
- net LA28_P renamed FMC_LA28_P
- net LA29_N renamed FMC_LA29_N
- net LA29_P renamed FMC_LA29_P
- net LA30_N renamed FMC_LA30_N
- net LA30_P renamed FMC_LA30_P
- net LA31_N renamed FMC_LA31_N
- net LA31_P renamed FMC_LA31_P
- net LA32_N renamed FMC_LA32_N
- net LA32_P renamed FMC_LA32_P
- net LA33_N renamed FMC_LA33_N
- net LA33_P renamed FMC_LA33_P
- net ODT renamed DDR_ODT
- net RAS_N renamed DDR_RAS_N
- net REF_N renamed DDR_REF_N
- net REF_P renamed DDR_REF_P
- net RESET renamed DDR_RESET
- net WE_N renamed DDR_WE_N
- new net FMC_VREF_A_M2C: U1.A19 (VCCO_17), U1.B16 (VCCO_17), U1.C13 (VCCO_18), U1.D10 (VCCO_18), U1.D20 (VCCO_17), U1.E17 (VCCO_17), U1.E27 (VCCO_16), U1.F14 (VCCO_18), U1.F24 (VCCO_16), U1.G11 (VCCO_18), U1.G21 (VCCO_17), U1.H18 (VCCO_17), U1.H28 (VCCO_16), U1.J15 (VCCO_18), U1.K12 (VCCO_18), U1.L19 (VCCO_17)
Other:
- moved on the sheet: U1A, U1B, U1C, U1D, U1E, U1F, U1G, U1H, U1I, U1J

Commit message: Oct 18 journal
Connections:
- net +2V5: no longer U1.A29 (VCCO_16), U1.B26 (VCCO_16), U1.C23 (VCCO_16), U1.D30 (VCCO_16)
- net DDR_CAS_N renamed ~{DDR_CAS}
- net DDR_CS_N renamed ~{DDR_CS}
- net DDR_RAS_N renamed ~{DDR_RAS}
- net DDR_WE_N renamed ~{DDR_WE}
- net FMC_VREF_A_M2C renamed VADJ_P
- net VADJ_P: now also U1.A29 (VCCO_16), U1.B26 (VCCO_16), U1.C23 (VCCO_16), U1.D30 (VCCO_16)
Changed lines of the file:
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@@
 		)
 	)
-	(global_label "DDR_WE_N"
+	(global_label "~{DDR_WE}"
 		(shape output)
 		(at 358.14 68.58 180)
@@
 		)
 	)
-	(global_label "DDR_CS_N"
+	(global_label "~{DDR_CS}"
 		(shape output)
 		(at 358.14 43.18 180)
@@
 		)
 	)
-	(global_label "FMC_VREF_A_M2C"
-		(shape output)
-		(at 808.99 29.21 0)
-		(fields_autoplaced yes)
-		(effects
-			(font
-				(size 1.27 1.27)
-			)
-			(justify left)
-		)
-		(property "Intersheetrefs" "${INTERSHEET_REFS}"
-			(at 823.5261 29.21 0)
-			(hide yes)
-			(show_name no)
-			(do_not_autoplace no)
-			(effects
-				(font
-					(size 1.27 1.27)
-				)
-				(justify left)
-			)
-		)
-	)
 	(global_label "DDR_DQ40"
 		(shape bidirectional)
@@
 		)
 	)
-	(global_label "DDR_RAS_N"
+	(global_label "~{DDR_RAS}"
 		(shape output)
 		(at 317.5 142.24 0)
@@
 		)
 	)
-	(global_label "DDR_CAS_N"
+	(global_label "~{DDR_CAS}"
 		(shape output)
 		(at 317.5 116.84 0)
@@
 	)
 	(symbol
-		(lib_id "power:+3V3")
-		(at 816.61 39.37 0)
-		(unit 1)
-		(body_style 1)
-		(exclude_from_sim no)
-		(in_bom yes)
-		(on_board yes)
-		(in_pos_files yes)
-		(dnp no)
-		(fields_autoplaced yes)
-		(property "Reference" "#PWR037"
-			(at 816.61 43.18 0)
-			(hide yes)
-			(show_name no)
-			(do_not_autoplace no)
-			(effects
-				(font
-					(size 1.27 1.27)
-				)
-			)
-		)
-		(property "Value" "FMC_VREF_A_M2C"
-			(at 816.61 34.29 0)
-			(show_name no)
-			(do_not_autoplace no)
-			(effects
-				(font
-					(size 1.27 1.27)
-				)
-			)
-		)
-		(property "Footprint" ""
-			(at 816.61 39.37 0)
-			(hide yes)
-			(show_name no)
-			(do_not_autoplace no)
-			(effects
-				(font
-					(size 1.27 1.27)
-				)
-			)
-		)
-		(property "Datasheet" ""
-			(at 816.61 39.37 0)
-			(hide yes)
-			(show_name no)
-			(do_not_autoplace no)
-			(effects
-				(font
-					(size 1.27 1.27)
-				)
-			)
-		)
-		(property "Description" "Power symbol creates a global label with name \"+3V3\""
-			(at 816.61 39.37 0)
-			(hide yes)
-			(show_name no)
-			(do_not_autoplace no)
-			(effects
-				(font
-					(size 1.27 1.27)
-				)
-			)
-		)
-		(pin "1"
-		)
-		(instances
-			(project "uranus-fpga-board"
-				(path "/11d4e4d4-71ba-48aa-ae73-e6b6dc32b11b/9b31d439-c2fe-44d5-bcd7-596f029a918d"
-					(reference "#PWR037")
-					(unit 1)
-				)
-			)
-		)
-	)
-	(symbol
 		(lib_id "power:+1V0")
 		(at 93.98 341.63 90)
@@
 		(dnp no)
 		(fields_autoplaced yes)
-		(property "Reference" "#PWR05"
+		(property "Reference" "#PWR04"
 			(at 58.42 401.32 0)
 			(hide yes)
@@
 			(project "uranus-fpga-board"
 				(path "/11d4e4d4-71ba-48aa-ae73-e6b6dc32b11b/9b31d439-c2fe-44d5-bcd7-596f029a918d"
-					(reference "#PWR05")
+					(reference "#PWR04")
 					(unit 1)
 				)
@@
 	)
 	(symbol
+		(lib_id "power:+1V5")
+		(at 808.99 29.21 270)
+		(unit 1)
+		(body_style 1)
+		(exclude_from_sim no)
+		(in_bom yes)
+		(on_board yes)
+		(in_pos_files yes)
+		(dnp no)
+		(fields_autoplaced yes)
+		(property "Reference" "#PWR037"
+			(at 805.18 29.21 0)
+			(hide yes)
+			(show_name no)
+			(do_not_autoplace no)
+			(effects
+				(font
+					(size 1.27 1.27)
+				)
+			)
+		)
+		(property "Value" "VADJ_P"
+			(at 812.8 29.2099 90)
+			(show_name no)
+			(do_not_autoplace no)
+			(effects
+				(font
+					(size 1.27 1.27)
+				)
+				(justify left)
+			)
+		)
+		(property "Footprint" ""
+			(at 808.99 29.21 0)
+			(hide yes)
+			(show_name no)
+			(do_not_autoplace no)
+			(effects
+				(font
+					(size 1.27 1.27)
+				)
+			)
+		)
+		(property "Datasheet" ""
+			(at 808.99 29.21 0)
+			(hide yes)
+			(show_name no)
+			(do_not_autoplace no)
+			(effects
+				(font
+					(size 1.27 1.27)
+				)
+			)
+		)
+		(property "Description" "Power symbol creates a global label with name \"+1V5\""
+			(at 808.99 29.21 0)
+			(hide yes)
+			(show_name no)
+			(do_not_autoplace no)
+			(effects
+				(font
+					(size 1.27 1.27)
+				)
+			)
+		)
+		(pin "1"
+		)
+		(instances
+			(project "uranus-fpga-board"
+				(path "/11d4e4d4-71ba-48aa-ae73-e6b6dc32b11b/9b31d439-c2fe-44d5-bcd7-596f029a918d"
+					(reference "#PWR037")
+					(unit 1)
+				)
+			)
+		)
+	)
+	(symbol
 		(lib_id "power:GND")
 		(at 143.51 349.25 90)
@@
 		(dnp no)
 		(fields_autoplaced yes)
-		(property "Reference" "#PWR04"
+		(property "Reference" "#PWR05"
 			(at 62.23 314.96 0)
 			(hide yes)
@@
 			(project "uranus-fpga-board"
 				(path "/11d4e4d4-71ba-48aa-ae73-e6b6dc32b11b/9b31d439-c2fe-44d5-bcd7-596f029a918d"
-					(reference "#PWR04")
+					(reference "#PWR05")
 					(unit 1)
 				)
@@
 	)
 	(symbol
+		(lib_id "power:+1V5")
+		(at 699.77 156.21 90)
+		(mirror x)
+		(unit 1)
+		(body_style 1)
+		(exclude_from_sim no)
+		(in_bom yes)
+		(on_board yes)
+		(in_pos_files yes)
+		(dnp no)
+		(fields_autoplaced yes)
+		(property "Reference" "#PWR033"
+			(at 703.58 156.21 0)
+			(hide yes)
+			(show_name no)
+			(do_not_autoplace no)
+			(effects
+				(font
+					(size 1.27 1.27)
+				)
+			)
+		)
+		(property "Value" "VADJ_P"
+			(at 695.96 156.2099 90)
+			(show_name no)
+			(do_not_autoplace no)
+			(effects
+				(font
+					(size 1.27 1.27)
+				)
+				(justify left)
+			)
+		)
+		(property "Footprint" ""
+			(at 699.77 156.21 0)
+			(hide yes)
+			(show_name no)
+			(do_not_autoplace no)
+			(effects
+				(font
+					(size 1.27 1.27)
+				)
+			)
+		)
+		(property "Datasheet" ""
+			(at 699.77 156.21 0)
+			(hide yes)
+			(show_name no)
+			(do_not_autoplace no)
+			(effects
+				(font
+					(size 1.27 1.27)
+				)
+			)
+		)
+		(property "Description" "Power symbol creates a global label with name \"+1V5\""
+			(at 699.77 156.21 0)
+			(hide yes)
+			(show_name no)
+			(do_not_autoplace no)
+			(effects
+				(font
+					(size 1.27 1.27)
+				)
+			)
+		)
+		(pin "1"
+		)
+		(instances
+			(project "uranus-fpga-board"
+				(path "/11d4e4d4-71ba-48aa-ae73-e6b6dc32b11b/9b31d439-c2fe-44d5-bcd7-596f029a918d"
+					(reference "#PWR033")
+					(unit 1)
+				)
+			)
+		)
+	)
+	(symbol
 		(lib_id "power:GND")
 		(at 181.61 356.87 90)
@@
 					(unit 1)
 				)
-			)
-		)
-	)
-	(symbol
-		(lib_id "power:+1V0")
-		(at 699.77 156.21 90)
-		(unit 1)
-		(body_style 1)
-		(exclude_from_sim no)
-		(in_bom yes)
-		(on_board yes)
-		(in_pos_files yes)
-		(dnp no)
-		(fields_autoplaced yes)
-		(property "Reference" "#PWR033"
-			(at 703.58 156.21 0)
-			(hide yes)
-			(show_name no)
-			(do_not_autoplace no)
-			(effects
-				(font
-					(size 1.27 1.27)
-				)
-			)
-		)
-		(property "Value" "+2V5"
-			(at 695.96 156.2101 90)
-			(show_name no)
-			(do_not_autoplace no)
-			(effects
-				(font
-					(size 1.27 1.27)
-				)
-				(justify left)
-			)
-		)
-		(property "Footprint" "Package_DFN_QFN:Renesas_UQFN-16_2x2mm_P0.4mm"
-			(at 699.77 156.21 0)
-			(hide yes)
-			(show_name no)
-			(do_not_autoplace no)
-			(effects
-				(font
-					(size 1.27 1.27)
-				)
-			)
-		)
-		(property "Datasheet" ""
-			(at 699.77 156.21 0)
-			(hide yes)
-			(show_name no)
-			(do_not_autoplace no)
-			(effects
-				(font
-					(size 1.27 1.27)
-				)
-			)
-		)
-		(property "Description" "Power symbol creates a global label with name \"+1V0\""
-			(at 699.77 156.21 0)
-			(hide yes)
-			(show_name no)
-			(do_not_autoplace no)
-			(effects
-				(font
-					(size 1.27 1.27)
-				)
-			)
-		)
-		(pin "1"
-		)
-		(instances
-			(project "uranus-fpga-board"
-				(path "/11d4e4d4-71ba-48aa-ae73-e6b6dc32b11b/9b31d439-c2fe-44d5-bcd7-596f029a918d"
-					(reference "#PWR033")
-					(unit 1)
-				)

Commit message: big things happening in JOURNAL
Parts:
- added C17, C20: 47 μF, symbol Device:C
- C12: value C_Small -> 4.7 μF
- U1: value XC7K325T-3FFG900E -> XC7K325T; MANUFACTURER (none) -> AMD; MP (none) -> XC7K325T-3FFG900E
- renumbered C17 to C18, C18 to C19, C20 to C21, C21 to C22, C22 to C23, C19 to C24
Connections:
- net +2V5: no longer C18.1, C19.1
- net +3V3: now also C20.1
- net GND: now also C17.2, C20.2
- net VADJ_P renamed VADJ
- net VADJ: now also C18.1, C19.1, C17.1
Other:
- note added: "VCCO_15"
- note added: "VCCO_18"
- note removed: "100 μF"
- note removed: "330 μF"
- note removed: "4.7 μF"
- note removed: "47 μF"
- moved on the sheet: U1B, U1H
