File: KiCad/uranus-fpga-board/fpga.kicad_sch (KiCad schematic)
At the start: 25 parts, among them U1 XC7K325T

Commit message: big things happening in schematic quality
Other:
- added sheet Config (fpga_config.kicad_sch)
- added sheet GTX (fpga_gtx.kicad_sch)
- added sheet IO Banks (fpga_io_banks.kicad_sch)
- added sheet Power (fpga_power.kicad_sch)

Commit message: Big things have mostly happened in schematic quality
Parts:
- removed C1, C2, C3: 330 μF, symbol Device:C
- removed C10, C11, C12, C13, C9: 4.7 μF, symbol Device:C_Small
- removed C14, C15, C16, C17, C18, C19, C20, C21, C22, C23, C24, C4, C5, C6: 47 μF, symbol Device:C
- removed C7, C8: 100 μF, symbol Device:C
Other:
- sheet Config ports: added {FMC_JTAG}; removed none
- sheet GTX ports: added {FMC_GTXCLK}, {FMC_GTXDB}; removed none
- sheet IO Banks ports: added IDC_B13_CLK, IDC_B13_WRT, IDC_B14_CLK, IDC_B14_WRT, {FMC_CLK}, {FMC_DB_B16}, {FMC_DB_B17}, {FMC_DB_B18}, {FMC_I2C}; removed none
- note removed: "VCCAUX"
- note removed: "VCCAUX_IO"
- note removed: "VCCBRAM"
- note removed: "VCCINT"
- note removed: "VCCO_0"
- note removed: "VCCO_15"
- note removed: "VCCO_16"
- note removed: "VCCO_17"
- note removed: "VCCO_18"
- note removed: "VCCO_32"
- note removed: "VCCO_33"
- note removed: "VCCO_34"

Commit message: I finally did it
Parts:
- removed U1: XC7K325T, XC7K325T-3FFG900E:FFG900XC7K325T_AMD, symbol 2026-10-05_20-13-35:XC7K325T-3FFG900E
Other:
- sheet IO Banks ports: added J2_B13{DB}, J2_B15{DB}, {I2C}; removed B13{IDC_DB}, B14{IDC_DB}, {FMC_I2C}
