File: KiCad/uranus-fpga-board/highspeed.kicad_sch (KiCad schematic)
At the start: 2 parts, among them J2 ASP-134488-01

Commit message: New entry and schematic
Parts:
- removed R14: 10kΩ, ASP-134488-01:SAMTEC_ASP-134488-01, symbol Device:R
- added J2: TYPE-C-31-M-12, Connector_USB:USB_C_Receptacle_HRO_TYPE-C-31-M-12, symbol Connector:USB_C_Receptacle_USB2.0_16P
- added U6: FT232HL-REEL, FT232HL:LQFP48_FT232HL_FTD, symbol 2026-10-10_17-23-44:FT232HL-REEL
- added U7: 93LC56BT, Package_TO_SOT_SMD:SOT-23-6, symbol Memory_EEPROM:93LCxxAxxOT
- added U8: USBLC6-2SC6, Package_TO_SOT_SMD:SOT-23-6, symbol Battery_Management:BQ21040DBV
- added U9: W25Q128JVSIQ, SOIC_128JVSIQ_WIN, symbol 2026-10-10_22-05-10:W25Q128JVSIQ
- added Y2: 3225-12-20-10-10/4B, Crystal:Crystal_SMD_3225-4Pin_3.2x2.5mm, symbol Oscillator:ASE-xxxMHz
- J1: renamed from J2; footprint ASP-134488-01:SAMTEC_ASP-134488-01 -> Connector_Samtec:Samtec_FMC_ASP-134486-01_10x40_P1.27mm_Vertical
Connections:
- net GND: now also Y2.2 (GND); no longer J1.A1, J1.A12, J1.A13, J1.A16, J1.A17, J1.A20, J1.A21, J1.A24, J1.A25, J1.A28, J1.A29, J1.A32, J1.A33, J1.A36, J1.A37, J1.A4, J1.A40, J1.A5, J1.A8, J1.A9, J1.B10, J1.B11, J1.B14, J1.B15, J1.B18, J1.B19, J1.B2, J1.B22, J1.B23, J1.B26, J1.B27, J1.B3, J1.B30, J1.B31, J1.B34, J1.B35, J1.B38, J1.B39, J1.B6, J1.B7, J1.C1, J1.C12, J1.C13, J1.C16, J1.C17, J1.C20, J1.C21, J1.C24, J1.C25, J1.C28, J1.C29, J1.C32, J1.C33, J1.C36, J1.C38, J1.C4, J1.C40, J1.C5, J1.C8, J1.C9, J1.D10, J1.D13, J1.D16, J1.D19, J1.D2, J1.D22, J1.D25, J1.D28, J1.D3, J1.D37, J1.D39, J1.D6, J1.D7, J1.E1, J1.E11, J1.E14, J1.E17, J1.E20, J1.E23, J1.E26, J1.E29, J1.E32, J1.E35, J1.E38, J1.E4, J1.E40, J1.E5, J1.E8, J1.F12, J1.F15, J1.F18, J1.F2, J1.F21, J1.F24, J1.F27, J1.F3, J1.F30, J1.F33, J1.F36, J1.F39, J1.F6, J1.F9, J1.G1, J1.G11, J1.G14, J1.G17, J1.G20, J1.G23, J1.G26, J1.G29, J1.G32, J1.G35, J1.G38, J1.G4, J1.G40, J1.G5, J1.G8, J1.H12, J1.H15, J1.H18, J1.H21, J1.H24, J1.H27, J1.H3, J1.H30, J1.H33, J1.H36, J1.H39, J1.H6, J1.H9, J1.J1, J1.J11, J1.J14, J1.J17, J1.J20, J1.J23, J1.J26, J1.J29, J1.J32, J1.J35, J1.J38, J1.J4, J1.J40, J1.J5, J1.J8, J1.K12, J1.K15, J1.K18, J1.K2, J1.K21, J1.K24, J1.K27, J1.K3, J1.K30, J1.K33, J1.K36, J1.K39, J1.K6, J1.K9
- net LS2: now reaches J1.H1
- net +12V0: no longer names the net of J1.C37
- net +12V0: no longer J1.C35
- removed net +3V3: J1.C39, J1.D36, J1.D38, J1.D40
- net +3V3AUX renamed DATA17_P
- net CLK0_M2C_N renamed DATA29_N
- net CLK0_M2C_P renamed DATA29_P
- net CLK1_M2C_N renamed DATA19_N
- net CLK1_M2C_P renamed DATA19_P
- net CLK2_BIDIR_N: no longer names the net of J1.K5
- net CLK2_BIDIR_P: no longer names the net of J1.K4
- net CLK3_BIDIR_N: no longer names the net of J1.J3
- net CLK3_BIDIR_P: no longer names the net of J1.J2
- net CLK_DIR: no longer names the net of J1.B1
- net DP0_C2M_N renamed DATA0_N
- net DP0_C2M_P renamed DATA0_P
- net DP0_M2C_N renamed DATA1_N
- net DP0_M2C_P renamed DATA1_P
- net DP1_C2M_N: no longer names the net of J1.A23
- net DP1_C2M_P: no longer names the net of J1.A22
- net DP1_M2C_N: no longer names the net of J1.A3
- net DP1_M2C_P: no longer names the net of J1.A2
- net DP2_C2M_N: no longer names the net of J1.A27
- net DP2_C2M_P: no longer names the net of J1.A26
- net DP2_M2C_N: no longer names the net of J1.A7
- net DP2_M2C_P: no longer names the net of J1.A6
- net DP3_C2M_N: no longer names the net of J1.A31
- net DP3_C2M_P: no longer names the net of J1.A30
- net DP3_M2C_N: no longer names the net of J1.A11
- net DP3_M2C_P: no longer names the net of J1.A10
- net DP4_C2M_N: no longer names the net of J1.A35
- net DP4_C2M_P: no longer names the net of J1.A34
- net DP4_M2C_N: no longer names the net of J1.A15
- net DP4_M2C_P: no longer names the net of J1.A14
- net DP5_C2M_N: no longer names the net of J1.A39
- net DP5_C2M_P: no longer names the net of J1.A38
- net DP5_M2C_N: no longer names the net of J1.A19
- net DP5_M2C_P: no longer names the net of J1.A18
- net DP6_C2M_N: no longer names the net of J1.B37
- net DP6_C2M_P: no longer names the net of J1.B36
- net DP6_M2C_N: no longer names the net of J1.B17
- net DP6_M2C_P: no longer names the net of J1.B16
- net DP7_C2M_N: no longer names the net of J1.B33
- net DP7_C2M_P: no longer names the net of J1.B32
- net DP7_M2C_N: no longer names the net of J1.B13
- net DP7_M2C_P: no longer names the net of J1.B12
- net DP8_C2M_N: no longer names the net of J1.B29
- net DP8_C2M_P: no longer names the net of J1.B28
- net DP8_M2C_N: no longer names the net of J1.B9
- net DP8_M2C_P: no longer names the net of J1.B8
- net DP9_C2M_N: no longer names the net of J1.B25
- net DP9_C2M_P: no longer names the net of J1.B24
- net DP9_M2C_N: no longer names the net of J1.B5
- net DP9_M2C_P: no longer names the net of J1.B4
- net FMC_DETECT: no longer names the net of J1.H2
- net GA0 renamed DATA8_P
- net GA1: no longer names the net of J1.D35
- net GPTCLK0_M2C_P renamed DATA10_N
- net DATA10_N: no longer J1.D4
- net GPT_CLK1_M2C_N: no longer names the net of J1.B21
- net GPT_CLK1_M2C_P: no longer names the net of J1.B20
- net HA00_N_CC: no longer names the net of J1.F5
- net HA00_P_CC: no longer names the net of J1.F4
- net HA01_N_CC: no longer names the net of J1.E3
- net HA01_P_CC: no longer names the net of J1.E2
- net HA02_N: no longer names the net of J1.K8
- net HA02_P: no longer names the net of J1.K7
- net HA03_N: no longer names the net of J1.J7
- net HA03_P: no longer names the net of J1.J6
- net HA04_N: no longer names the net of J1.F8
- net HA04_P: no longer names the net of J1.F7
- net HA05_N: no longer names the net of J1.E7
- net HA05_P: no longer names the net of J1.E6
- net HA06_N: no longer names the net of J1.K11
- net HA06_P: no longer names the net of J1.K10
- net HA07_N: no longer names the net of J1.J10
- net HA07_P: no longer names the net of J1.J9
- net HA08_N: no longer names the net of J1.F11
- net HA08_P: no longer names the net of J1.F10
- net HA09_N: no longer names the net of J1.E10
- net HA09_P: no longer names the net of J1.E9
- net HA10_N: no longer names the net of J1.K14
- net HA10_P: no longer names the net of J1.K13
- net HA11_N: no longer names the net of J1.J13
- net HA11_P: no longer names the net of J1.J12
- net HA12_N: no longer names the net of J1.F14
- net HA12_P: no longer names the net of J1.F13
- net HA13_N: no longer names the net of J1.E13
- net HA13_P: no longer names the net of J1.E12
- net HA14_N: no longer names the net of J1.J16
- net HA14_P: no longer names the net of J1.J15
- net HA15_N: no longer names the net of J1.F17
- net HA15_P: no longer names the net of J1.F16
- net HA16_N: no longer names the net of J1.E16
- net HA16_P: no longer names the net of J1.E15
- net HA17_N_CC: no longer names the net of J1.K17
- net HA17_P_CC: no longer names the net of J1.K16
- net HA18_N: no longer names the net of J1.J19
- net HA18_P: no longer names the net of J1.J18
- net HA19_N: no longer names the net of J1.F20
- net HA19_P: no longer names the net of J1.F19
- net HA20_N: no longer names the net of J1.E19
- net HA20_P: no longer names the net of J1.E18
- net HA21_N: no longer names the net of J1.K20
- net HA21_P: no longer names the net of J1.K19
- net HA22_N: no longer names the net of J1.J22
- net HA22_P: no longer names the net of J1.J21
- net HA23_N: no longer names the net of J1.K23
- net HA23_P: no longer names the net of J1.K22
- net HB00_N_CC: no longer names the net of J1.K26
- net HB00_P_CC: no longer names the net of J1.K25
- net HB01_N: no longer names the net of J1.J25
- net HB01_P: no longer names the net of J1.J24
- net HB02_N: no longer names the net of J1.F23
- net HB02_P: no longer names the net of J1.F22
- net HB03_N: no longer names the net of J1.E22
- net HB03_P: no longer names the net of J1.E21
- net HB04_N: no longer names the net of J1.F26
- net HB04_P: no longer names the net of J1.F25
- net HB05_N: no longer names the net of J1.E25
- net HB05_P: no longer names the net of J1.E24
- net HB06_N: no longer names the net of J1.K29
- net HB06_P: no longer names the net of J1.K28
- net HB07_N: no longer names the net of J1.J28
- net HB07_P: no longer names the net of J1.J27
- net HB08_N: no longer names the net of J1.F29
- net HB08_P: no longer names the net of J1.F28
- net HB09_N: no longer names the net of J1.E28
- net HB09_P: no longer names the net of J1.E27
- net HB10_N: no longer names the net of J1.K32
- net HB10_P: no longer names the net of J1.K31
- net HB11_N: no longer names the net of J1.J31
- net HB11_P: no longer names the net of J1.J30
- net HB12_N: no longer names the net of J1.F32
- net HB12_P: no longer names the net of J1.F31
- net HB13_N: no longer names the net of J1.E31
- net HB13_P: no longer names the net of J1.E30
- net HB14_N: no longer names the net of J1.K35
- net HB14_P: no longer names the net of J1.K34
- net HB15_N: no longer names the net of J1.F35
- net HB15_N: no longer J1.J34
- net HB15_P: no longer names the net of J1.F34
- net HB15_P: no longer J1.J33
- net HB17_N_CC: no longer names the net of J1.K38
- net HB17_P_CC: no longer names the net of J1.K37
- net HB18_N: no longer names the net of J1.J37
- net HB18_P: no longer names the net of J1.J36
- net HB19_N: no longer names the net of J1.E34
- net HB19_P: no longer names the net of J1.E33
- net HB20_N: no longer names the net of J1.F38
- net HB20_P: no longer names the net of J1.F37
- net HB21_N: no longer names the net of J1.E37
- net HB21_P: no longer names the net of J1.E36
- net LA00_N_CC renamed DATA20_N
- net LA00_P_CC renamed DATA20_P
- net LA01_N_CC renamed DATA11_N
- net LA01_P_CC renamed DATA11_P
- net LA02_N renamed DATA30_P
- net LA02_P: no longer names the net of J1.H7
- net LA03_N renamed DATA21_P
- net LA03_P: no longer names the net of J1.G9
- net LA04_N: no longer names the net of J1.H11
- net LA04_P: no longer names the net of J1.H10
- net LA05_N renamed DATA12_P
- net LA05_P: no longer names the net of J1.D11
- net LA06_N renamed DATA2_N
- net LA06_P renamed DATA2_P
- net LA07_N: no longer names the net of J1.H14
- net LA07_P renamed DATA31_N
- net LA08_N: no longer names the net of J1.G13
- net LA08_P: no longer names the net of J1.G12
- net LA09_N: no longer names the net of J1.D15
- net LA09_P: no longer names the net of J1.D14
- net LA10_N renamed DATA3_N
- net LA10_P renamed DATA3_P
- net LA11_N renamed CLK0_N
- net LA11_P renamed CLK0_P
- net LA12_N: no longer names the net of J1.G16
- net LA12_P renamed DATA22_N
- net LA13_N: no longer names the net of J1.D18
- net LA13_P renamed DATA13_N
- net LA14_N renamed DATA4_N
- net LA14_P renamed DATA4_P
- net LA15_N renamed GPIO0
- net LA15_P: no longer names the net of J1.H19
- net LA16_N renamed DATA23_N
- net LA16_P renamed DATA23_P
- net LA17_N_CC renamed DATA14_N
- net LA17_P_CC renamed DATA14_P
- net LA18_N_CC renamed DATA5_N
- net LA18_P_CC renamed DATA5_P
- net LA19_N: no longer names the net of J1.H23
- net LA19_P: no longer names the net of J1.H22
- net LA20_N renamed DATA24_P
- net LA20_P: no longer names the net of J1.G21
- net LA21_N: no longer names the net of J1.H26
- net LA21_P renamed GPIO3
- net LA22_N: no longer names the net of J1.G25
- net LA22_P: no longer names the net of J1.G24
- net LA23_N renamed DATA15_P
- net LA23_P: no longer names the net of J1.D23
- net LA24_N renamed GPIO5
- net LA24_P renamed GPIO4
- net LA25_N: no longer names the net of J1.G28
- net LA25_P renamed DATA25_N
- net LA26_N: no longer names the net of J1.D27
- net LA26_P: no longer names the net of J1.D26
- net LA27_N renamed DATA6_N
- net LA27_P renamed DATA6_P
- net LA28_N renamed GPIO6
- net LA28_P: no longer names the net of J1.H31
- net LA29_N renamed DATA26_N
- net LA29_P renamed DATA26_P
- net LA30_N: no longer names the net of J1.H35
- net LA30_P: no longer names the net of J1.H34
- net LA31_N renamed DATA27_P
- net LA31_P: no longer names the net of J1.G33
- net LA32_N renamed LS4
- net LA32_P: no longer names the net of J1.H37
- net LA33_N: no longer names the net of J1.G37
- net LA33_P: no longer names the net of J1.G36
- net PG_C2M renamed LS0
- net PG_M2C: no longer names the net of J1.F1
- net RES0: no longer names the net of J1.B40
- net SCL renamed DATA7_P
- net SDA renamed DATA7_N
- net TCK renamed DATA16_N
- net TDI: no longer names the net of J1.D30
- net TDO: no longer names the net of J1.D31
- net TMS renamed DATA17_N
- net TRST_L: no longer names the net of J1.D34
- removed net VADJ: J1.E39, J1.F40, J1.G39, J1.H40
- net VIO_B_M2C: no longer names the net of J1.J39
- net VIO_B_M2C: no longer J1.K40
- new net: J2.A1 (GND), J2.A12 (GND), J2.B1 (GND), J2.B12 (GND)
- new net: J2.A4 (VBUS), J2.A9 (VBUS), J2.B4 (VBUS), J2.B9 (VBUS)
- new net DATA10_P: J1.D4
- new net DATA12_N: J1.D13
- new net DATA13_P: J1.D16
- new net DATA15_N: J1.D25
- new net DATA16_P: J1.D28
- new net DATA18_N: J1.D37
- new net DATA18_P: J1.D36
- new net DATA21_N: J1.G11
- new net DATA22_P: J1.G14
- new net DATA24_N: J1.G23
- new net DATA25_P: J1.G26
- new net DATA27_N: J1.G35
- new net DATA28_N: J1.G39
- new net DATA28_P: J1.G38
- new net DATA30_N: J1.H9
- new net DATA31_P: J1.H12
- new net DATA8_N: J1.C35
- new net DATA9_N: J1.C39
- new net DATA9_P: J1.C38
- new net GPIO1: J1.H21
- new net GPIO2: J1.H24
- new net GPIO7: J1.H33
- new net LS1: J1.D40
- new net LS3: J1.H40
- new net LS5: J1.H36
Other:
- note added: "LPC Rows"
- moved on the sheet: J1A, J1B, J1C, J1D, J1E

Commit message: New journal entry
Connections:
- net DATA12_N is gone; now on net GND: J1.D13
- net DATA13_P is gone; now on net GND: J1.D16
- net DATA15_N is gone; now on net GND: J1.D25
- net DATA16_P is gone; now on net GND: J1.D28
- net DATA18_N is gone; now on net GND: J1.D37
- net DATA18_P is gone; now on net +3V3: J1.D36
- net DATA21_N is gone; now on net GND: J1.G11
- net DATA22_P is gone; now on net GND: J1.G14
- net DATA24_N is gone; now on net GND: J1.G23
- net DATA25_P is gone; now on net GND: J1.G26
- net DATA27_N is gone; now on net GND: J1.G35
- net DATA28_P is gone; now on net GND: J1.G38
- net DATA30_N is gone; now on net GND: J1.H9
- net DATA31_P is gone; now on net GND: J1.H12
- net DATA8_N is gone; now on net +12V0: J1.C35
- net DATA9_N is gone; now on net +3V3: J1.C39
- net DATA9_P is gone; now on net GND: J1.C38
- net GPIO1 is gone; now on net GND: J1.H21
- net GPIO2 is gone; now on net GND: J1.H24
- net GPIO7 is gone; now on net GND: J1.H33
- net LS1 is gone; now on net +3V3: J1.D40
- net LS3 is gone; now on net VADJ: J1.H40
- net LS5 is gone; now on net GND: J1.H36
- net GND: now also J1.C1, J1.C12, J1.C13, J1.C16, J1.C17, J1.C20, J1.C21, J1.C24, J1.C25, J1.C28, J1.C29, J1.C32, J1.C33, J1.C36, J1.C4, J1.C40, J1.C5, J1.C8, J1.C9, J1.D10, J1.D19, J1.D2, J1.D22, J1.D3, J1.D39, J1.D6, J1.D7, J1.G1, J1.G17, J1.G20, J1.G29, J1.G32, J1.G4, J1.G40, J1.G5, J1.G8, J1.H15, J1.H18, J1.H27, J1.H3, J1.H30, J1.H39, J1.H6
- net LA08_P: now reaches J1.G12
- net LA08_N: now reaches J1.G13
- net LA12_N: now reaches J1.G16
- net LA20_P: now reaches J1.G21
- net LA22_P: now reaches J1.G24
- net LA22_N: now reaches J1.G25
- net LA25_N: now reaches J1.G28
- net LA31_P: now reaches J1.G33
- net LA33_P: now reaches J1.G36
- net LA33_N: now reaches J1.G37
- net LA03_P: now reaches J1.G9
- net LA04_P: now reaches J1.H10
- net LA04_N: now reaches J1.H11
- net LA07_N: now reaches J1.H14
- net LA15_P: now reaches J1.H19
- net PRSNT_M2C_L: now reaches J1.H2
- net LA19_P: now reaches J1.H22
- net LA19_N: now reaches J1.H23
- net LA21_N: now reaches J1.H26
- net LA28_P: now reaches J1.H31
- net LA30_P: now reaches J1.H34
- net LA30_N: now reaches J1.H35
- net LA32_P: now reaches J1.H37
- net LA02_P: now reaches J1.H7
- net +12V0: now reaches J1.C37
- net LA05_P: now reaches J1.D11
- net LA09_P: now reaches J1.D14
- net LA09_N: now reaches J1.D15
- net LA13_N: now reaches J1.D18
- net LA23_P: now reaches J1.D23
- net LA26_P: now reaches J1.D26
- net LA26_N: now reaches J1.D27
- net TDI: now reaches J1.D30
- net TDO: now reaches J1.D31
- net TRST_L: now reaches J1.D34
- net GA1: now reaches J1.D35
- net +3V3: now reaches J1.D38
- net CLK0_N renamed LA11_N
- net CLK0_P renamed LA11_P
- net DATA0_N renamed DP0_C2M_N
- net DATA0_P renamed DP0_C2M_P
- net DATA10_N renamed GBTCLK0_M2C_N
- net DATA10_P renamed GPTCLK0_M2C_P
- net DATA11_N renamed LA01_N
- net DATA11_P renamed LA01_P
- net DATA12_P renamed LA05_N
- net DATA13_N renamed LA13_P
- net DATA14_N renamed LA17_CC_N
- net DATA14_P renamed LA17_CC_P
- net DATA15_P renamed LA23_N
- net DATA16_N renamed TCK
- net DATA17_N renamed TMS
- net DATA17_P renamed +3V3AUX
- net DATA19_N renamed CLK1_M2C_N
- net DATA19_P renamed CLK1_M2C_P
- net DATA1_N renamed DP0_M2C_N
- net DATA1_P renamed DP0_M2C_P
- net DATA20_N renamed LA00_CC_N
- net DATA20_P renamed LA00_CC_P
- net DATA21_P renamed LA03_N
- net DATA22_N renamed LA12_P
- net DATA23_N renamed LA16_N
- net DATA23_P renamed LA16_P
- net DATA24_P renamed LA20_N
- net DATA25_N renamed LA25_P
- net DATA26_N renamed LA29_N
- net DATA26_P renamed LA29_P
- net DATA27_P renamed LA31_N
- net DATA28_N renamed VADJ
- net DATA29_N renamed CLK0_M2C_N
- net DATA29_P renamed CLK0_M2C_P
- net DATA2_N renamed LA06_N
- net DATA2_P renamed LA06_P
- net DATA30_P renamed LA02_N
- net DATA31_N renamed LA07_P
- net DATA3_N renamed LA10_N
- net DATA3_P renamed LA10_P
- net DATA4_N renamed LA14_N
- net DATA4_P renamed LA14_P
- net DATA5_N renamed LA18_CC_N
- net DATA5_P renamed LA18_CC_P
- net DATA6_N renamed LA27_N
- net DATA6_P renamed LA27_P
- net DATA7_N renamed SDA
- net DATA7_P renamed SCL
- net DATA8_P renamed GA0
- net GPIO0 renamed LA15_N
- net GPIO3 renamed LA21_P
- net GPIO4 renamed LA24_P
- net GPIO5 renamed LA24_N
- net GPIO6 renamed LA28_N
- net LS0 renamed PG_C2M
- net LS2 renamed VREF_A_M2C
- net LS4 renamed LA32_N

Commit message: New journal entry, progress on schematic and PCB
Parts:
- removed J1: ASP-134488-01, Connector_Samtec:Samtec_FMC_ASP-134486-01_10x40_P1.27mm_Vertical, symbol ASP-134488-01:ASP-134488-01
- added J1: 1040100018, Connector_PinHeader_1.27mm:PinHeader_2x25_P1.27mm_Vertical_SMD, symbol Connector_Generic:Conn_02x25_Odd_Even
- added J4: ASP-134486-01, ASP-134486-01:SAMTEC_ASP-134486-01, symbol ASP-134486-01:ASP-134486-01
Connections:
- net +12V0: now also J4.C35, J4.C37
- net +3V3: now also J4.C39, J4.D36, J4.D38, J4.D40
- net +3V3AUX: now also J4.D32
- net CLK0_M2C_N: now also J4.H05
- net CLK0_M2C_P: now also J4.H04
- net CLK1_M2C_N: now also J4.G03
- net CLK1_M2C_P: now also J4.G02
- net DP0_C2M_N: now also J4.C03
- net DP0_C2M_P: now also J4.C02
- net DP0_M2C_N: now also J4.C07
- net DP0_M2C_P: now also J4.C06
- net GA0: now also J4.C34
- net GA1: now also J4.D35
- net GBTCLK0_M2C_N: now also J4.D05
- net GND: now also J1.1 (Pin_1), J1.17 (Pin_17), J1.18 (Pin_18), J1.2 (Pin_2), J1.33 (Pin_33), J1.34 (Pin_34), J1.37 (Pin_37), J1.38 (Pin_38), J1.41 (Pin_41), J1.42 (Pin_42), J1.45 (Pin_45), J1.46 (Pin_46), J1.49 (Pin_49), J1.50 (Pin_50), J4.C01, J4.C04, J4.C05, J4.C08, J4.C09, J4.C12, J4.C13, J4.C16, J4.C17, J4.C20, J4.C21, J4.C24, J4.C25, J4.C28, J4.C29, J4.C32, J4.C33, J4.C36, J4.C38, J4.C40, J4.D02, J4.D03, J4.D06, J4.D07, J4.D10, J4.D13, J4.D16, J4.D19, J4.D22, J4.D25, J4.D28, J4.D37, J4.D39, J4.G01, J4.G04, J4.G05, J4.G08, J4.G11, J4.G14, J4.G17, J4.G20, J4.G23, J4.G26, J4.G29, J4.G32, J4.G35, J4.G38, J4.G40, J4.H03, J4.H06, J4.H09, J4.H12, J4.H15, J4.H18, J4.H21, J4.H24, J4.H27, J4.H30, J4.H33, J4.H36, J4.H39
- net GPTCLK0_M2C_P: now also J4.D04
- net LA00_CC_N: now also J4.G07
- net LA00_CC_P: now also J4.G06
- net LA01_N: now also J4.D09
- net LA01_P: now also J4.D08
- net LA02_N: now also J4.H08
- net LA02_P: now also J4.H07
- net LA03_N: now also J4.G10
- net LA03_P: now also J4.G09
- net LA04_N: now also J4.H11
- net LA04_P: now also J4.H10
- net LA05_N: now also J4.D12
- net LA05_P: now also J4.D11
- net LA06_N: now also J4.C11
- net LA06_P: now also J4.C10
- net LA07_N: now also J4.H14
- net LA07_P: now also J4.H13
- net LA08_N: now also J4.G13
- net LA08_P: now also J4.G12
- net LA09_N: now also J4.D15
- net LA09_P: now also J4.D14
- net LA10_N: now also J4.C15
- net LA10_P: now also J4.C14
- net LA11_N: now also J4.H17
- net LA11_P: now also J4.H16
- net LA12_N: now also J4.G16
- net LA12_P: now also J4.G15
- net LA13_N: now also J4.D18
- net LA13_P: now also J4.D17
- net LA14_N: now also J4.C19
- net LA14_P: now also J4.C18
- net LA15_N: now also J4.H20
- net LA15_P: now also J4.H19
- net LA16_N: now also J4.G19
- net LA16_P: now also J4.G18
- net LA17_CC_N: now also J4.D21
- net LA17_CC_P: now also J4.D20
- net LA18_CC_N: now also J4.C23
- net LA18_CC_P: now also J4.C22
- net LA19_N: now also J4.H23
- net LA19_P: now also J4.H22
- net LA20_N: now also J4.G22
- net LA20_P: now also J4.G21
- net LA21_N: now also J4.H26
- net LA21_P: now also J4.H25
- net LA22_N: now also J4.G25
- net LA22_P: now also J4.G24
- net LA23_N: now also J4.D24
- net LA23_P: now also J4.D23
- net LA24_N: now also J4.H29
- net LA24_P: now also J4.H28
- net LA25_N: now also J4.G28
- net LA25_P: now also J4.G27
- net LA26_N: now also J4.D27
- net LA26_P: now also J4.D26
- net LA27_N: now also J4.C27
- net LA27_P: now also J4.C26
- net LA28_N: now also J4.H32
- net LA28_P: now also J4.H31
- net LA29_N: now also J4.G31
- net LA29_P: now also J4.G30
- net LA30_N: now also J4.H35
- net LA30_P: now also J4.H34
- net LA31_N: now also J4.G34
- net LA31_P: now also J4.G33
- net LA32_N: now also J4.H38
- net LA32_P: now also J4.H37
- net LA33_N: now also J4.G37
- net LA33_P: now also J4.G36
- net PG_C2M: now also J4.D01
- net PRSNT_M2C_L: now also J4.H02
- net SCL: now also J4.C30
- net SDA: now also J4.C31
- net TCK: now also J4.D29
- net TDI: now also J4.D30
- net TDO: now also J4.D31
- net TMS: now also J4.D33
- net TRST_L: now also J4.D34
- net VADJ: now also J4.G39, J4.H40
- net VREF_A_M2C: now also J4.H01
- new net CLK0: J1.43 (Pin_43)
- new net CLK1: J1.44 (Pin_44)
- new net DATA00: J1.3 (Pin_3)
- new net DATA01: J1.5 (Pin_5)
- new net DATA02: J1.7 (Pin_7)
- new net DATA03: J1.9 (Pin_9)
- new net DATA04: J1.11 (Pin_11)
- new net DATA05: J1.13 (Pin_13)
- new net DATA06: J1.15 (Pin_15)
- new net DATA07: J1.19 (Pin_19)
- new net DATA08: J1.21 (Pin_21)
- new net DATA09: J1.23 (Pin_23)
- new net DATA10: J1.25 (Pin_25)
- new net DATA11: J1.27 (Pin_27)
- new net DATA12: J1.29 (Pin_29)
- new net DATA13: J1.31 (Pin_31)
- new net DATA14: J1.35 (Pin_35)
- new net DATA15: J1.39 (Pin_39)
- new net DATA16: J1.4 (Pin_4)
- new net DATA17: J1.6 (Pin_6)
- new net DATA18: J1.8 (Pin_8)
- new net DATA19: J1.10 (Pin_10)
- new net DATA20: J1.12 (Pin_12)
- new net DATA21: J1.14 (Pin_14)
- new net DATA22: J1.16 (Pin_16)
- new net DATA23: J1.20 (Pin_20)
- new net DATA24: J1.22 (Pin_22)
- new net DATA25: J1.24 (Pin_24)
- new net DATA26: J1.26 (Pin_26)
- new net DATA27: J1.28 (Pin_28)
- new net DATA28: J1.30 (Pin_30)
- new net DATA29: J1.32 (Pin_32)
- new net DATA30: J1.36 (Pin_36)
- new net DATA31: J1.40 (Pin_40)
- new net WRT0: J1.47 (Pin_47)
- new net WRT1: J1.48 (Pin_48)
