File: KiCad/uranus-fpga-board/fpga_bank_15.kicad_sch (KiCad schematic)
At the start: 1 part, among them U20 XC7K325T-3FFG900E

Commit message: Big things have mostly happened in schematic quality
Parts:
- renumbered U20 to U12
Changed lines of the file:
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@@
 		(dnp no)
 		(fields_autoplaced yes)
-		(property "Reference" "U20"
+		(property "Reference" "U12"
 			(at 144.78 92.71 0)
 			(hide yes)
@@
 			(project "uranus-fpga-board"
 				(path "/11d4e4d4-71ba-48aa-ae73-e6b6dc32b11b/ae4670d8-3f7e-4e25-83c4-e414aeb132b8/e70af11b-d02c-4276-ba11-71fb729ac221/df160b42-b095-480e-a002-f23f31e7d2a8"
-					(reference "U20")
+					(reference "U12")
 					(unit 4)
 				)
