File: KiCad/uranus-fpga-board/fpga_banks_13_14.kicad_sch (KiCad schematic)
At the start: 1 part, among them U20 XC7K325T-3FFG900E

Commit message: Big things have mostly happened in schematic quality
Parts:
- renumbered U20 to U12
Changed lines of the file:
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@@
 		)
 	)
+	(hierarchical_label "IDC_B14_WRT"
+		(shape output)
+		(at 215.9 38.1 0)
+		(effects
+			(font
+				(size 1.27 1.27)
+			)
+			(justify left)
+		)
+	)
+	(hierarchical_label "IDC_B13_CLK"
+		(shape output)
+		(at 215.9 26.67 0)
+		(effects
+			(font
+				(size 1.27 1.27)
+			)
+			(justify left)
+		)
+	)
+	(hierarchical_label "IDC_B14_CLK"
+		(shape output)
+		(at 215.9 35.56 0)
+		(effects
+			(font
+				(size 1.27 1.27)
+			)
+			(justify left)
+		)
+	)
+	(hierarchical_label "IDC_B13_WRT"
+		(shape output)
+		(at 215.9 29.21 0)
+		(effects
+			(font
+				(size 1.27 1.27)
+			)
+			(justify left)
+		)
+	)
 	(symbol
 		(lib_name "XC7K325T-3FFG900E_1")
@@
 		(dnp no)
 		(fields_autoplaced yes)
-		(property "Reference" "U20"
+		(property "Reference" "U12"
 			(at 186.69 88.9 0)
 			(hide yes)
@@
 			(project "uranus-fpga-board"
 				(path "/11d4e4d4-71ba-48aa-ae73-e6b6dc32b11b/ae4670d8-3f7e-4e25-83c4-e414aeb132b8/e70af11b-d02c-4276-ba11-71fb729ac221/20a1cd87-7584-4a0d-9865-d63069f231d1"
-					(reference "U20")
+					(reference "U12")
 					(unit 3)
 				)
@@
 		(dnp no)
 		(fields_autoplaced yes)
-		(property "Reference" "U20"
+		(property "Reference" "U12"
 			(at 104.14 87.63 0)
 			(hide yes)
@@
 			(project "uranus-fpga-board"
 				(path "/11d4e4d4-71ba-48aa-ae73-e6b6dc32b11b/ae4670d8-3f7e-4e25-83c4-e414aeb132b8/e70af11b-d02c-4276-ba11-71fb729ac221/20a1cd87-7584-4a0d-9865-d63069f231d1"
-					(reference "U20")
+					(reference "U12")
 					(unit 2)
 				)
