File: KiCad/uranus-fpga-board/fmc_power.kicad_sch (KiCad schematic)
At the start: 31 parts, among them Q1 2N7002, U22 TMUX1108, U6 TPS2553DBVR, U7 SY6288F1ABC, U8 SY6874DBC

Commit message: Big things have mostly happened in schematic quality
Parts:
- removed C70, C74, C95: 100 nF, symbol Device:C_Small
- removed C71, C72, C73, C75: 10 μF, symbol Device:C_Small
- removed C76, C96, C98, C99: 10 nF, symbol Device:C_Small
- removed Q1: 2N7002, Package_TO_SOT_SMD:SOT-23, symbol Transistor_FET:2N7002
- removed R14: 10 kΩ, Resistor_SMD:R_0201_0603Metric, symbol Device:R
- removed R15: 200 kΩ, Resistor_SMD:R_0402_1005Metric, symbol Device:R_Small
- removed R16: 7.5 kΩ, Resistor_SMD:R_0201_0603Metric, symbol Device:R
- removed R21: 232 kΩ, Resistor_SMD:R_0402_1005Metric, symbol Device:R_Small
- removed R24, R26, R54: 57.6 kΩ, Resistor_SMD:R_0402_1005Metric, symbol Device:R_Small
- removed R49: 1.8 kΩ, Resistor_SMD:R_0402_1005Metric, symbol Device:R_Small
- removed R55: 41.2 kΩ, Resistor_SMD:R_0402_1005Metric, symbol Device:R_Small
- removed R56: 27.4 kΩ, Resistor_SMD:R_0402_1005Metric, symbol Device:R_Small
- removed R57: 21.5 kΩ, Resistor_SMD:R_0402_1005Metric, symbol Device:R_Small
- removed R58: 15.8 kΩ, Resistor_SMD:R_0402_1005Metric, symbol Device:R_Small
- removed R59, R60, R61: 200 kΩ, Resistor_SMD:R_0201_0603Metric, symbol Device:R_Small
- removed U22: TMUX1108, Package_SO:TSSOP-16_4.4x5mm_P0.65mm, symbol Analog_Switch:TMUX1108PW
- removed U6: TPS2553DBVR, Package_TO_SOT_SMD:SOT-23-6, symbol Battery_Management:BQ21040DBV
- removed U7: SY6288F1ABC, Package_TO_SOT_SMD:SOT-23-6, symbol Power_Management:AP2171W
- removed U8: SY6874DBC, Package_DFN_QFN:DFN-10-1EP_3x3mm_P0.5mm_EP1.75x2.7mm, symbol Connector_Generic:Conn_02x05_Counter_Clockwise
- added C26: 100 nF, symbol Device:C_Small
- added J1: ASP-134486-01, ASP-134486-01:SAMTEC_ASP-134486-01, symbol ASP-134486-01:ASP-134486-01
Connections:
- net +12V0: now also J1.C35 (12P0V), J1.C37 (12P0V)
- net +3V3AUX: now also J1.D32 (3P3VAUX)
- net +3V3_P: now also J1.C39 (3P3V), J1.D36 (3P3V), J1.D38 (3P3V), J1.D40 (3P3V)
- net GND: now also C26.2, J1.C01 (GND), J1.C04 (GND), J1.C05 (GND), J1.C08 (GND), J1.C09 (GND), J1.C12 (GND), J1.C13 (GND), J1.C16 (GND), J1.C17 (GND), J1.C20 (GND), J1.C21 (GND), J1.C24 (GND), J1.C25 (GND), J1.C28 (GND), J1.C29 (GND), J1.C32 (GND), J1.C33 (GND), J1.C36 (GND), J1.C38 (GND), J1.C40 (GND), J1.D02 (GND), J1.D03 (GND), J1.D06 (GND), J1.D07 (GND), J1.D10 (GND), J1.D13 (GND), J1.D16 (GND), J1.D19 (GND), J1.D22 (GND), J1.D25 (GND), J1.D28 (GND), J1.D37 (GND), J1.D39 (GND), J1.G01 (GND), J1.G04 (GND), J1.G05 (GND), J1.G08 (GND), J1.G11 (GND), J1.G14 (GND), J1.G17 (GND), J1.G20 (GND), J1.G23 (GND), J1.G26 (GND), J1.G29 (GND), J1.G32 (GND), J1.G35 (GND), J1.G38 (GND), J1.G40 (GND), J1.H03 (GND), J1.H06 (GND), J1.H09 (GND), J1.H12 (GND), J1.H15 (GND), J1.H18 (GND), J1.H21 (GND), J1.H24 (GND), J1.H27 (GND), J1.H30 (GND), J1.H33 (GND), J1.H36 (GND), J1.H39 (GND)
- new net VADJ: C26.1, J1.G39 (VADJ), J1.H40 (VADJ)
- no-connect marks 4 -> 0
Other:
- removed sheet Window Comparator +12V0_P
- removed sheet Window Comparator +3V3AUX
- removed sheet Window Comparator +3V3_P
- removed sheet Window Comparator VADJ
- note removed: "+12V0 Checker"
- note removed: "+12V0 Protector"
- note removed: "+3V3 Protector"
- note removed: "+3V3AUX Checker"
- note removed: "+3V3AUX Protector"
- note removed: "+3V3_P Checker"
- note removed: "VADJ Checker"
- note removed: "~{PRSNT} Inverter"

Commit message: I finally did it
Parts:
- renumbered C26 to C85
Changed lines of the file:
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@@
 		(in_pos_files yes)
 		(dnp no)
-		(property "Reference" "#PWR099"
+		(property "Reference" "#PWR0122"
 			(at 170.18 49.53 0)
 			(hide yes)
@@
 			(project "uranus-fpga-board"
 				(path "/11d4e4d4-71ba-48aa-ae73-e6b6dc32b11b/2757140f-486d-491c-90f5-6e7ccbeb0281/943df020-d875-4b0f-9a11-8717c8c1b835"
-					(reference "#PWR099")
+					(reference "#PWR0122")
 					(unit 1)
 				)
@@
 		(dnp no)
 		(fields_autoplaced yes)
-		(property "Reference" "#PWR095"
+		(property "Reference" "#PWR0123"
 			(at 173.99 71.12 0)
 			(hide yes)
@@
 			(project "uranus-fpga-board"
 				(path "/11d4e4d4-71ba-48aa-ae73-e6b6dc32b11b/2757140f-486d-491c-90f5-6e7ccbeb0281/943df020-d875-4b0f-9a11-8717c8c1b835"
-					(reference "#PWR095")
+					(reference "#PWR0123")
 					(unit 1)
 				)
@@
 		(in_pos_files yes)
 		(dnp no)
-		(property "Reference" "#PWR098"
+		(property "Reference" "#PWR0121"
 			(at 161.29 49.53 0)
 			(hide yes)
@@
 			(project "uranus-fpga-board"
 				(path "/11d4e4d4-71ba-48aa-ae73-e6b6dc32b11b/2757140f-486d-491c-90f5-6e7ccbeb0281/943df020-d875-4b0f-9a11-8717c8c1b835"
-					(reference "#PWR098")
+					(reference "#PWR0121")
 					(unit 1)
 				)
@@
 		(in_pos_files yes)
 		(dnp no)
-		(property "Reference" "#PWR094"
+		(property "Reference" "#PWR0124"
 			(at 177.8 49.53 0)
 			(hide yes)
@@
 			(project "uranus-fpga-board"
 				(path "/11d4e4d4-71ba-48aa-ae73-e6b6dc32b11b/2757140f-486d-491c-90f5-6e7ccbeb0281/943df020-d875-4b0f-9a11-8717c8c1b835"
-					(reference "#PWR094")
+					(reference "#PWR0124")
 					(unit 1)
 				)
@@
 		(in_pos_files yes)
 		(dnp no)
-		(property "Reference" "#PWR0100"
+		(property "Reference" "#PWR0119"
 			(at 120.65 50.8 0)
 			(hide yes)
@@
 			(project "uranus-fpga-board"
 				(path "/11d4e4d4-71ba-48aa-ae73-e6b6dc32b11b/2757140f-486d-491c-90f5-6e7ccbeb0281/943df020-d875-4b0f-9a11-8717c8c1b835"
-					(reference "#PWR0100")
+					(reference "#PWR0119")
 					(unit 1)
 				)
@@
 		(in_pos_files yes)
 		(dnp no)
-		(property "Reference" "C26"
+		(property "Reference" "C85"
 			(at 176.53 60.96 0)
 			(show_name no)
@@
 			(project "uranus-fpga-board"
 				(path "/11d4e4d4-71ba-48aa-ae73-e6b6dc32b11b/2757140f-486d-491c-90f5-6e7ccbeb0281/943df020-d875-4b0f-9a11-8717c8c1b835"
-					(reference "C26")
+					(reference "C85")
 					(unit 1)
 				)
@@
 		(dnp no)
 		(fields_autoplaced yes)
-		(property "Reference" "#PWR097"
+		(property "Reference" "#PWR0120"
 			(at 140.97 151.13 0)
 			(hide yes)
@@
 			(project "uranus-fpga-board"
 				(path "/11d4e4d4-71ba-48aa-ae73-e6b6dc32b11b/2757140f-486d-491c-90f5-6e7ccbeb0281/943df020-d875-4b0f-9a11-8717c8c1b835"
-					(reference "#PWR097")
+					(reference "#PWR0120")
 					(unit 1)
 				)
