File: KiCad/uranus-fpga-board/fmc_power_management.kicad_sch (KiCad schematic)
At the start: 31 parts, among them Q1 2N7002, U10 SY6874DBC, U11 TMUX1108, U8 TPS2553DBVR, U9 SY6288F1ABC

Commit message: I finally did it
Parts:
- renumbered C34 to C70, C36 to C71, C35 to C72, C37 to C73, C38 to C74, C39 to C75, C42 to C76, C40 to C77, C41 to C78, C43 to C79, C44 to C80, R14 to R15, R15 to R16, R16 to R17, R17 to R18, R18 to R20, R20 to R21, R28 to R22, R27 to R23, R23 to R24, R22 to R25, R24 to R26, R25 to R27, R26 to R28, R21 to R29, U10 to U6, U8 to U7, U9 to U8, U11 to U9
