File: KiCad/uranus-fpga-board/fpga_bank_12.kicad_sch (KiCad schematic)
At the start: 1 part, among them U20 XC7K325T-3FFG900E

Commit message: Big things have mostly happened in schematic quality
Parts:
- renumbered U20 to U12
Changed lines of the file:
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@@
 		(dnp no)
 		(fields_autoplaced yes)
-		(property "Reference" "U20"
+		(property "Reference" "U12"
 			(at 143.51 95.25 0)
 			(hide yes)
@@
 			(project "uranus-fpga-board"
 				(path "/11d4e4d4-71ba-48aa-ae73-e6b6dc32b11b/ae4670d8-3f7e-4e25-83c4-e414aeb132b8/e70af11b-d02c-4276-ba11-71fb729ac221/4cb2768f-bfdc-42c9-a077-fdf8ea6fb703"
-					(reference "U20")
+					(reference "U12")
 					(unit 1)
 				)

Commit message: I finally did it
Parts:
- U1: renamed from U12; footprint (none) -> Package_BGA:Xilinx_FFG900_FFG901
Changed lines of the file:
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@@
 		(dnp no)
 		(fields_autoplaced yes)
-		(property "Reference" "U12"
+		(property "Reference" "U1"
 			(at 143.51 95.25 0)
 			(hide yes)
@@
 			)
 		)
-		(property "Footprint" ""
+		(property "Footprint" "Package_BGA:Xilinx_FFG900_FFG901"
 			(at 143.51 96.52 0)
 			(hide yes)
@@
 			(project "uranus-fpga-board"
 				(path "/11d4e4d4-71ba-48aa-ae73-e6b6dc32b11b/ae4670d8-3f7e-4e25-83c4-e414aeb132b8/e70af11b-d02c-4276-ba11-71fb729ac221/4cb2768f-bfdc-42c9-a077-fdf8ea6fb703"
-					(reference "U12")
+					(reference "U1")
 					(unit 1)
 				)
