File: KiCad/uranus-fpga-board/fpga_banks_13_15.kicad_sch (KiCad schematic)
At the start: 1 part, among them U12 XC7K325T-3FFG900E

Commit message: I finally did it
Parts:
- removed unit 3 of U12
- added unit 4 of U1
- U1: renamed from U12; footprint (none) -> Package_BGA:Xilinx_FFG900_FFG901
Changed lines of the file:
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@@
 	(generator_version "10.0")
 	(paper "A4")
-	(hierarchical_label "B14{IDC_DB}"
+	(hierarchical_label "J2_B15{DB}"
 		(shape bidirectional)
 		(at 153.67 33.02 180)
@@
 		)
 	)
-	(hierarchical_label "B13{IDC_DB}"
+	(hierarchical_label "J2_B13{DB}"
 		(shape bidirectional)
 		(at 49.53 33.02 180)
@@
 	)
 	(symbol
-		(lib_name "XC7K325T-3FFG900E_1")
 		(lib_id "XC7K325T-3FFG900E:XC7K325T-3FFG900E")
-		(at 186.69 90.17 0)
-		(unit 3)
+		(at 186.69 88.9 0)
+		(unit 4)
 		(body_style 1)
 		(exclude_from_sim no)
@@
 		(dnp no)
 		(fields_autoplaced yes)
-		(property "Reference" "U12"
-			(at 186.69 88.9 0)
+		(property "Reference" "U1"
+			(at 186.69 87.63 0)
 			(hide yes)
 			(show_name no)
@@
 		)
 		(property "Value" "XC7K325T-3FFG900E"
-			(at 186.69 91.44 0)
+			(at 186.69 90.17 0)
 			(hide yes)
 			(show_name no)
@@
 			)
 		)
-		(property "Footprint" ""
-			(at 186.69 90.17 0)
+		(property "Footprint" "Package_BGA:Xilinx_FFG900_FFG901"
+			(at 186.69 88.9 0)
 			(hide yes)
 			(show_name no)
@@
 		)
 		(property "Datasheet" ""
-			(at 186.69 90.17 0)
+			(at 186.69 88.9 0)
 			(show_name no)
 			(do_not_autoplace no)
@@
 		)
 		(property "Description" "Kintex 7 T 325 XC7K325T-FFG900"
-			(at 186.69 90.17 0)
+			(at 186.69 88.9 0)
 			(hide yes)
 			(show_name no)
@@
 			(project "uranus-fpga-board"
 				(path "/11d4e4d4-71ba-48aa-ae73-e6b6dc32b11b/ae4670d8-3f7e-4e25-83c4-e414aeb132b8/e70af11b-d02c-4276-ba11-71fb729ac221/20a1cd87-7584-4a0d-9865-d63069f231d1"
-					(reference "U12")
-					(unit 3)
+					(reference "U1")
+					(unit 4)
 				)
 			)
@@
 		(dnp no)
 		(fields_autoplaced yes)
-		(property "Reference" "U12"
+		(property "Reference" "U1"
 			(at 104.14 87.63 0)
 			(hide yes)
@@
 			)
 		)
-		(property "Footprint" ""
+		(property "Footprint" "Package_BGA:Xilinx_FFG900_FFG901"
 			(at 104.14 88.9 0)
 			(hide yes)
@@
 			(project "uranus-fpga-board"
 				(path "/11d4e4d4-71ba-48aa-ae73-e6b6dc32b11b/ae4670d8-3f7e-4e25-83c4-e414aeb132b8/e70af11b-d02c-4276-ba11-71fb729ac221/20a1cd87-7584-4a0d-9865-d63069f231d1"
-					(reference "U12")
+					(reference "U1")
 					(unit 2)
 				)
