File: KiCad/uranus-fpga-board/fpga_banks_16_17_18.kicad_sch (KiCad schematic)
At the start: 1 part, among them U20 XC7K325T-3FFG900E

Commit message: Big things have mostly happened in schematic quality
Parts:
- renumbered U20 to U12
Connections:
- net LA25_N: now reaches U12.A16 (IO_L20P_T3_17)
- net LA25_P: now reaches U12.A17 (IO_L20N_T3_17)
- net LA22_P: now reaches U12.A18 (IO_L22N_T3_17)
- net LA15_N: now reaches U12.A20 (IO_L21P_T3_DQS_17)
- net LA15_P: now reaches U12.A21 (IO_L21N_T3_DQS_17)
- net LA16_N: now reaches U12.A22 (IO_L23N_T3_17)
- net LA21_P: now reaches U12.B17 (IO_L17N_T2_17)
- net LA22_N: now reaches U12.B18 (IO_L22P_T3_17)
- net LA19_P: now reaches U12.B19 (IO_L24N_T3_17)
- net LA20_P: now reaches U12.B20 (IO_L19N_T3_VREF_17)
- net LA16_P: now reaches U12.B22 (IO_L23P_T3_17)
- net LA14_N: now reaches U12.C16 (IO_L15N_T2_DQS_17)
- net LA21_N: now reaches U12.C17 (IO_L17P_T2_17)
- net LA19_N: now reaches U12.C19 (IO_L24P_T3_17)
- net LA20_N: now reaches U12.C20 (IO_L19P_T3_17)
- net LA10_N: now reaches U12.C21 (IO_L8N_T1_17)
- net LA09_N: now reaches U12.C22 (IO_L10N_T1_17)
- net LA14_P: now reaches U12.D16 (IO_L15P_T2_DQS_17)
- net LA18_CC_P: now reaches U12.D17 (IO_L13P_T2_MRCC_17)
- net LA18_CC_N: now reaches U12.D18 (IO_L13N_T2_MRCC_17)
- net LA13_N: now reaches U12.D19 (IO_L14N_T2_SRCC_17)
- net LA10_P: now reaches U12.D21 (IO_L8P_T1_17)
- net LA09_P: now reaches U12.D22 (IO_L10P_T1_17)
- net LA13_P: now reaches U12.E19 (IO_L14P_T2_SRCC_17)
- net LA30_N: now reaches U12.A11 (IO_L17P_T2_18)
- net LA30_P: now reaches U12.A12 (IO_L17N_T2_18)
- net LA31_P: now reaches U12.A13 (IO_L22N_T3_18)
- net LA29_P: now reaches U12.A15 (IO_L24N_T3_18)
- net LA33_P: now reaches U12.B12 (IO_L15N_T2_DQS_18)
- net LA31_N: now reaches U12.B13 (IO_L22P_T3_18)
- net LA29_N: now reaches U12.B14 (IO_L24P_T3_18)
- net LA24_P: now reaches U12.B15 (IO_L23N_T3_18)
- net LA32_P: now reaches U12.C11 (IO_L18N_T2_18)
- net LA33_N: now reaches U12.C12 (IO_L15P_T2_DQS_18)
- net LA28_P: now reaches U12.C14 (IO_L21N_T3_DQS_18)
- net LA24_N: now reaches U12.C15 (IO_L23P_T3_18)
- net LA32_N: now reaches U12.D11 (IO_L18P_T2_18)
- net LA17_CC_P: now reaches U12.D12 (IO_L13P_T2_MRCC_18)
- net LA17_CC_N: now reaches U12.D13 (IO_L13N_T2_MRCC_18)
- net LA28_N: now reaches U12.D14 (IO_L21P_T3_DQS_18)
- net LA26_N: now reaches U12.E11 (IO_L16N_T2_18)
- net LA27_N: now reaches U12.E14 (IO_L20P_T3_18)
- net LA27_P: now reaches U12.E15 (IO_L20N_T3_18)
- net LA23_P: now reaches U12.E16 (IO_L19N_T3_VREF_18)
- net LA26_P: now reaches U12.F11 (IO_L16P_T2_18)
- net LA23_N: now reaches U12.F15 (IO_L19P_T3_18)
- net LA11_N: now reaches U12.A23 (IO_L1N_T0_16)
- net LA07_N: now reaches U12.A27 (IO_L7N_T1_16)
- net LA08_N: now reaches U12.A28 (IO_L9N_T1_DQS_16)
- net LA03_N: now reaches U12.A30 (IO_L17N_T2_16)
- net LA11_P: now reaches U12.B23 (IO_L1P_T0_16)
- net LA12_N: now reaches U12.B24 (IO_L8N_T1_16)
- net LA07_P: now reaches U12.B27 (IO_L7P_T1_16)
- net LA08_P: now reaches U12.B28 (IO_L9P_T1_DQS_16)
- net LA04_N: now reaches U12.B29 (IO_L15N_T2_DQS_16)
- net LA03_P: now reaches U12.B30 (IO_L17P_T2_16)
- net LA12_P: now reaches U12.C24 (IO_L8P_T1_16)
- net LA00_CC_N: now reaches U12.C27 (IO_L13N_T2_MRCC_16)
- net LA04_P: now reaches U12.C29 (IO_L15P_T2_DQS_16)
- net LA02_P: now reaches U12.C30 (IO_L16N_T2_16)
- net LA05_N: now reaches U12.D23 (IO_L2N_T0_16)
- net LA06_N: now reaches U12.D24 (IO_L4N_T0_16)
- net LA00_CC_P: now reaches U12.D27 (IO_L13P_T2_MRCC_16)
- net LA02_N: now reaches U12.D29 (IO_L16P_T2_16)
- net LA05_P: now reaches U12.E23 (IO_L2P_T0_16)
- net LA06_P: now reaches U12.E24 (IO_L4P_T0_16)
- net LA01_N: now reaches U12.E29 (IO_L18P_T2_16)
- net LA01_P: now reaches U12.E30 (IO_L18N_T2_16)

Commit message: I finally did it
Parts:
- U1: renamed from U12; footprint (none) -> Package_BGA:Xilinx_FFG900_FFG901
Connections:
- net CLK0_N: now reaches U1.B25 (IO_L12N_T1_MRCC_16)
- net CLK0_P: now reaches U1.C25 (IO_L12P_T1_MRCC_16)
- net CLK1_N: now reaches U1.D28 (IO_L14N_T2_SRCC_16)
- net CLK1_P: now reaches U1.E28 (IO_L14P_T2_SRCC_16)
Changed lines of the file:
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@@
 	)
 	(bus_entry
+		(at 48.26 86.36)
+		(size 2.54 2.54)
+		(stroke
+			(width 0)
+			(type default)
+		)
+	)
+	(bus_entry
 		(at 261.62 85.09)
 		(size -2.54 2.54)
@@
 	)
 	(bus_entry
+		(at 48.26 92.71)
+		(size 2.54 2.54)
+		(stroke
+			(width 0)
+			(type default)
+		)
+	)
+	(bus_entry
 		(at 48.26 58.42)
 		(size 2.54 2.54)
@@
 	)
 	(bus_entry
+		(at 48.26 90.17)
+		(size 2.54 2.54)
+		(stroke
+			(width 0)
+			(type default)
+		)
+	)
+	(bus_entry
 		(at 48.26 153.67)
 		(size 2.54 2.54)
@@
 	)
 	(bus_entry
+		(at 48.26 83.82)
+		(size 2.54 2.54)
+		(stroke
+			(width 0)
+			(type default)
+		)
+	)
+	(bus_entry
 		(at 142.24 148.59)
 		(size -2.54 2.54)
@@
 	(bus
 		(pts
-			(xy 162.56 59.69) (xy 261.62 59.69)
+			(xy 266.7 59.69) (xy 261.62 59.69)
 		)
 		(stroke
@@
 	(wire
 		(pts
+			(xy 130.81 35.56) (xy 128.27 35.56)
+		)
+		(stroke
+			(width 0)
+			(type default)
+		)
+	)
+	(wire
+		(pts
 			(xy 50.8 45.72) (xy 62.23 45.72)
 		)
@@
 		)
 	)
+	(bus
+		(pts
+			(xy 48.26 81.28) (xy 48.26 92.71)
+		)
+		(stroke
+			(width 0)
+			(type default)
+		)
+	)
 	(wire
 		(pts
@@
 	(wire
 		(pts
+			(xy 50.8 95.25) (xy 53.34 95.25)
+		)
+		(stroke
+			(width 0)
+			(type default)
+		)
+	)
+	(wire
+		(pts
 			(xy 128.27 176.53) (xy 139.7 176.53)
 		)
@@
 	(wire
 		(pts
+			(xy 50.8 92.71) (xy 53.34 92.71)
+		)
+		(stroke
+			(width 0)
+			(type default)
+		)
+	)
+	(wire
+		(pts
 			(xy 128.27 166.37) (xy 139.7 166.37)
 		)
@@
 	(wire
 		(pts
+			(xy 130.81 33.02) (xy 128.27 33.02)
+		)
+		(stroke
+			(width 0)
+			(type default)
+		)
+	)
+	(wire
+		(pts
 			(xy 50.8 158.75) (xy 62.23 158.75)
 		)
@@
 	(wire
 		(pts
+			(xy 50.8 86.36) (xy 62.23 86.36)
+		)
+		(stroke
+			(width 0)
+			(type default)
+		)
+	)
+	(wire
+		(pts
 			(xy 50.8 156.21) (xy 62.23 156.21)
 		)
@@
 		)
 	)
+	(bus
+		(pts
+			(xy 43.18 81.28) (xy 48.26 81.28)
+		)
+		(stroke
+			(width 0)
+			(type default)
+		)
+	)
 	(wire
 		(pts
@@
 	(wire
 		(pts
+			(xy 50.8 88.9) (xy 62.23 88.9)
+		)
+		(stroke
+			(width 0)
+			(type default)
+		)
+	)
+	(wire
+		(pts
 			(xy 50.8 38.1) (xy 62.23 38.1)
 		)
@@
 		)
 	)
+	(label "CLK0_P"
+		(at 62.23 86.36 180)
+		(effects
+			(font
+				(size 1.27 1.27)
+			)
+			(justify right bottom)
+		)
+	)
 	(label "LA05_N"
 		(at 52.07 38.1 0)
@@
 		)
 	)
+	(label "CLK1_N"
+		(at 130.81 35.56 0)
+		(effects
+			(font
+				(size 1.27 1.27)
+			)
+			(justify left)
+		)
+	)
 	(label "LA05_P"
 		(at 52.07 35.56 0)
@@
 		)
 	)
+	(label "CLK0_N"
+		(at 62.23 88.9 180)
+		(effects
+			(font
+				(size 1.27 1.27)
+			)
+			(justify right bottom)
+		)
+	)
 	(label "LA13_N"
 		(at 128.27 125.73 0)
@@
 		)
 	)
+	(label "CLK1_P"
+		(at 53.34 92.71 0)
+		(effects
+			(font
+				(size 1.27 1.27)
+			)
+			(justify left)
+		)
+	)
 	(label "LA22_N"
 		(at 128.27 163.83 0)
@@
 		)
 	)
+	(label "CLK1_N"
+		(at 53.34 95.25 0)
+		(effects
+			(font
+				(size 1.27 1.27)
+			)
+			(justify left)
+		)
+	)
 	(label "LA18_CC_N"
 		(at 128.27 120.65 0)
@@
 		)
 	)
-	(hierarchical_label "{FMC_CLK}"
-		(shape input)
-		(at 25.4 13.97 180)
+	(label "CLK1_P"
+		(at 130.81 33.02 0)
 		(effects
 			(font
 				(size 1.27 1.27)
 			)
-			(justify right)
+			(justify left)
 		)
 	)
-	(hierarchical_label "{FMC_DB_B18}"
-		(shape bidirectional)
-		(at 162.56 59.69 180)
+	(hierarchical_label "{FMC_CLK}"
+		(shape input)
+		(at 43.18 81.28 180)
 		(effects
 			(font
@@
 		)
 	)
-	(hierarchical_label "{FMC_I2C}"
+	(hierarchical_label "{FMC_DB_B18}"
 		(shape bidirectional)
-		(at 25.4 21.59 180)
+		(at 266.7 59.69 0)
 		(effects
 			(font
 				(size 1.27 1.27)
 			)
-			(justify right)
+			(justify left)
 		)
 	)
@@
 		(dnp no)
 		(fields_autoplaced yes)
-		(property "Reference" "U12"
+		(property "Reference" "U1"
 			(at 95.25 147.32 0)
 			(hide yes)
@@
 			)
 		)
-		(property "Footprint" ""
+		(property "Footprint" "Package_BGA:Xilinx_FFG900_FFG901"
 			(at 95.25 148.59 0)
 			(hide yes)
@@
 			(project "uranus-fpga-board"
 				(path "/11d4e4d4-71ba-48aa-ae73-e6b6dc32b11b/ae4670d8-3f7e-4e25-83c4-e414aeb132b8/e70af11b-d02c-4276-ba11-71fb729ac221/c6904e6f-e817-4de3-b782-439e253960e0"
-					(reference "U12")
+					(reference "U1")
 					(unit 6)
 				)
@@
 		(dnp no)
 		(fields_autoplaced yes)
-		(property "Reference" "U12"
+		(property "Reference" "U1"
 			(at 214.63 93.98 0)
 			(hide yes)
@@
 			)
 		)
-		(property "Footprint" ""
+		(property "Footprint" "Package_BGA:Xilinx_FFG900_FFG901"
 			(at 214.63 95.25 0)
 			(hide yes)
@@
 			(project "uranus-fpga-board"
 				(path "/11d4e4d4-71ba-48aa-ae73-e6b6dc32b11b/ae4670d8-3f7e-4e25-83c4-e414aeb132b8/e70af11b-d02c-4276-ba11-71fb729ac221/c6904e6f-e817-4de3-b782-439e253960e0"
-					(reference "U12")
+					(reference "U1")
 					(unit 7)
 				)
@@
 		(dnp no)
 		(fields_autoplaced yes)
-		(property "Reference" "U12"
+		(property "Reference" "U1"
 			(at 95.25 57.15 0)
 			(hide yes)
@@
 			)
 		)
-		(property "Footprint" ""
+		(property "Footprint" "Package_BGA:Xilinx_FFG900_FFG901"
 			(at 95.25 58.42 0)
 			(hide yes)
@@
 			(project "uranus-fpga-board"
 				(path "/11d4e4d4-71ba-48aa-ae73-e6b6dc32b11b/ae4670d8-3f7e-4e25-83c4-e414aeb132b8/e70af11b-d02c-4276-ba11-71fb729ac221/c6904e6f-e817-4de3-b782-439e253960e0"
-					(reference "U12")
+					(reference "U1")
 					(unit 5)
 				)
