File: KiCad/uranus-fpga-board/fpga_config.kicad_sch (KiCad schematic)
At the start: 1 part, among them U20 XC7K325T-3FFG900E

Commit message: Big things have mostly happened in schematic quality
Parts:
- renumbered U20 to U12
Changed lines of the file:
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@@
 	(generator_version "10.0")
 	(paper "A4")
+	(hierarchical_label "{FMC_JTAG}"
+		(shape bidirectional)
+		(at 97.79 36.83 180)
+		(effects
+			(font
+				(size 1.27 1.27)
+			)
+			(justify right)
+		)
+	)
 	(symbol
 		(lib_name "XC7K325T-3FFG900E_12")
 		(lib_id "XC7K325T-3FFG900E:XC7K325T-3FFG900E")
 		(at 140.97 92.71 0)
+		(mirror y)
 		(unit 11)
 		(body_style 1)
@@
 		(in_pos_files yes)
 		(dnp no)
-		(fields_autoplaced yes)
-		(property "Reference" "U20"
+		(property "Reference" "U12"
 			(at 140.97 91.44 0)
 			(hide yes)
@@
 			(project "uranus-fpga-board"
 				(path "/11d4e4d4-71ba-48aa-ae73-e6b6dc32b11b/ae4670d8-3f7e-4e25-83c4-e414aeb132b8/ebe21894-3116-4927-b5b1-2b3b5358a9f8"
-					(reference "U20")
+					(reference "U12")
 					(unit 11)
 				)

Commit message: I finally did it
Parts:
- U1: renamed from U12; footprint (none) -> Package_BGA:Xilinx_FFG900_FFG901
Changed lines of the file:
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@@
 		(in_pos_files yes)
 		(dnp no)
-		(property "Reference" "U12"
+		(property "Reference" "U1"
 			(at 140.97 91.44 0)
 			(hide yes)
@@
 			)
 		)
-		(property "Footprint" ""
+		(property "Footprint" "Package_BGA:Xilinx_FFG900_FFG901"
 			(at 140.97 92.71 0)
 			(hide yes)
@@
 			(project "uranus-fpga-board"
 				(path "/11d4e4d4-71ba-48aa-ae73-e6b6dc32b11b/ae4670d8-3f7e-4e25-83c4-e414aeb132b8/ebe21894-3116-4927-b5b1-2b3b5358a9f8"
-					(reference "U12")
+					(reference "U1")
 					(unit 11)
 				)
