File: KiCad/uranus-fpga-board/fpga_io_banks.kicad_sch (KiCad schematic)
At the start: 0 parts

Commit message: Big things have mostly happened in schematic quality
Other:
- sheet 13 14 ports: added IDC_B13_CLK, IDC_B13_WRT, IDC_B14_CLK, IDC_B14_WRT; removed none
- sheet 16 17 18 ports: added {FMC_CLK}, {FMC_DB_B16}, {FMC_DB_B17}, {FMC_DB_B18}, {FMC_I2C}; removed none

Commit message: I finally did it
Other:
- sheet 13 14 renamed 13 15
- sheet 15 renamed 14
- sheet 13 15: file fpga_banks_13_14.kicad_sch -> fpga_banks_13_15.kicad_sch
- sheet 13 15 ports: added J2_B13{DB}, J2_B15{DB}; removed B13{IDC_DB}, B14{IDC_DB}
- sheet 14: file fpga_bank_15.kicad_sch -> fpga_bank_14.kicad_sch
- sheet 14 ports: added {I2C}; removed none
- sheet 16 17 18 ports: added none; removed {FMC_I2C}
Changed lines of the file:
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@@
+	(bus
+		(pts
+			(xy 210.82 63.5) (xy 213.36 63.5)
+		)
+		(stroke
+			(width 0)
+			(type default)
+		)
+	)
 	(bus
 		(pts
@@
 		)
 	)
-	(bus
-		(pts
-			(xy 140.97 76.2) (xy 143.51 76.2)
-		)
-		(stroke
-			(width 0)
-			(type default)
-		)
-	)
 	(wire
 		(pts
@@
 		)
 	)
-	(hierarchical_label "B13{IDC_DB}"
+	(hierarchical_label "J2_B13{DB}"
 		(shape bidirectional)
 		(at 60.96 111.76 180)
@@
 		)
 	)
-	(hierarchical_label "{FMC_I2C}"
-		(shape bidirectional)
-		(at 140.97 76.2 180)
+	(hierarchical_label "{I2C}"
+		(shape bidirectional)
+		(at 210.82 63.5 180)
 		(effects
 			(font
@@
 		)
 	)
-	(hierarchical_label "B14{IDC_DB}"
+	(hierarchical_label "J2_B15{DB}"
 		(shape bidirectional)
 		(at 60.96 120.65 180)
@@
 			(color 0 0 0 0)
 		)
-		(property "Sheetname" "13 14"
+		(property "Sheetname" "13 15"
 			(at 63.5 108.5084 0)
 			(show_name no)
@@
 			)
 		)
-		(property "Sheetfile" "fpga_banks_13_14.kicad_sch"
+		(property "Sheetfile" "fpga_banks_13_15.kicad_sch"
 			(at 63.5 136.4746 0)
 			(show_name no)
@@
 			)
 		)
-		(pin "B13{IDC_DB}" bidirectional
+		(pin "J2_B13{DB}" bidirectional
 			(at 63.5 111.76 180)
 			(effects
@@
 			)
 		)
-		(pin "B14{IDC_DB}" bidirectional
+		(pin "J2_B15{DB}" bidirectional
 			(at 63.5 120.65 180)
 			(effects
@@
 			(project "uranus-fpga-board"
 				(path "/11d4e4d4-71ba-48aa-ae73-e6b6dc32b11b/ae4670d8-3f7e-4e25-83c4-e414aeb132b8/e70af11b-d02c-4276-ba11-71fb729ac221"
-					(page "17")
+					(page "11")
 				)
 			)
@@
 			(project "uranus-fpga-board"
 				(path "/11d4e4d4-71ba-48aa-ae73-e6b6dc32b11b/ae4670d8-3f7e-4e25-83c4-e414aeb132b8/e70af11b-d02c-4276-ba11-71fb729ac221"
-					(page "18")
+					(page "12")
 				)
 			)
@@
 			(project "uranus-fpga-board"
 				(path "/11d4e4d4-71ba-48aa-ae73-e6b6dc32b11b/ae4670d8-3f7e-4e25-83c4-e414aeb132b8/e70af11b-d02c-4276-ba11-71fb729ac221"
-					(page "14")
+					(page "8")
 				)
 			)
@@
 			)
 		)
-		(pin "{FMC_I2C}" bidirectional
-			(at 143.51 76.2 180)
-			(effects
-				(font
-					(size 1.27 1.27)
-				)
-				(justify left)
-			)
-		)
 		(instances
 			(project "uranus-fpga-board"
 				(path "/11d4e4d4-71ba-48aa-ae73-e6b6dc32b11b/ae4670d8-3f7e-4e25-83c4-e414aeb132b8/e70af11b-d02c-4276-ba11-71fb729ac221"
-					(page "15")
+					(page "9")
 				)
 			)
@@
 			(color 0 0 0 0)
 		)
-		(property "Sheetname" "15"
+		(property "Sheetname" "14"
 			(at 213.36 55.1684 0)
 			(show_name no)
@@
 			)
 		)
-		(property "Sheetfile" "fpga_bank_15.kicad_sch"
+		(property "Sheetfile" "fpga_bank_14.kicad_sch"
 			(at 213.36 83.1346 0)
 			(show_name no)
@@
 		(pin "{VADJ_CTRL}" output
 			(at 213.36 58.42 180)
+			(effects
+				(font
+					(size 1.27 1.27)
+				)
+				(justify left)
+			)
+		)
+		(pin "{I2C}" bidirectional
+			(at 213.36 63.5 180)
 			(effects
 				(font
@@
 			(project "uranus-fpga-board"
 				(path "/11d4e4d4-71ba-48aa-ae73-e6b6dc32b11b/ae4670d8-3f7e-4e25-83c4-e414aeb132b8/e70af11b-d02c-4276-ba11-71fb729ac221"
-					(page "16")
-				)
-			)
+					(page "10")
+				)
+			)
