File: KiCad/uranus-fpga-board/fpga_power.kicad_sch (KiCad schematic)
At the start: 1 part, among them U20 XC7K325T-3FFG900E

Commit message: Big things have mostly happened in schematic quality
Parts:
- renumbered U20 to U12
Connections:
- net +1V8: no longer U12.V11 (VCCAUX_IO_G0), U12.W10 (VCCAUX_IO_G0), U12.W12 (VCCAUX_IO_G0)
- new net +2V0: U12.V11 (VCCAUX_IO_G0), U12.W10 (VCCAUX_IO_G0), U12.W12 (VCCAUX_IO_G0)
Other:
- added sheet Decoupling (fpga_power_decoupling.kicad_sch)

Commit message: I finally did it
Parts:
- U1: renamed from U12; footprint (none) -> Package_BGA:Xilinx_FFG900_FFG901
Connections:
- net +1V8: no longer U1.V15 (VCCAUX), U1.W14 (VCCAUX)
- new net: U1.V15 (VCCAUX), U1.W14 (VCCAUX)
Changed lines of the file:
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@@
 	)
 	(junction
-		(at 110.49 29.21)
-		(diameter 0)
-		(color 0 0 0 0)
-	)
-	(junction
 		(at 209.55 86.36)
 		(diameter 0)
@@
 	(wire
 		(pts
-			(xy 110.49 26.67) (xy 110.49 29.21)
+			(xy 110.49 26.67) (xy 110.49 27.94)
 		)
 		(stroke
@@
 		(dnp no)
 		(fields_autoplaced yes)
-		(property "Reference" "U12"
+		(property "Reference" "U1"
 			(at 57.15 60.96 0)
 			(hide yes)
@@
 			)
 		)
-		(property "Footprint" ""
+		(property "Footprint" "Package_BGA:Xilinx_FFG900_FFG901"
 			(at 57.15 62.23 0)
 			(hide yes)
@@
 			(project "uranus-fpga-board"
 				(path "/11d4e4d4-71ba-48aa-ae73-e6b6dc32b11b/ae4670d8-3f7e-4e25-83c4-e414aeb132b8/7b0890b0-33af-4ace-99bd-c62d0e3b3168"
-					(reference "U12")
+					(reference "U1")
 					(unit 14)
 				)
@@
 		(dnp no)
 		(fields_autoplaced yes)
-		(property "Reference" "#PWR0157"
+		(property "Reference" "#PWR013"
 			(at 88.9 24.13 0)
 			(hide yes)
@@
 			(project "uranus-fpga-board"
 				(path "/11d4e4d4-71ba-48aa-ae73-e6b6dc32b11b/ae4670d8-3f7e-4e25-83c4-e414aeb132b8/7b0890b0-33af-4ace-99bd-c62d0e3b3168"
-					(reference "#PWR0157")
+					(reference "#PWR013")
 					(unit 1)
 				)
@@
 		(dnp no)
 		(fields_autoplaced yes)
-		(property "Reference" "#PWR0155"
+		(property "Reference" "#PWR011"
 			(at 25.4 74.93 0)
 			(hide yes)
@@
 			(project "uranus-fpga-board"
 				(path "/11d4e4d4-71ba-48aa-ae73-e6b6dc32b11b/ae4670d8-3f7e-4e25-83c4-e414aeb132b8/7b0890b0-33af-4ace-99bd-c62d0e3b3168"
-					(reference "#PWR0155")
+					(reference "#PWR011")
 					(unit 1)
 				)
@@
 		(dnp no)
 		(fields_autoplaced yes)
-		(property "Reference" "#PWR0154"
+		(property "Reference" "#PWR010"
 			(at 25.4 24.13 0)
 			(hide yes)
@@
 			(project "uranus-fpga-board"
 				(path "/11d4e4d4-71ba-48aa-ae73-e6b6dc32b11b/ae4670d8-3f7e-4e25-83c4-e414aeb132b8/7b0890b0-33af-4ace-99bd-c62d0e3b3168"
-					(reference "#PWR0154")
+					(reference "#PWR010")
 					(unit 1)
 				)
@@
 		(dnp no)
 		(fields_autoplaced yes)
-		(property "Reference" "#PWR0159"
+		(property "Reference" "#PWR015"
 			(at 105.41 24.13 0)
 			(hide yes)
@@
 			(project "uranus-fpga-board"
 				(path "/11d4e4d4-71ba-48aa-ae73-e6b6dc32b11b/ae4670d8-3f7e-4e25-83c4-e414aeb132b8/7b0890b0-33af-4ace-99bd-c62d0e3b3168"
-					(reference "#PWR0159")
+					(reference "#PWR015")
 					(unit 1)
 				)
@@
 		(dnp no)
 		(fields_autoplaced yes)
-		(property "Reference" "#PWR0160"
+		(property "Reference" "#PWR017"
 			(at 105.41 49.53 0)
 			(hide yes)
@@
 			(project "uranus-fpga-board"
 				(path "/11d4e4d4-71ba-48aa-ae73-e6b6dc32b11b/ae4670d8-3f7e-4e25-83c4-e414aeb132b8/7b0890b0-33af-4ace-99bd-c62d0e3b3168"
-					(reference "#PWR0160")
+					(reference "#PWR017")
 					(unit 1)
 				)
@@
 		(dnp no)
 		(fields_autoplaced yes)
-		(property "Reference" "U12"
+		(property "Reference" "U1"
 			(at 227.33 76.2 0)
 			(hide yes)
@@
 			)
 		)
-		(property "Footprint" ""
+		(property "Footprint" "Package_BGA:Xilinx_FFG900_FFG901"
 			(at 227.33 77.47 0)
 			(hide yes)
@@
 			(project "uranus-fpga-board"
 				(path "/11d4e4d4-71ba-48aa-ae73-e6b6dc32b11b/ae4670d8-3f7e-4e25-83c4-e414aeb132b8/7b0890b0-33af-4ace-99bd-c62d0e3b3168"
-					(reference "U12")
+					(reference "U1")
 					(unit 17)
 				)
@@
 		(dnp no)
 		(fields_autoplaced yes)
-		(property "Reference" "#PWR0162"
+		(property "Reference" "#PWR019"
 			(at 105.41 76.2 0)
 			(hide yes)
@@
 			(project "uranus-fpga-board"
 				(path "/11d4e4d4-71ba-48aa-ae73-e6b6dc32b11b/ae4670d8-3f7e-4e25-83c4-e414aeb132b8/7b0890b0-33af-4ace-99bd-c62d0e3b3168"
-					(reference "#PWR0162")
+					(reference "#PWR019")
 					(unit 1)
 				)
@@
 		(dnp no)
 		(fields_autoplaced yes)
-		(property "Reference" "#PWR0163"
+		(property "Reference" "#PWR020"
 			(at 166.37 24.13 0)
 			(hide yes)
@@
 			(project "uranus-fpga-board"
 				(path "/11d4e4d4-71ba-48aa-ae73-e6b6dc32b11b/ae4670d8-3f7e-4e25-83c4-e414aeb132b8/7b0890b0-33af-4ace-99bd-c62d0e3b3168"
-					(reference "#PWR0163")
+					(reference "#PWR020")
 					(unit 1)
 				)
@@
 		(dnp no)
 		(fields_autoplaced yes)
-		(property "Reference" "U12"
+		(property "Reference" "U1"
 			(at 135.89 110.49 0)
 			(hide yes)
@@
 			)
 		)
-		(property "Footprint" ""
+		(property "Footprint" "Package_BGA:Xilinx_FFG900_FFG901"
 			(at 135.89 111.76 0)
 			(hide yes)
@@
 			(project "uranus-fpga-board"
 				(path "/11d4e4d4-71ba-48aa-ae73-e6b6dc32b11b/ae4670d8-3f7e-4e25-83c4-e414aeb132b8/7b0890b0-33af-4ace-99bd-c62d0e3b3168"
-					(reference "U12")
+					(reference "U1")
 					(unit 15)
 				)
@@
 		(dnp no)
 		(fields_autoplaced yes)
-		(property "Reference" "U12"
+		(property "Reference" "U1"
 			(at 135.89 44.45 0)
 			(hide yes)
@@
 			)
 		)
-		(property "Footprint" ""
+		(property "Footprint" "Package_BGA:Xilinx_FFG900_FFG901"
 			(at 135.89 45.72 0)
 			(hide yes)
@@
 			(project "uranus-fpga-board"
 				(path "/11d4e4d4-71ba-48aa-ae73-e6b6dc32b11b/ae4670d8-3f7e-4e25-83c4-e414aeb132b8/7b0890b0-33af-4ace-99bd-c62d0e3b3168"
-					(reference "U12")
+					(reference "U1")
 					(unit 16)
 				)
@@
 		(dnp no)
 		(fields_autoplaced yes)
-		(property "Reference" "#PWR0158"
+		(property "Reference" "#PWR014"
 			(at 88.9 57.15 0)
 			(hide yes)
@@
 			(project "uranus-fpga-board"
 				(path "/11d4e4d4-71ba-48aa-ae73-e6b6dc32b11b/ae4670d8-3f7e-4e25-83c4-e414aeb132b8/7b0890b0-33af-4ace-99bd-c62d0e3b3168"
-					(reference "#PWR0158")
+					(reference "#PWR014")
 					(unit 1)
 				)
@@
 		(dnp no)
 		(fields_autoplaced yes)
-		(property "Reference" "#PWR0161"
+		(property "Reference" "#PWR018"
 			(at 105.41 62.23 0)
 			(hide yes)
@@
 			(project "uranus-fpga-board"
 				(path "/11d4e4d4-71ba-48aa-ae73-e6b6dc32b11b/ae4670d8-3f7e-4e25-83c4-e414aeb132b8/7b0890b0-33af-4ace-99bd-c62d0e3b3168"
-					(reference "#PWR0161")
+					(reference "#PWR018")
 					(unit 1)
 				)
@@
 		(dnp no)
 		(fields_autoplaced yes)
-		(property "Reference" "#PWR0213"
+		(property "Reference" "#PWR016"
 			(at 105.41 39.37 0)
 			(hide yes)
@@
 			(project "uranus-fpga-board"
 				(path "/11d4e4d4-71ba-48aa-ae73-e6b6dc32b11b/ae4670d8-3f7e-4e25-83c4-e414aeb132b8/7b0890b0-33af-4ace-99bd-c62d0e3b3168"
-					(reference "#PWR0213")
+					(reference "#PWR016")
 					(unit 1)
 				)
@@
 		(dnp no)
 		(fields_autoplaced yes)
-		(property "Reference" "U12"
+		(property "Reference" "U1"
 			(at 265.43 74.93 0)
 			(hide yes)
@@
 			)
 		)
-		(property "Footprint" ""
+		(property "Footprint" "Package_BGA:Xilinx_FFG900_FFG901"
 			(at 265.43 76.2 0)
 			(hide yes)
@@
 			(project "uranus-fpga-board"
 				(path "/11d4e4d4-71ba-48aa-ae73-e6b6dc32b11b/ae4670d8-3f7e-4e25-83c4-e414aeb132b8/7b0890b0-33af-4ace-99bd-c62d0e3b3168"
-					(reference "U12")
+					(reference "U1")
 					(unit 18)
 				)
@@
 		(dnp no)
 		(fields_autoplaced yes)
-		(property "Reference" "#PWR0156"
+		(property "Reference" "#PWR012"
 			(at 25.4 90.17 0)
 			(hide yes)
@@
 			(project "uranus-fpga-board"
 				(path "/11d4e4d4-71ba-48aa-ae73-e6b6dc32b11b/ae4670d8-3f7e-4e25-83c4-e414aeb132b8/7b0890b0-33af-4ace-99bd-c62d0e3b3168"
-					(reference "#PWR0156")
+					(reference "#PWR012")
 					(unit 1)
 				)
@@
 		(dnp no)
 		(fields_autoplaced yes)
-		(property "Reference" "#PWR0164"
+		(property "Reference" "#PWR021"
 			(at 246.38 144.78 0)
 			(hide yes)
@@
 			(project "uranus-fpga-board"
 				(path "/11d4e4d4-71ba-48aa-ae73-e6b6dc32b11b/ae4670d8-3f7e-4e25-83c4-e414aeb132b8/7b0890b0-33af-4ace-99bd-c62d0e3b3168"
-					(reference "#PWR0164")
+					(reference "#PWR021")
 					(unit 1)
 				)
@@
 			(project "uranus-fpga-board"
 				(path "/11d4e4d4-71ba-48aa-ae73-e6b6dc32b11b/ae4670d8-3f7e-4e25-83c4-e414aeb132b8/7b0890b0-33af-4ace-99bd-c62d0e3b3168"
-					(page "28")
+					(page "4")
 				)
 			)
