File: KiCad/uranus-fpga-board/fpga_power_decoupling.kicad_sch (KiCad schematic)
At the start: 24 parts

Commit message: I finally did it
Parts:
- renumbered C13 to C1, C97 to C10, C2 to C11, C96 to C12, C1 to C13, C95 to C14, C94 to C15, C93 to C16, C23 to C17, C6 to C18, C24 to C19, C17 to C2, C5 to C20, C4 to C21, C9 to C22, C8 to C23, C7 to C24, C12 to C3, C14 to C4, C11 to C5, C15 to C6, C10 to C7, C16 to C8, C3 to C9
