File: KiCad/uranus-fpga-board/misc.kicad_sch (KiCad schematic)
At the start: 6 parts, among them J3 TYPE-C-31-M-12, U14 W25Q128JVSIQ, U15 FT232HL-REEL, U16 93LC56BT, U17 USBLC6-2SC6, Y2 3225-12-20-10-10/4B

Commit message: Big things have mostly happened in schematic quality
Parts:
- renumbered U14 to U2, U15 to U3, U16 to U4, U17 to U5, Y2 to Y1
Changed lines of the file:
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@@
 		(dnp no)
 		(fields_autoplaced yes)
-		(property "Reference" "#PWR0208"
+		(property "Reference" "#PWR0124"
 			(at 168.91 113.03 0)
 			(hide yes)
@@
 			(project "uranus-fpga-board"
 				(path "/11d4e4d4-71ba-48aa-ae73-e6b6dc32b11b/7d64c5c4-ac4a-4d73-b01d-5f6ce408deba"
-					(reference "#PWR0208")
+					(reference "#PWR0124")
 					(unit 1)
 				)
@@
 		(dnp no)
 		(fields_autoplaced yes)
-		(property "Reference" "U17"
+		(property "Reference" "U5"
 			(at 165.1 123.19 0)
 			(hide yes)
@@
 			(project "uranus-fpga-board"
 				(path "/11d4e4d4-71ba-48aa-ae73-e6b6dc32b11b/7d64c5c4-ac4a-4d73-b01d-5f6ce408deba"
-					(reference "U17")
+					(reference "U5")
 					(unit 1)
 				)
@@
 		(in_pos_files yes)
 		(dnp no)
-		(property "Reference" "Y2"
+		(property "Reference" "Y1"
 			(at 187.96 92.6398 0)
 			(hide yes)
@@
 			(project "uranus-fpga-board"
 				(path "/11d4e4d4-71ba-48aa-ae73-e6b6dc32b11b/7d64c5c4-ac4a-4d73-b01d-5f6ce408deba"
-					(reference "Y2")
+					(reference "Y1")
 					(unit 1)
 				)
@@
 		(dnp no)
 		(fields_autoplaced yes)
-		(property "Reference" "U14"
+		(property "Reference" "U2"
 			(at 78.994 122.682 0)
 			(hide yes)
@@
 			(project "uranus-fpga-board"
 				(path "/11d4e4d4-71ba-48aa-ae73-e6b6dc32b11b/7d64c5c4-ac4a-4d73-b01d-5f6ce408deba"
-					(reference "U14")
+					(reference "U2")
 					(unit 1)
 				)
@@
 		(dnp no)
 		(fields_autoplaced yes)
-		(property "Reference" "U15"
+		(property "Reference" "U3"
 			(at 116.84 17.78 0)
 			(hide yes)
@@
 			(project "uranus-fpga-board"
 				(path "/11d4e4d4-71ba-48aa-ae73-e6b6dc32b11b/7d64c5c4-ac4a-4d73-b01d-5f6ce408deba"
-					(reference "U15")
+					(reference "U3")
 					(unit 1)
 				)
@@
 		(dnp no)
 		(fields_autoplaced yes)
-		(property "Reference" "U16"
+		(property "Reference" "U4"
 			(at 118.9833 102.87 0)
 			(hide yes)
@@
 			(project "uranus-fpga-board"
 				(path "/11d4e4d4-71ba-48aa-ae73-e6b6dc32b11b/7d64c5c4-ac4a-4d73-b01d-5f6ce408deba"
-					(reference "U16")
+					(reference "U4")
 					(unit 1)
 				)

Commit message: I finally did it
Parts:
- renumbered J3 to J4, U2 to U14, U3 to U15, U4 to U16, U5 to U17, Y1 to Y2
Changed lines of the file:
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@@
 		(dnp no)
 		(fields_autoplaced yes)
-		(property "Reference" "#PWR0124"
+		(property "Reference" "#PWR0128"
 			(at 168.91 113.03 0)
 			(hide yes)
@@
 			(project "uranus-fpga-board"
 				(path "/11d4e4d4-71ba-48aa-ae73-e6b6dc32b11b/7d64c5c4-ac4a-4d73-b01d-5f6ce408deba"
-					(reference "#PWR0124")
+					(reference "#PWR0128")
 					(unit 1)
 				)
@@
 		(dnp no)
 		(fields_autoplaced yes)
-		(property "Reference" "U5"
+		(property "Reference" "U17"
 			(at 165.1 123.19 0)
 			(hide yes)
@@
 			(project "uranus-fpga-board"
 				(path "/11d4e4d4-71ba-48aa-ae73-e6b6dc32b11b/7d64c5c4-ac4a-4d73-b01d-5f6ce408deba"
-					(reference "U5")
+					(reference "U17")
 					(unit 1)
 				)
@@
 		(in_pos_files yes)
 		(dnp no)
-		(property "Reference" "Y1"
+		(property "Reference" "Y2"
 			(at 187.96 92.6398 0)
 			(hide yes)
@@
 			(project "uranus-fpga-board"
 				(path "/11d4e4d4-71ba-48aa-ae73-e6b6dc32b11b/7d64c5c4-ac4a-4d73-b01d-5f6ce408deba"
-					(reference "Y1")
+					(reference "Y2")
 					(unit 1)
 				)
@@
 		(dnp no)
 		(fields_autoplaced yes)
-		(property "Reference" "U2"
+		(property "Reference" "U14"
 			(at 78.994 122.682 0)
 			(hide yes)
@@
 			(project "uranus-fpga-board"
 				(path "/11d4e4d4-71ba-48aa-ae73-e6b6dc32b11b/7d64c5c4-ac4a-4d73-b01d-5f6ce408deba"
-					(reference "U2")
+					(reference "U14")
 					(unit 1)
 				)
@@
 		(dnp no)
 		(fields_autoplaced yes)
-		(property "Reference" "J3"
+		(property "Reference" "J4"
 			(at 121.92 135.89 0)
-			(hide yes)
 			(show_name no)
 			(do_not_autoplace no)
@@
 			(project "uranus-fpga-board"
 				(path "/11d4e4d4-71ba-48aa-ae73-e6b6dc32b11b/7d64c5c4-ac4a-4d73-b01d-5f6ce408deba"
-					(reference "J3")
+					(reference "J4")
 					(unit 1)
 				)
@@
 		(dnp no)
 		(fields_autoplaced yes)
-		(property "Reference" "U3"
+		(property "Reference" "U15"
 			(at 116.84 17.78 0)
 			(hide yes)
@@
 			(project "uranus-fpga-board"
 				(path "/11d4e4d4-71ba-48aa-ae73-e6b6dc32b11b/7d64c5c4-ac4a-4d73-b01d-5f6ce408deba"
-					(reference "U3")
+					(reference "U15")
 					(unit 1)
 				)
@@
 		(dnp no)
 		(fields_autoplaced yes)
-		(property "Reference" "U4"
+		(property "Reference" "U16"
 			(at 118.9833 102.87 0)
 			(hide yes)
@@
 			(project "uranus-fpga-board"
 				(path "/11d4e4d4-71ba-48aa-ae73-e6b6dc32b11b/7d64c5c4-ac4a-4d73-b01d-5f6ce408deba"
-					(reference "U4")
+					(reference "U16")
 					(unit 1)
 				)
