File: KiCad/uranus-fpga-board/ram_chip.kicad_sch (KiCad schematic)
At the start: 15 parts, among them U2 NT5CB64M16GP-FL

Commit message: Big things have mostly happened in schematic quality
Parts:
- removed C25, C26, C27, C28, C29, C30, C31, C32, C33: 100 nF, symbol Device:C_Small
- added C45, C46, C47, C48, C49, C50, C51, C52, C53: 100 nF, symbol Device:C
- renumbered C34 to C54, C35 to C55, R1 to R29, R2 to R30, R3 to R31, U2 to U13
Connections:
- net +1V5: now also C45.1, C46.1, C47.1, C48.1, C49.1, C50.1, C51.1, C52.1, C53.1
- net GND: now also C45.2, C46.2, C47.2, C48.2, C49.2, C50.2, C51.2, C52.2, C53.2
Other:
- moved on the sheet: C54

Commit message: I finally did it
Parts:
- renumbered C45 to C26, C46 to C27, C47 to C28, C48 to C29, C49 to C30, C50 to C31, C51 to C32, C52 to C33, C53 to C34, C54 to C35, C55 to C36, R29 to R1, R30 to R2, R31 to R3, U13 to U2
