File: KiCad/uranus-fpga-board/uranus-fpga-board.kicad_pcb (KiCad board)
At the start: 8 copper layers, 101.6 x 100.3 mm, 11 parts, among them J1 ASP-134488-01, J2 ASP-134488-01, U6 AS4C256M16D3, U7 AS4C256M16D3, U8 AS4C256M16D3, U9 AS4C256M16D3

Commit message: New entry and schematic
Parts:
- removed REF**: FFG676_XIL, footprints:FFG676_XIL
- added U1: XC7K325T-3FFG900E, XC7K325T-3FFG900E:FFG900XC7K325T_AMD, F.Cu at (113.3, 114.9)
- added U6: FT232HL-REEL, FT232HL:LQFP48_FT232HL_FTD, F.Cu at (70.6, 142.5)
- added U7: 93LC56BT, Package_TO_SOT_SMD:SOT-23-6, F.Cu at (181.7, 68.8)
- added U8: USBLC6-2SC6, Package_TO_SOT_SMD:SOT-23-6, F.Cu at (183.7, 77.4)
- added Y1: SX7DF200.000B20F30DNN, Oscillator:Oscillator_SMD_IDT_JU6-6_7.0x5.0mm_P2.54mm, F.Cu at (164.5, 67.7)
- added Y2: 3225-12-20-10-10/4B, Crystal:Crystal_SMD_3225-4Pin_3.2x2.5mm, F.Cu at (178.1, 61.9)
- J1: footprint FMC-HPC:SAMTEC_ASP-134488-01 -> Connector_Samtec:Samtec_FMC_ASP-134486-01_10x40_P1.27mm_Vertical
- J2: value ASP-134488-01 -> TYPE-C-31-M-12; footprint FMC-HPC:SAMTEC_ASP-134488-01 -> Connector_USB:USB_C_Receptacle_HRO_TYPE-C-31-M-12
- moved J2 116.5 mm to (197.7, 69.3)
- moved U3 55.9 mm to (89.4, 149.2)
- moved U4 33.9 mm to (129.0, 148.9)
- moved J1 32.8 mm to (113.9, 86.5)
- moved U2 30.8 mm to (102.1, 149.1)
- moved U5 29.3 mm to (115.1, 148.3)
- renumbered R12 to R10, R10 to R13, R9 to R4, R11 to R7, U6 to U2, U8 to U3, U9 to U4, U7 to U5
Connections:
- J1 pad C10: unconnected-(J1-PadC10) -> DATA2_P
- J1 pad C11: unconnected-(J1-PadC11) -> DATA2_N
- J1 pad C14: unconnected-(J1-PadC14) -> DATA3_P
- J1 pad C15: unconnected-(J1-PadC15) -> DATA3_N
- J1 pad C18: unconnected-(J1-PadC18) -> DATA4_P
- J1 pad C19: unconnected-(J1-PadC19) -> DATA4_N
- J1 pad C2: unconnected-(J1-PadC2) -> DATA0_P
- J1 pad C22: unconnected-(J1-PadC22) -> DATA5_P
- J1 pad C23: unconnected-(J1-PadC23) -> DATA5_N
- J1 pad C26: unconnected-(J1-PadC26) -> DATA6_P
- J1 pad C27: unconnected-(J1-PadC27) -> DATA6_N
- J1 pad C3: unconnected-(J1-PadC3) -> DATA0_N
- J1 pad C30: unconnected-(J1-PadC30) -> DATA7_P
- J1 pad C31: unconnected-(J1-PadC31) -> DATA7_N
- J1 pad C34: unconnected-(J1-PadC34) -> DATA8_P
- J1 pad C35: unconnected-(J1-PadC35) -> DATA8_N
- J1 pad C38: unconnected-(J1-PadC38) -> DATA9_P
- J1 pad C39: unconnected-(J1-PadC39) -> DATA9_N
- J1 pad C6: unconnected-(J1-PadC6) -> DATA1_P
- J1 pad C7: unconnected-(J1-PadC7) -> DATA1_N
- J1 pad D1: unconnected-(J1-PadD1) -> LS0
- J1 pad D12: unconnected-(J1-PadD12) -> DATA12_P
- J1 pad D13: unconnected-(J1-PadD13) -> DATA12_N
- J1 pad D16: unconnected-(J1-PadD16) -> DATA13_P
- J1 pad D17: unconnected-(J1-PadD17) -> DATA13_N
- J1 pad D20: unconnected-(J1-PadD20) -> DATA14_P
- J1 pad D21: unconnected-(J1-PadD21) -> DATA14_N
- J1 pad D24: unconnected-(J1-PadD24) -> DATA15_P
- J1 pad D25: unconnected-(J1-PadD25) -> DATA15_N
- J1 pad D28: unconnected-(J1-PadD28) -> DATA16_P
- J1 pad D29: unconnected-(J1-PadD29) -> DATA16_N
- J1 pad D32: unconnected-(J1-PadD32) -> DATA17_P
- J1 pad D33: unconnected-(J1-PadD33) -> DATA17_N
- J1 pad D36: unconnected-(J1-PadD36) -> DATA18_P
- J1 pad D37: unconnected-(J1-PadD37) -> DATA18_N
- J1 pad D4: unconnected-(J1-PadD4) -> DATA10_P
- J1 pad D40: unconnected-(J1-PadD40) -> LS1
- J1 pad D5: unconnected-(J1-PadD5) -> DATA10_N
- J1 pad D8: unconnected-(J1-PadD8) -> DATA11_P
- J1 pad D9: unconnected-(J1-PadD9) -> DATA11_N
- J1 pad G10: unconnected-(J1-PadG10) -> DATA21_P
- J1 pad G11: unconnected-(J1-PadG11) -> DATA21_N
- J1 pad G14: unconnected-(J1-PadG14) -> DATA22_P
- J1 pad G15: unconnected-(J1-PadG15) -> DATA22_N
- J1 pad G18: unconnected-(J1-PadG18) -> DATA23_P
- J1 pad G19: unconnected-(J1-PadG19) -> DATA23_N
- J1 pad G2: unconnected-(J1-PadG2) -> DATA19_P
- J1 pad G22: unconnected-(J1-PadG22) -> DATA24_P
- J1 pad G23: unconnected-(J1-PadG23) -> DATA24_N
- J1 pad G26: unconnected-(J1-PadG26) -> DATA25_P
- J1 pad G27: unconnected-(J1-PadG27) -> DATA25_N
- J1 pad G3: unconnected-(J1-PadG3) -> DATA19_N
- J1 pad G30: unconnected-(J1-PadG30) -> DATA26_P
- J1 pad G31: unconnected-(J1-PadG31) -> DATA26_N
- J1 pad G34: unconnected-(J1-PadG34) -> DATA27_P
- J1 pad G35: unconnected-(J1-PadG35) -> DATA27_N
- J1 pad G38: unconnected-(J1-PadG38) -> DATA28_P
- J1 pad G39: unconnected-(J1-PadG39) -> DATA28_N
- J1 pad G6: unconnected-(J1-PadG6) -> DATA20_P
- J1 pad G7: unconnected-(J1-PadG7) -> DATA20_N
- J1 pad H1: unconnected-(J1-PadH1) -> LS2
- J1 pad H12: unconnected-(J1-PadH12) -> DATA31_P
- J1 pad H13: unconnected-(J1-PadH13) -> DATA31_N
- J1 pad H16: unconnected-(J1-PadH16) -> CLK0_P
- J1 pad H17: unconnected-(J1-PadH17) -> CLK0_N
- J1 pad H20: unconnected-(J1-PadH20) -> GPIO0
- J1 pad H21: unconnected-(J1-PadH21) -> GPIO1
- J1 pad H24: unconnected-(J1-PadH24) -> GPIO2
- J1 pad H25: unconnected-(J1-PadH25) -> GPIO3
- J1 pad H28: unconnected-(J1-PadH28) -> GPIO4
- J1 pad H29: unconnected-(J1-PadH29) -> GPIO5
- J1 pad H32: unconnected-(J1-PadH32) -> GPIO6
- J1 pad H33: unconnected-(J1-PadH33) -> GPIO7
- J1 pad H36: unconnected-(J1-PadH36) -> LS5
- J1 pad H38: unconnected-(J1-PadH38) -> LS4
- J1 pad H4: unconnected-(J1-PadH4) -> DATA29_P
- J1 pad H40: unconnected-(J1-PadH40) -> LS3
- J1 pad H5: unconnected-(J1-PadH5) -> DATA29_N
- J1 pad H8: unconnected-(J1-PadH8) -> DATA30_P
- J1 pad H9: unconnected-(J1-PadH9) -> DATA30_N
- J2 pad A1: unconnected-(J2-PadA1) -> Net-(J2-GND-PadA1)
- J2 pad A12: unconnected-(J2-PadA12) -> Net-(J2-GND-PadA1)
- J2 pad A4: unconnected-(J2-PadA4) -> Net-(J2-VBUS-PadA4)
- J2 pad A9: unconnected-(J2-PadA9) -> Net-(J2-VBUS-PadA4)
- J2 pad B1: unconnected-(J2-PadB1) -> Net-(J2-GND-PadA1)
- J2 pad B12: unconnected-(J2-PadB12) -> Net-(J2-GND-PadA1)
- J2 pad B4: unconnected-(J2-PadB4) -> Net-(J2-VBUS-PadA4)
- J2 pad B9: unconnected-(J2-PadB9) -> Net-(J2-VBUS-PadA4)
Routing:
- net unconnected-(J1-PadE17): vias 0 -> 1
- net (no net): vias 1 -> 0

Commit message: New journal entry, progress on schematic and PCB
Parts:
- added J4: ASP-134486-01, ASP-134486-01:SAMTEC_ASP-134486-01, B.Cu at (107.7, 77.6)
- J1: value ASP-134488-01 -> 1040100018; footprint Connector_Samtec:Samtec_FMC_ASP-134486-01_10x40_P1.27mm_Vertical -> Connector_PinHeader_1.27mm:PinHeader_2x25_P1.27mm_Vertical_SMD
- R10, R13, R4, R7: footprint Package_DIP:DIP-8_W7.62mm -> Resistor_SMD:R_0402_1005Metric; moved to B.Cu
- moved J2 146.0 mm to (58.5, 113.2), turned to -90 degrees
- moved U8 129.9 mm to (62.0, 123.0)
- moved U7 124.2 mm to (62.0, 102.0)
- moved Y2 113.8 mm to (72.0, 103.0)
- moved R7 104.4 mm to (85.0, 150.0), turned to 180 degrees
- moved Y1 104.0 mm to (80.9, 129.5)
- moved R10 87.2 mm to (115.0, 150.0), turned to 180 degrees
- moved R13 77.2 mm to (105.0, 150.0), turned to 180 degrees
- moved R4 76.6 mm to (95.0, 150.0), turned to 180 degrees
- moved J1 39.0 mm to (141.4, 114.2)
- moved U6 29.5 mm to (71.2, 113.0)
- moved U4 17.0 mm to (112.0, 148.0)
- moved U5 13.1 mm to (102.0, 148.0)
- moved U2 10.2 mm to (92.0, 148.0)
- moved U1 8.95 mm to (104.5, 113.2)
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Connections:
- U1 pad A11: unconnected-(U1F-IO_L17P_T2_18-PadA11) -> LA30_N
- U1 pad A12: unconnected-(U1F-IO_L17N_T2_18-PadA12) -> LA30_P
- U1 pad A13: unconnected-(U1G-IO_L22N_T3_18-PadA13) -> LA31_P
- U1 pad A15: unconnected-(U1G-IO_L24N_T3_18-PadA15) -> LA29_P
- U1 pad A16: unconnected-(U1F-IO_L20P_T3_17-PadA16) -> LA25_N
- U1 pad A17: unconnected-(U1F-IO_L20N_T3_17-PadA17) -> LA25_P
- U1 pad A18: unconnected-(U1G-IO_L22N_T3_17-PadA18) -> LA22_P
- U1 pad A20: unconnected-(U1G-IO_L21P_T3_DQS_17-PadA20) -> LA15_N
- U1 pad A21: unconnected-(U1G-IO_L21N_T3_DQS_17-PadA21) -> LA15_P
- U1 pad A22: unconnected-(U1G-IO_L23N_T3_17-PadA22) -> LA16_N
- U1 pad A23: unconnected-(U1C-IO_L1N_T0_16-PadA23) -> LA11_N
- U1 pad A27: unconnected-(U1D-IO_L7N_T1_16-PadA27) -> LA07_N
- U1 pad A28: unconnected-(U1D-IO_L9N_T1_DQS_16-PadA28) -> LA08_N
- U1 pad A29: unconnected-(U1I-VCCO_16-PadA29) -> +2V5
- U1 pad A30: unconnected-(U1F-IO_L17N_T2_16-PadA30) -> LA03_N
- U1 pad B12: DATA13_N -> LA33_P
- U1 pad B13: unconnected-(U1G-IO_L22P_T3_18-PadB13) -> LA31_N
- U1 pad B14: unconnected-(U1G-IO_L24P_T3_18-PadB14) -> LA29_N
- U1 pad B15: unconnected-(U1G-IO_L23N_T3_18-PadB15) -> LA24_P
- U1 pad B17: unconnected-(U1F-IO_L17N_T2_17-PadB17) -> LA21_P
- U1 pad B18: unconnected-(U1G-IO_L22P_T3_17-PadB18) -> LA22_N
- U1 pad B19: unconnected-(U1G-IO_L24N_T3_17-PadB19) -> LA19_P
- U1 pad B20: unconnected-(U1F-IO_L19N_T3_VREF_17-PadB20) -> LA20_P
- U1 pad B22: unconnected-(U1G-IO_L23P_T3_17-PadB22) -> LA16_P
- U1 pad B23: unconnected-(U1C-IO_L1P_T0_16-PadB23) -> LA11_P
- U1 pad B24: unconnected-(U1D-IO_L8N_T1_16-PadB24) -> LA12_N
- U1 pad B26: unconnected-(U1I-VCCO_16-PadB26) -> +2V5
- U1 pad B27: unconnected-(U1D-IO_L7P_T1_16-PadB27) -> LA07_P
- U1 pad B28: unconnected-(U1D-IO_L9P_T1_DQS_16-PadB28) -> LA08_P
- U1 pad B29: unconnected-(U1E-IO_L15N_T2_DQS_16-PadB29) -> LA04_N
- U1 pad B30: unconnected-(U1F-IO_L17P_T2_16-PadB30) -> LA03_P
- U1 pad C11: DATA15_N -> LA32_P
- U1 pad C12: DATA13_P -> LA33_N
- U1 pad C14: unconnected-(U1G-IO_L21N_T3_DQS_18-PadC14) -> LA28_P
- U1 pad C15: unconnected-(U1G-IO_L23P_T3_18-PadC15) -> LA24_N
- U1 pad C16: DATA29_N -> unconnected-(U1E-IO_L15N_T2_DQS_17-PadC16)
- U1 pad C17: unconnected-(U1F-IO_L17P_T2_17-PadC17) -> LA21_N
- U1 pad C19: unconnected-(U1G-IO_L24P_T3_17-PadC19) -> LA19_N
- U1 pad C20: unconnected-(U1F-IO_L19P_T3_17-PadC20) -> LA20_N
- U1 pad C21: DATA22_N -> unconnected-(U1D-IO_L8N_T1_17-PadC21)
- U1 pad C22: DATA24_N -> unconnected-(U1D-IO_L10N_T1_17-PadC22)
- U1 pad C23: unconnected-(U1I-VCCO_16-PadC23) -> +2V5
- U1 pad C24: unconnected-(U1D-IO_L8P_T1_16-PadC24) -> LA12_P
- U1 pad C27: unconnected-(U1E-IO_L13N_T2_MRCC_16-PadC27) -> LA00_CC_N
- U1 pad C29: unconnected-(U1E-IO_L15P_T2_DQS_16-PadC29) -> LA04_P
- U1 pad C30: unconnected-(U1F-IO_L16N_T2_16-PadC30) -> LA02_P
- U1 pad D11: DATA15_P -> LA32_N
- U1 pad D12: DATA11_P -> unconnected-(U1E-IO_L13P_T2_MRCC_18-PadD12)
- U1 pad D13: DATA11_N -> unconnected-(U1E-IO_L13N_T2_MRCC_18-PadD13)
- U1 pad D14: unconnected-(U1G-IO_L21P_T3_DQS_18-PadD14) -> LA28_N
- U1 pad D16: DATA29_P -> unconnected-(U1E-IO_L15P_T2_DQS_17-PadD16)
- U1 pad D17: DATA27_P -> LA18_CC_P
- U1 pad D18: DATA27_N -> LA18_CC_N
- U1 pad D19: DATA28_N -> unconnected-(U1E-IO_L14N_T2_SRCC_17-PadD19)
- U1 pad D21: DATA22_P -> unconnected-(U1D-IO_L8P_T1_17-PadD21)
- U1 pad D22: DATA24_P -> unconnected-(U1D-IO_L10P_T1_17-PadD22)
- U1 pad D27: unconnected-(U1E-IO_L13P_T2_MRCC_16-PadD27) -> LA00_CC_P
- U1 pad D29: unconnected-(U1F-IO_L16P_T2_16-PadD29) -> LA02_N
- U1 pad D30: unconnected-(U1I-VCCO_16-PadD30) -> +2V5
- U1 pad E11: DATA14_N -> unconnected-(U1F-IO_L16N_T2_18-PadE11)
- U1 pad E13: DATA12_N -> unconnected-(U1E-IO_L14N_T2_SRCC_18-PadE13)
- U1 pad E19: DATA28_P -> unconnected-(U1E-IO_L14P_T2_SRCC_17-PadE19)
- U1 pad E20: DATA26_N -> unconnected-(U1E-IO_L12N_T1_MRCC_17-PadE20)
- U1 pad E21: DATA25_N -> unconnected-(U1E-IO_L11N_T1_SRCC_17-PadE21)
- U1 pad E27: unconnected-(U1J-VCCO_16-PadE27) -> +2V5
- U1 pad F11: DATA14_P -> unconnected-(U1F-IO_L16P_T2_18-PadF11)
- U1 pad F12: DATA12_P -> unconnected-(U1E-IO_L14P_T2_SRCC_18-PadF12)
- U1 pad F13: DATA10_N -> unconnected-(U1E-IO_L12N_T1_MRCC_18-PadF13)
- U1 pad F17: DATA31_N -> unconnected-(U1F-IO_L18N_T2_17-PadF17)
- U1 pad F18: DATA30_N -> unconnected-(U1F-IO_L16N_T2_17-PadF18)
- U1 pad F20: DATA26_P -> unconnected-(U1E-IO_L12P_T1_MRCC_17-PadF20)
- U1 pad F21: DATA9_N -> unconnected-(U1E-IO_L11P_T1_SRCC_17-PadF21)
- U1 pad F22: DATA23_N -> unconnected-(U1D-IO_L9N_T1_DQS_17-PadF22)
- U1 pad F24: unconnected-(U1J-VCCO_16-PadF24) -> +2V5
- U1 pad G13: DATA10_P -> unconnected-(U1E-IO_L12P_T1_MRCC_18-PadG13)
- U1 pad G14: DATA9_N -> unconnected-(U1E-IO_L11N_T1_SRCC_18-PadG14)
- U1 pad G15: DATA5_N -> unconnected-(U1D-IO_L7N_T1_18-PadG15)
- U1 pad G17: DATA31_P -> unconnected-(U1F-IO_L18P_T2_17-PadG17)
- U1 pad G18: DATA30_P -> unconnected-(U1F-IO_L16P_T2_17-PadG18)
- U1 pad G20: DATA17_N -> unconnected-(U1C-IO_L2N_T0_17-PadG20)
- U1 pad G22: DATA23_P -> unconnected-(U1D-IO_L9P_T1_DQS_17-PadG22)
- U1 pad H11: DATA8_P -> unconnected-(U1D-IO_L10P_T1_18-PadH11)
- U1 pad H12: DATA8_N -> unconnected-(U1D-IO_L10N_T1_18-PadH12)
- U1 pad H14: DATA9_P -> unconnected-(U1E-IO_L11P_T1_SRCC_18-PadH14)
- U1 pad H15: DATA5_P -> unconnected-(U1D-IO_L7P_T1_18-PadH15)
- U1 pad H16: DATA7_N -> unconnected-(U1D-IO_L9N_T1_DQS_18-PadH16)
- U1 pad H17: DATA18_N -> unconnected-(U1C-IO_L3N_T0_DQS_17-PadH17)
- U1 pad H19: DATA19_N -> unconnected-(U1C-IO_L4N_T0_17-PadH19)
- U1 pad H20: DATA17_P -> unconnected-(U1C-IO_L2P_T0_17-PadH20)
- U1 pad H21: DATA21_P -> unconnected-(U1D-IO_L7P_T1_17-PadH21)
- U1 pad H22: DATA21_N -> unconnected-(U1D-IO_L7N_T1_17-PadH22)
- U1 pad H28: unconnected-(U1J-VCCO_16-PadH28) -> +2V5
- U1 pad J11: DATA6_P -> unconnected-(U1D-IO_L8P_T1_18-PadJ11)
- U1 pad J12: DATA6_N -> unconnected-(U1D-IO_L8N_T1_18-PadJ12)
- U1 pad J13: DATA3_N -> unconnected-(U1C-IO_L4N_T0_18-PadJ13)
- U1 pad J14: DATA4_N -> unconnected-(U1C-IO_L5N_T0_18-PadJ14)
- U1 pad J16: DATA7_P -> unconnected-(U1D-IO_L9P_T1_DQS_18-PadJ16)
- U1 pad J17: DATA18_P -> unconnected-(U1C-IO_L3P_T0_DQS_17-PadJ17)
- U1 pad J18: DATA16_N -> unconnected-(U1C-IO_L1N_T0_17-PadJ18)
- U1 pad J19: DATA19_P -> unconnected-(U1C-IO_L4P_T0_17-PadJ19)
- U1 pad K13: DATA3_P -> unconnected-(U1C-IO_L4P_T0_18-PadK13)
- U1 pad K14: DATA4_P -> unconnected-(U1C-IO_L5P_T0_18-PadK14)
- U1 pad K15: DATA1_N -> unconnected-(U1C-IO_L2N_T0_18-PadK15)
- U1 pad K16: DATA0_N -> unconnected-(U1C-IO_L1N_T0_18-PadK16)
- U1 pad K18: DATA16_P -> unconnected-(U1C-IO_L1P_T0_17-PadK18)
- U1 pad L12: DATA2_P -> unconnected-(U1C-IO_L3P_T0_DQS_18-PadL12)
- U1 pad L13: DATA2_N -> unconnected-(U1C-IO_L3N_T0_DQS_18-PadL13)
- U1 pad L15: DATA1_P -> unconnected-(U1C-IO_L2P_T0_18-PadL15)
- U1 pad L16: DATA0_P -> unconnected-(U1C-IO_L1P_T0_18-PadL16)
- U1 pad L17: DATA20_P -> unconnected-(U1C-IO_L5P_T0_17-PadL17)
- U1 pad L18: DATA20_N -> unconnected-(U1C-IO_L5N_T0_17-PadL18)
Routing:
- net unconnected-(J1-PadE17): vias 1 -> 0
Other:
- board size 101.6 x 100.3 mm -> 100 x 100 mm

Commit message: New journal, moved BOMS into a new directory
Parts:
- U2, U3, U4, U5: value AS4C256M16D3 -> NT5CB64M16GP-FL
- moved U3 0.15 mm to (81.8, 148.0)
- renumbered J4 to J1, J1 to J2, J2 to J3, R13 to R12, R4 to R3, R7 to R6, R10 to R9, U6 to U7, U7 to U8, U8 to U9
Connections:
- net A0 renamed DDR_A0
- net A1 renamed DDR_A1
- net A10 renamed DDR_A10
- net A11 renamed DDR_A11
- net A12 renamed DDR_A12
- net A2 renamed DDR_A2
- net A3 renamed DDR_A3
- net A4 renamed DDR_A4
- net A5 renamed DDR_A5
- net A6 renamed DDR_A6
- net A7 renamed DDR_A7
- net A8 renamed DDR_A8
- net A9 renamed DDR_A9
- net BA0 renamed DDR_BA0
- net BA1 renamed DDR_BA1
- net BA2 renamed DDR_BA2
- net CAS renamed DDR_CAS
- net CAS_N renamed DDR_CAS_N
- net CKE renamed DDR_CKE
- net CK_N renamed DDR_CK_N
- net CK_P renamed DDR_CK_P
- net CLK0_M2C_N renamed FMC_CLK0_M2C_N
- net CLK0_M2C_P renamed FMC_CLK0_M2C_P
- net CLK1_M2C_N renamed FMC_CLK1_M2C_N
- net CLK1_M2C_P renamed FMC_CLK1_M2C_P
- net CLK_N renamed DDR_CLK_N
- net CLK_P renamed DDR_CLK_P
- net CS renamed DDR_CS
- net CS_N renamed DDR_CS_N
- net DATA00 renamed J2_DB2
- net DATA01 renamed J2_DB3
- net DATA02 renamed J2_DB4
- net DATA03 renamed J2_DB5
- net DATA04 renamed J2_DB6
- net DATA06 renamed J2_DB7
- net DATA07 renamed J2_DB8
- net DATA08 renamed J2_DB9
- net DATA09 renamed J2_DB10
- net DATA10 renamed J2_DB11
- net DATA11 renamed J2_DB12
- net DATA12 renamed J2_DB13
- net DATA14 renamed J2_DB14
- net DATA16 renamed J2_DB18
- net DATA17 renamed J2_DB19
- net DATA18 renamed J2_DB20
- net DATA19 renamed J2_DB21
- net DATA20 renamed J2_DB22
- net DATA22 renamed J2_DB23
- net DATA23 renamed J2_DB24
- net DATA24 renamed J2_DB25
- net DATA25 renamed J2_DB26
- net DATA26 renamed J2_DB27
- net DATA27 renamed J2_DB28
- net DATA28 renamed J2_DB29
- net DATA30 renamed J2_DB30
- net DM0 renamed DDR_DM0
- net DM1 renamed DDR_DM1
- net DM2 renamed DDR_DM2
- net DM3 renamed DDR_DM3
- net DM4 renamed DDR_DM4
- net DM5 renamed DDR_DM5
- net DM6 renamed DDR_DM6
- net DM7 renamed DDR_DM7
- net DP0_C2M_N renamed FMC_DP0_C2M_N
- net DP0_C2M_P renamed FMC_DP0_C2M_P
- net DP0_M2C_N renamed FMC_DP0_M2C_N
- net DP0_M2C_P renamed FMC_DP0_M2C_P
- net DQ00 renamed DDR_DQ00
- net DQ01 renamed DDR_DQ01
- net DQ02 renamed DDR_DQ02
- net DQ03 renamed DDR_DQ03
- net DQ04 renamed DDR_DQ04
- net DQ05 renamed DDR_DQ05
- net DQ06 renamed DDR_DQ06
- net DQ07 renamed DDR_DQ07
- net DQ08 renamed DDR_DQ08
- net DQ09 renamed DDR_DQ09
- net DQ10 renamed DDR_DQ10
- net DQ11 renamed DDR_DQ11
- net DQ12 renamed DDR_DQ12
- net DQ13 renamed DDR_DQ13
- net DQ14 renamed DDR_DQ14
- net DQ15 renamed DDR_DQ15
- net DQ16 renamed DDR_DQ16
- net DQ17 renamed DDR_DQ17
- net DQ18 renamed DDR_DQ18
- net DQ19 renamed DDR_DQ19
- net DQ20 renamed DDR_DQ20
- net DQ21 renamed DDR_DQ21
- net DQ22 renamed DDR_DQ22
- net DQ23 renamed DDR_DQ23
- net DQ24 renamed DDR_DQ24
- net DQ25 renamed DDR_DQ25
- net DQ26 renamed DDR_DQ26
- net DQ27 renamed DDR_DQ27
- net DQ28 renamed DDR_DQ28
- net DQ29 renamed DDR_DQ29
- net DQ30 renamed DDR_DQ30
- net DQ31 renamed DDR_DQ31
- net DQ32 renamed DDR_DQ32
- net DQ33 renamed DDR_DQ33
- net DQ34 renamed DDR_DQ34
- net DQ35 renamed DDR_DQ35
- net DQ36 renamed DDR_DQ36
- net DQ37 renamed DDR_DQ37
- net DQ38 renamed DDR_DQ38
- net DQ39 renamed DDR_DQ39
- net DQ40 renamed DDR_DQ40
- net DQ41 renamed DDR_DQ41
- net DQ42 renamed DDR_DQ42
- net DQ43 renamed DDR_DQ43
- net DQ44 renamed DDR_DQ44
- net DQ45 renamed DDR_DQ45
- net DQ46 renamed DDR_DQ46
- net DQ47 renamed DDR_DQ47
- net DQ48 renamed DDR_DQ48
- net DQ49 renamed DDR_DQ49
- net DQ50 renamed DDR_DQ50
- net DQ51 renamed DDR_DQ51
- net DQ52 renamed DDR_DQ52
- net DQ53 renamed DDR_DQ53
- net DQ54 renamed DDR_DQ54
- net DQ55 renamed DDR_DQ55
- net DQ56 renamed DDR_DQ56
- net DQ57 renamed DDR_DQ57
- net DQ58 renamed DDR_DQ58
- net DQ59 renamed DDR_DQ59
- net DQ60 renamed DDR_DQ60
- net DQ61 renamed DDR_DQ61
- net DQ62 renamed DDR_DQ62
- net DQ63 renamed DDR_DQ63
- net DQS_N0 renamed DDR_DQS_N0
- net DQS_N1 renamed DDR_DQS_N1
- net DQS_N2 renamed DDR_DQS_N2
- net DQS_N3 renamed DDR_DQS_N3
- net DQS_N4 renamed DDR_DQS_N4
- net DQS_N5 renamed DDR_DQS_N5
- net DQS_N6 renamed DDR_DQS_N6
- net DQS_N7 renamed DDR_DQS_N7
- net DQS_P0 renamed DDR_DQS_P0
- net DQS_P1 renamed DDR_DQS_P1
- net DQS_P2 renamed DDR_DQS_P2
- net DQS_P3 renamed DDR_DQS_P3
- net DQS_P4 renamed DDR_DQS_P4
- net DQS_P5 renamed DDR_DQS_P5
- net DQS_P6 renamed DDR_DQS_P6
- net DQS_P7 renamed DDR_DQS_P7
- net GA0 renamed FMC_GA0
- net GA1 renamed FMC_GA1
- net GBTCLK0_M2C_N renamed FMC_GBTCLK0_M2C_N
- net GPTCLK0_M2C_P renamed FMC_GPTCLK0_M2C_P
- net LA00_CC_N renamed FMC_LA00_CC_N
- net LA00_CC_P renamed FMC_LA00_CC_P
- net LA01_N renamed FMC_LA01_N
- net LA01_P renamed FMC_LA01_P
- net LA02_N renamed FMC_LA02_N
- net LA02_P renamed FMC_LA02_P
- net LA03_N renamed FMC_LA03_N
- net LA03_P renamed FMC_LA03_P
- net LA04_N renamed FMC_LA04_N
- net LA04_P renamed FMC_LA04_P
- net LA05_N renamed FMC_LA05_N
- net LA05_P renamed FMC_LA05_P
- net LA06_N renamed FMC_LA06_N
- net LA06_P renamed FMC_LA06_P
- net LA07_N renamed FMC_LA07_N
- net LA07_P renamed FMC_LA07_P
- net LA08_N renamed FMC_LA08_N
- net LA08_P renamed FMC_LA08_P
- net LA09_N renamed FMC_LA09_N
- net LA09_P renamed FMC_LA09_P
- net LA10_N renamed FMC_LA10_N
- net LA10_P renamed FMC_LA10_P
- net LA11_N renamed FMC_LA11_N
- net LA11_P renamed FMC_LA11_P
- net LA12_N renamed FMC_LA12_N
- net LA12_P renamed FMC_LA12_P
- net LA13_N renamed FMC_LA13_N
- net LA13_P renamed FMC_LA13_P
- net LA14_N renamed FMC_LA14_N
- net LA14_P renamed FMC_LA14_P
- net LA15_N renamed FMC_LA15_N
- net LA15_P renamed FMC_LA15_P
- net LA16_N renamed FMC_LA16_N
- net LA16_P renamed FMC_LA16_P
- net LA17_CC_N renamed FMC_LA17_CC_N
- net LA17_CC_P renamed FMC_LA17_CC_P
- net LA18_CC_N renamed FMC_LA18_CC_N
- net LA18_CC_P renamed FMC_LA18_CC_P
- net LA19_N renamed FMC_LA19_N
- net LA19_P renamed FMC_LA19_P
- net LA20_N renamed FMC_LA20_N
- net LA20_P renamed FMC_LA20_P
- net LA21_N renamed FMC_LA21_N
- net LA21_P renamed FMC_LA21_P
- net LA22_N renamed FMC_LA22_N
- net LA22_P renamed FMC_LA22_P
- net LA23_N renamed FMC_LA23_N
- net LA23_P renamed FMC_LA23_P
- net LA24_N renamed FMC_LA24_N
- net LA24_P renamed FMC_LA24_P
- net LA25_N renamed FMC_LA25_N
- net LA25_P renamed FMC_LA25_P
- net LA26_N renamed FMC_LA26_N
- net LA26_P renamed FMC_LA26_P
- net LA27_N renamed FMC_LA27_N
- net LA27_P renamed FMC_LA27_P
- net LA28_N renamed FMC_LA28_N
- net LA28_P renamed FMC_LA28_P
- net LA29_N renamed FMC_LA29_N
- net LA29_P renamed FMC_LA29_P
- net LA30_N renamed FMC_LA30_N
- net LA30_P renamed FMC_LA30_P
- net LA31_N renamed FMC_LA31_N
- net LA31_P renamed FMC_LA31_P
- net LA32_N renamed FMC_LA32_N
- net LA32_P renamed FMC_LA32_P
- net LA33_N renamed FMC_LA33_N
- net LA33_P renamed FMC_LA33_P
- net ODT renamed DDR_ODT
- net PG_C2M renamed FMC_PG_C2M
- net PRSNT_M2C_L renamed FMC_PRSNT_M2C_L
- net RAS renamed DDR_RAS
- net RAS_N renamed DDR_RAS_N
- net REF_N renamed DDR_REF_N
- net REF_P renamed DDR_REF_P
- net RESET renamed DDR_RESET
- net SCL renamed FMC_SCL
- net SDA renamed FMC_SDA
- net TCK renamed FMC_TCK
- net TDI renamed FMC_TDI
- net TDO renamed FMC_TDO
- net TMS renamed FMC_TMS
- net TRST_L renamed FMC_TRST_L
- net VREF_1 renamed U3_VREF
- net VREF_2 renamed U4_VREF
- net VREF_A_M2C renamed FMC_VREF_A_M2C
- net WE renamed DDR_WE
- net WE_N renamed DDR_WE_N
- J2 pad 17: DATA05 -> GND
- J2 pad 18: DATA21 -> GND
- J2 pad 3: GND -> J2_DB0
- J2 pad 33: DATA13 -> GND
- J2 pad 34: DATA29 -> GND
- J2 pad 37: DATA15 -> GND
- J2 pad 38: DATA31 -> GND
- J2 pad 39: GND -> J2_DB15
- J2 pad 4: GND -> J2_DB16
- J2 pad 40: GND -> J2_DB31
- J2 pad 41: CLK0 -> GND
- J2 pad 42: CLK1 -> GND
- J2 pad 43: GND -> J2_CLK0
- J2 pad 44: GND -> J2_CLK1
- J2 pad 45: WRT0 -> GND
- J2 pad 46: WRT1 -> GND
- J2 pad 47: GND -> J2_WRT0
- J2 pad 48: GND -> J2_WRT1
- J2 pad 5: GND -> J2_DB1
- J2 pad 6: GND -> J2_DB17
- U2 pad H1: VREF_0 -> U2_VREF
- U2 pad M8: VREF_0 -> U2_VREF
- U5 pad H1: VREF_0 -> U5_VREF
- U5 pad M8: VREF_0 -> U5_VREF
