File: KiCad/uranus-fpga-board/uranus-fpga-board.kicad_pcb (KiCad board)
At the start: 8 copper layers, 100 x 100 mm, 17 parts, among them J1 ASP-134486-01, J2 1040100018, J3 TYPE-C-31-M-12, U1 XC7K325T-3FFG900E, U2 NT5CB64M16GP-FL, U3 NT5CB64M16GP-FL, U4 NT5CB64M16GP-FL, U5 NT5CB64M16GP-FL, U7 FT232HL-REEL, U8 93LC56BT, U9 USBLC6-2SC6, Y1 SX7DF200.000B20F30DNN, Y2 3225-12-20-10-10/4B

Commit message: Oct 18 journal
Parts:
- added Q1: 2N7002, Package_TO_SOT_SMD:SOT-23, F.Cu at (175.7, 114.3)
- added R16: 200 kΩ, Resistor_SMD:R_0402_1005Metric, F.Cu at (166.2, 92.4)
- added R19: 57.6 kΩ, Resistor_SMD:R_0402_1005Metric, F.Cu at (201.5, 114.9)
- added R20: 499 Ω, Resistor_SMD:R_0201_0603Metric, F.Cu at (201.5, 117.4)
- added R21: 7.68 kΩ, Resistor_SMD:R_0402_1005Metric, F.Cu at (201.5, 119.9)
- added R22: 232 kΩ, Resistor_SMD:R_0402_1005Metric, F.Cu at (195.6, 109.2)
- added R23: 499 Ω, Resistor_SMD:R_0201_0603Metric, F.Cu at (195.6, 110.3)
- added R24: 7.68 kΩ, Resistor_SMD:R_0402_1005Metric, F.Cu at (195.6, 111.5)
- added R25: 57.6 kΩ, Resistor_SMD:R_0402_1005Metric, F.Cu at (192.8, 95.9)
- added R26: 499 Ω, Resistor_SMD:R_0201_0603Metric, F.Cu at (192.8, 97.0)
- added R27: 7.68 kΩ, Resistor_SMD:R_0402_1005Metric, F.Cu at (192.8, 98.1)
- added R29: 499 Ω, Resistor_SMD:R_0201_0603Metric, F.Cu at (170.2, 106.1)
- added R30: 7.68 kΩ, Resistor_SMD:R_0402_1005Metric, F.Cu at (174.2, 96.1)
- added R31: 15.8 kΩ, Resistor_SMD:R_0402_1005Metric, F.Cu at (169.7, 115.0)
- added R32: 21 kΩ, Resistor_SMD:R_0402_1005Metric, F.Cu at (179.5, 96.0)
- added R33: 27.4 kΩ, Resistor_SMD:R_0402_1005Metric, F.Cu at (174.2, 98.6)
- added R34: 41.2 kΩ, Resistor_SMD:R_0402_1005Metric, F.Cu at (174.2, 101.1)
- added R35: 57.6 kΩ, Resistor_SMD:R_0402_1005Metric, F.Cu at (174.2, 103.6)
- added R36: 200 kΩ, Resistor_SMD:R_0402_1005Metric, F.Cu at (170.2, 92.4)
- added R37: 200 kΩ, Resistor_SMD:R_0402_1005Metric, F.Cu at (174.3, 89.5)
- added R38: 499 Ω, Resistor_SMD:R_0201_0603Metric, F.Cu at (174.2, 106.2)
- added R39: 200 kΩ, Resistor_SMD:R_0402_1005Metric, F.Cu at (178.3, 92.4)
- added U10: TLV6700DDCR, Package_TO_SOT_SMD:SOT-23-6, F.Cu at (196.9, 120.4)
- added U11: TLV6700DDCR, Package_TO_SOT_SMD:SOT-23-6, F.Cu at (198.3, 109.7)
- added U12: TLV6700DDCR, Package_TO_SOT_SMD:SOT-23-6, F.Cu at (195.8, 96.6)
- added U13: TMUX1108PW, Package_SO:TSSOP-16_4.4x5mm_P0.65mm, F.Cu at (168.9, 110.7)
- added U14: TLV6700DDCR, Package_TO_SOT_SMD:SOT-23-6, F.Cu at (161.6, 115.5)
- added U6: TPS2553DBVR, Package_TO_SOT_SMD:SOT-23-6, F.Cu at (161.6, 92.4)
- added U7: SY6288F1ABC, Package_TO_SOT_SMD:SOT-23-6, F.Cu at (161.6, 97.0)
- added U8: SY6874DBC, Package_DFN_QFN:DFN-10-1EP_3x3mm_P0.5mm_EP1.75x2.7mm, F.Cu at (176.4, 109.8)
- added U9: TI TPS22975DSGR, Package_SON:Texas_DSG0008A_WSON-8-1EP_2x2mm_P0.5mm_EP0.9x1.6mm, F.Cu at (166.2, 115.9)
- R12, R3, R6, R9: value 240Ω -> 240 Ω
- moved R3 0.11 mm to (94.9, 150.0)
- renumbered U7 to U16, U8 to U17, U9 to U18
Connections:
- net +12V0 renamed +12V0_P
- J1 pad C34: FMC_GA0 -> GND
- J1 pad C39: +3V3 -> +3V3_P
- J1 pad D35: FMC_GA1 -> GND
- J1 pad D36: +3V3 -> +3V3_P
- J1 pad D38: +3V3 -> +3V3_P
- J1 pad D40: +3V3 -> +3V3_P
- J1 pad G39: VADJ -> VADJ_P
- J1 pad H01: FMC_VREF_A_M2C -> unconnected-(J1-PadH01)
- J1 pad H40: VADJ -> VADJ_P
- U1 pad A19: +2V5 -> VADJ_P
- U1 pad A29: +2V5 -> VADJ_P
- U1 pad AD9: DDR_RAS_N -> ~{DDR_RAS}
- U1 pad AE11: DDR_WE_N -> ~{DDR_WE}
- U1 pad AE9: DDR_CAS_N -> ~{DDR_CAS}
- U1 pad AF11: DDR_CS_N -> ~{DDR_CS}
- U1 pad B1: unconnected-(U1A-MGTXTXN2_118-PadB1) -> FMC_DP0_C2M_N
- U1 pad B16: +2V5 -> VADJ_P
- U1 pad B2: unconnected-(U1A-MGTXTXP2_118-PadB2) -> FMC_DP0_C2M_P
- U1 pad B26: +2V5 -> VADJ_P
- U1 pad B5: unconnected-(U1B-MGTXRXN2_118-PadB5) -> FMC_DP0_M2C_N
- U1 pad B6: unconnected-(U1B-MGTXRXP2_118-PadB6) -> FMC_DP0_M2C_P
- U1 pad C13: +2V5 -> VADJ_P
- U1 pad C16: unconnected-(U1E-IO_L15N_T2_DQS_17-PadC16) -> FMC_LA14_N
- U1 pad C21: unconnected-(U1D-IO_L8N_T1_17-PadC21) -> FMC_LA10_N
- U1 pad C22: unconnected-(U1D-IO_L10N_T1_17-PadC22) -> FMC_LA09_N
- U1 pad C23: +2V5 -> VADJ_P
- U1 pad C7: unconnected-(U1A-MGTREFCLK0N_118-PadC7) -> FMC_MGTREFCLK0_N
- U1 pad C8: unconnected-(U1A-MGTREFCLK0P_118-PadC8) -> FMC_MGTREFCLK0_P
- U1 pad D10: +2V5 -> VADJ_P
- U1 pad D12: unconnected-(U1E-IO_L13P_T2_MRCC_18-PadD12) -> FMC_LA17_CC_P
- U1 pad D13: unconnected-(U1E-IO_L13N_T2_MRCC_18-PadD13) -> FMC_LA17_CC_N
- U1 pad D16: unconnected-(U1E-IO_L15P_T2_DQS_17-PadD16) -> FMC_LA14_P
- U1 pad D19: unconnected-(U1E-IO_L14N_T2_SRCC_17-PadD19) -> FMC_LA13_N
- U1 pad D20: +2V5 -> VADJ_P
- U1 pad D21: unconnected-(U1D-IO_L8P_T1_17-PadD21) -> FMC_LA10_P
- U1 pad D22: unconnected-(U1D-IO_L10P_T1_17-PadD22) -> FMC_LA09_P
- U1 pad D23: unconnected-(U1C-IO_L2N_T0_16-PadD23) -> FMC_LA05_N
- U1 pad D24: unconnected-(U1C-IO_L4N_T0_16-PadD24) -> FMC_LA06_N
- U1 pad D30: +2V5 -> VADJ_P
- U1 pad E11: unconnected-(U1F-IO_L16N_T2_18-PadE11) -> FMC_LA26_N
- U1 pad E14: unconnected-(U1F-IO_L20P_T3_18-PadE14) -> FMC_LA27_N
- U1 pad E15: unconnected-(U1F-IO_L20N_T3_18-PadE15) -> FMC_LA27_P
- U1 pad E16: unconnected-(U1F-IO_L19N_T3_VREF_18-PadE16) -> FMC_LA23_P
- U1 pad E17: +2V5 -> VADJ_P
- U1 pad E19: unconnected-(U1E-IO_L14P_T2_SRCC_17-PadE19) -> FMC_LA13_P
- U1 pad E23: unconnected-(U1C-IO_L2P_T0_16-PadE23) -> FMC_LA05_P
- U1 pad E24: unconnected-(U1C-IO_L4P_T0_16-PadE24) -> FMC_LA06_P
- U1 pad E27: +2V5 -> VADJ_P
- U1 pad E29: unconnected-(U1F-IO_L18P_T2_16-PadE29) -> FMC_LA01_N
- U1 pad E30: unconnected-(U1F-IO_L18N_T2_16-PadE30) -> FMC_LA01_P
- U1 pad F11: unconnected-(U1F-IO_L16P_T2_18-PadF11) -> FMC_LA26_P
- U1 pad F14: +2V5 -> VADJ_P
- U1 pad F15: unconnected-(U1F-IO_L19P_T3_18-PadF15) -> FMC_LA23_N
- U1 pad F24: +2V5 -> VADJ_P
- U1 pad G11: +2V5 -> VADJ_P
- U1 pad G21: +2V5 -> VADJ_P
- U1 pad H18: +2V5 -> VADJ_P
- U1 pad H28: +2V5 -> VADJ_P
- U1 pad J15: +2V5 -> VADJ_P
- U1 pad K12: +2V5 -> VADJ_P
- U1 pad L19: +2V5 -> VADJ_P
- U2 pad J3: DDR_RAS -> ~{DDR_RAS}
- U2 pad K3: DDR_CAS -> ~{DDR_CAS}
- U2 pad L2: DDR_CS -> ~{DDR_CS}
- U2 pad L3: DDR_WE -> ~{DDR_WE}
- U3 pad J3: DDR_RAS -> ~{DDR_RAS}
- U3 pad K3: DDR_CAS -> ~{DDR_CAS}
- U3 pad L2: DDR_CS -> ~{DDR_CS}
- U3 pad L3: DDR_WE -> ~{DDR_WE}
- U4 pad J3: DDR_RAS -> ~{DDR_RAS}
- U4 pad K3: DDR_CAS -> ~{DDR_CAS}
- U4 pad L2: DDR_CS -> ~{DDR_CS}
- U4 pad L3: DDR_WE -> ~{DDR_WE}
- U5 pad J3: DDR_RAS -> ~{DDR_RAS}
- U5 pad K3: DDR_CAS -> ~{DDR_CAS}
- U5 pad L2: DDR_CS -> ~{DDR_CS}
- U5 pad L3: DDR_WE -> ~{DDR_WE}
Routing:
- net FMC_LA24_N: track 0.00 -> 22.9 mm, vias 0 -> 2
- net FMC_LA24_P: track 0.00 -> 21.9 mm, vias 0 -> 2
- net Net-(U12-INB-): track 0.00 -> 3.37 mm
- net Net-(U12-INA+): track 0.00 -> 3.09 mm
- net Net-(U11-INB-): track 0.00 -> 2.96 mm
- net Net-(U11-INA+): track 0.00 -> 2.90 mm
- net Net-(U2-ZQ): vias 0 -> 1

Commit message: big things happening in JOURNAL
Parts:
- removed the U9 at (166.2, 115.9)
- added L1: 2.2 μH, Inductor_SMD:L_Chilisin_BMRA00040415, F.Cu at (64.0, 121.2)
- added R1: 1 kΩ, Resistor_SMD:R_0402_1005Metric, F.Cu at (75.5, 112.8)
- added R10: 1 kΩ, Resistor_SMD:R_0402_1005Metric, F.Cu at (81.3, 114.7)
- added R11: 1 kΩ, Resistor_SMD:R_0402_1005Metric, F.Cu at (81.3, 116.7)
- added R13: 1.8 kΩ, Resistor_SMD:R_0402_1005Metric, F.Cu at (80.6, 92.2)
- added R14: 10 kΩ, Resistor_SMD:R_0201_0603Metric, F.Cu at (77.9, 88.5)
- added R16: 7.5 kΩ, Resistor_SMD:R_0201_0603Metric, F.Cu at (77.9, 90.2)
- added R17: 10 kΩ, Resistor_SMD:R_0201_0603Metric, F.Cu at (77.9, 92.0)
- added R2: 1 kΩ, Resistor_SMD:R_0402_1005Metric, F.Cu at (75.5, 114.7)
- added R27: 10 kΩ, Resistor_SMD:R_0201_0603Metric, F.Cu at (77.9, 93.7)
- added R39: 4.7 kΩ, Resistor_SMD:R_0402_1005Metric, F.Cu at (59.2, 119.3)
- added R4: 1 kΩ, Resistor_SMD:R_0402_1005Metric, F.Cu at (75.5, 118.7)
- added R40: 30 kΩ, Resistor_SMD:R_0201_0603Metric, F.Cu at (68.6, 121.0)
- added R41: 52.3 kΩ, Resistor_SMD:R_0402_1005Metric, F.Cu at (59.2, 121.3)
- added R42: 30.9 kΩ, Resistor_SMD:R_0402_1005Metric, F.Cu at (59.2, 123.3)
- added R43: 22.1 kΩ, Resistor_SMD:R_0402_1005Metric, F.Cu at (59.2, 125.3)
- added R44: 13 kΩ, Resistor_SMD:R_0402_1005Metric, F.Cu at (59.2, 127.3)
- added R45: 8.98 kΩ, Resistor_SMD:R_0603_1608Metric, F.Cu at (62.6, 125.3)
- added R46: 200 kΩ, Resistor_SMD:R_0201_0603Metric, F.Cu at (68.6, 122.7)
- added R47: 200 kΩ, Resistor_SMD:R_0201_0603Metric, F.Cu at (68.6, 124.5)
- added R48: 200 kΩ, Resistor_SMD:R_0201_0603Metric, F.Cu at (68.6, 126.2)
- added R5: 1 kΩ, Resistor_SMD:R_0402_1005Metric, F.Cu at (78.4, 112.8)
- added R7: 1 kΩ, Resistor_SMD:R_0402_1005Metric, F.Cu at (78.4, 116.7)
- added R8: 1 kΩ, Resistor_SMD:R_0402_1005Metric, F.Cu at (78.4, 118.7)
- added U15: FT232HL-REEL, FT232HL:LQFP48_FT232HL_FTD, F.Cu at (63.6, 93.4)
- added U19: TMUX1108PWR, Package_SO:TSSOP-16_4.4x5mm_P0.65mm, F.Cu at (62.5, 115.1)
- R12, R3, R6, R9: moved to F.Cu
- R31: renamed from R32; value 21 kΩ -> 21.5 kΩ
- R35: renamed from R36; footprint Resistor_SMD:R_0402_1005Metric -> Resistor_SMD:R_0201_0603Metric
- R36: renamed from R37; footprint Resistor_SMD:R_0402_1005Metric -> Resistor_SMD:R_0201_0603Metric
- R37: renamed from R39; footprint Resistor_SMD:R_0402_1005Metric -> Resistor_SMD:R_0201_0603Metric
- R38: value 499 Ω -> 10 kΩ
- U1: value XC7K325T-3FFG900E -> XC7K325T
- U16: value FT232HL-REEL -> 93LC56BT; footprint FT232HL:LQFP48_FT232HL_FTD -> Package_TO_SOT_SMD:SOT-23-6
- U17: value 93LC56BT -> USBLC6-2SC6
- U18: value USBLC6-2SC6 -> TPS564201DDCR
- moved R38 106.4 mm to (68.6, 119.2)
- moved R21 58.9 mm to (144.8, 79.4)
- moved R22 58.9 mm to (144.8, 80.5)
- moved R23 58.9 mm to (144.8, 81.7)
- moved U10 58.9 mm to (147.5, 79.9)
- moved R18 58.9 mm to (150.7, 85.1)
- moved R19 58.9 mm to (150.7, 87.6)
- moved R20 58.9 mm to (150.7, 90.1)
- moved R24 58.9 mm to (142.0, 66.1)
- moved R25 58.9 mm to (142.0, 67.2)
- moved R26 58.9 mm to (142.0, 68.3)
- moved U11 58.9 mm to (145.0, 66.8)
- moved U9 58.9 mm to (146.1, 90.7)
- moved R15 53.4 mm to (132.9, 134.2)
- moved R32 53.4 mm to (140.9, 140.4)
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- renumbered R16 to R15, R19 to R18, R20 to R19, R21 to R20, R22 to R21, R23 to R22, R24 to R23, R25 to R24, R26 to R25, R27 to R26, R29 to R28, R30 to R29, R31 to R30, R33 to R32, R34 to R33, R35 to R34, U11 to U10, U12 to U11, U13 to U12, U14 to U13, U10 to U9
Connections:
- net FMC_PRSNT_M2C_L renamed ~{FMC_PRSNT_M2C}
- net VADJ_VSW_A0 renamed VADJ_SEL_A0
- net VADJ_VSW_A1 renamed VADJ_SEL_A1
- net VADJ_VSW_A2 renamed VADJ_SEL_A2
- net ~{FMC_PRSNT} renamed FMC_PRSNT
- J1 pad G39: VADJ_P -> VADJ
- J1 pad H40: VADJ_P -> VADJ
- R30 pad 1: VADJ_P -> VADJ
- R31 pad 1: Net-(R32-Pad1) -> VADJ
- R32 pad 1: VADJ_P -> VADJ
- R33 pad 1: VADJ_P -> VADJ
- R34 pad 1: VADJ_P -> VADJ
- R38 pad 1: VADJ_P -> VADJ_REG_EN
- R38 pad 2: Net-(R32-Pad1) -> GND
- U1 pad A19: VADJ_P -> VADJ
- U1 pad A29: VADJ_P -> VADJ
- U1 pad B16: VADJ_P -> VADJ
- U1 pad B26: VADJ_P -> VADJ
- U1 pad C13: VADJ_P -> VADJ
- U1 pad C23: VADJ_P -> VADJ
- U1 pad D10: VADJ_P -> VADJ
- U1 pad D20: VADJ_P -> VADJ
- U1 pad D30: VADJ_P -> VADJ
- U1 pad E17: VADJ_P -> VADJ
- U1 pad E27: VADJ_P -> VADJ
- U1 pad F14: VADJ_P -> VADJ
- U1 pad F24: VADJ_P -> VADJ
- U1 pad G11: VADJ_P -> VADJ
- U1 pad G21: VADJ_P -> VADJ
- U1 pad H18: VADJ_P -> VADJ
- U1 pad H28: VADJ_P -> VADJ
- U1 pad J15: VADJ_P -> VADJ
- U1 pad K12: VADJ_P -> VADJ
- U1 pad L19: VADJ_P -> VADJ
- U18 pad 1: unconnected-(U18-USB_IO1-Pad1) -> GND
- U18 pad 2: unconnected-(U18-GND-Pad2) -> Net-(U18-SW)
- U18 pad 3: unconnected-(U18-USB_IO2-Pad3) -> +12V0
- U18 pad 4: unconnected-(U18-MCU_IO2-Pad4) -> Net-(U18-VFB)
- U18 pad 5: unconnected-(U18-VBUS-Pad5) -> VADJ_REG_EN
- U18 pad 6: unconnected-(U18-MCU_IO1-Pad6) -> Net-(U18-VBST)
- U6 pad 1: unconnected-(U6-~{FAULT}-Pad1) -> +3V3
- U6 pad 2: +3V3AUX -> GND
- U6 pad 3: Net-(U6-ILIM) -> +3V3
- U6 pad 4: +3V3 -> unconnected-(U6-~{FAULT}-Pad4)
- U6 pad 5: GND -> Net-(U6-ILIM)
- U6 pad 6: +3V3 -> +3V3AUX

Commit message: Big things have mostly happened in schematic quality
Routing:
- net FMC_LA24_N: track 22.9 -> 21.5 mm
Changed lines of the file:
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@@
 	)
 	(gr_line
-		(start 99.949999 98.849999)
-		(end 100.949999 98.849999)
+		(start 99.949999 99.357999)
+		(end 100.949999 99.357999)
 		(stroke
 			(width 0.1)
@@
 	)
 	(gr_line
-		(start 100.949999 99.599999)
-		(end 100.949999 100.849999)
+		(start 100.949999 100.107999)
+		(end 100.949999 101.357999)
 		(stroke
 			(width 0.1)
@@
 	)
 	(gr_line
-		(start 101.949999 99.849999)
-		(end 101.949999 98.849999)
+		(start 101.949999 100.357999)
+		(end 101.949999 99.357999)
 		(stroke
 			(width 0.1)
@@
 	)
 	(gr_line
-		(start 102.949999 99.849999)
-		(end 103.949999 98.849999)
+		(start 102.949999 100.357999)
+		(end 103.949999 99.357999)
 		(stroke
 			(width 0.1)
@@
 	)
 	(gr_line
-		(start 103.949999 99.849999)
-		(end 103.949999 100.849999)
+		(start 103.949999 100.357999)
+		(end 103.949999 101.357999)
 		(stroke
 			(width 0.1)
@@
 	)
 	(segment
-		(start 145.099033 80.549066)
-		(end 145.430933 80.549066)
+		(start 144.847794 79.870705)
+		(end 144.663811 80.054688)
+		(width 0.3048)
+		(layer "F.Cu")
+		(net "Net-(U10-INA+)")
+	)
+	(segment
+		(start 145.285619 79.43288)
+		(end 144.847794 79.870705)
+		(width 0.3048)
+		(layer "F.Cu")
+		(net "Net-(U10-INA+)")
+	)
+	(segment
+		(start 146.188167 79.059033)
+		(end 146.521433 78.725766)
 		(width 0.4064)
 		(layer "F.Cu")
-		(net "Net-(U10-INB-)")
-	)
-	(segment
-		(start 144.895669 81.04003)
-		(end 144.269033 81.666666)
+		(net "Net-(U10-INA+)")
+	)
+	(segment
+		(start 145.289033 79.431466)
+		(end 145.285619 79.43288)
+		(width 0.2)
+		(layer "F.Cu")
+		(net "Net-(U10-INA+)")
+	)
+	(arc
+		(start 144.663811 80.054688)
+		(mid 144.512253 80.28151)
+		(end 144.459033 80.549066)
 		(width 0.3048)
 		(layer "F.Cu")
-		(net "Net-(U10-INB-)")
+		(net "Net-(U10-INA+)")
 	)
 	(arc
-		(start 145.430933 80.549066)
-		(mid 146.021107 80.666459)
-		(end 146.521433 81.000766)
+		(start 145.285619 79.43288)
+		(mid 145.774074 79.33572)
+		(end 146.188167 79.059033)
 		(width 0.4064)
 		(layer "F.Cu")
-		(net "Net-(U10-INB-)")
-	)
-	(arc
-		(start 145.099033 80.549066)
-		(mid 145.04618 80.814774)
-		(end 144.895669 81.04003)
-		(width 0.3048)
-		(layer "F.Cu")
-		(net "Net-(U10-INB-)")
-	)
-	(segment
-		(start 142.520433 66.096466)
-		(end 142.981233 66.096466)
-		(width 0.4064)
-		(layer "F.Cu")
-		(net "Net-(U11-INA+)")
-	)
-	(segment
-		(start 142.520433 66.096466)
-		(end 141.893797 66.723102)
-		(width 0.3048)
-		(layer "F.Cu")
-		(net "Net-(U11-INA+)")
-	)
-	(arc
-		(start 141.893797 66.723102)
-		(mid 141.743286 66.948358)
-		(end 141.690433 67.214066)
-		(width 0.3048)
-		(layer "F.Cu")
-		(net "Net-(U11-INA+)")
-	)
-	(arc
-		(start 142.981233 66.096466)
-		(mid 143.571407 65.979073)
-		(end 144.071733 65.644766)
-		(width 0.4064)
-		(layer "F.Cu")
-		(net "Net-(U11-INA+)")
+		(net "Net-(U10-INA+)")
+	)
+	(via
+		(at 98.176 80.741)
+		(size 0.6)
+		(drill 0.3)
+		(layers "F.Cu" "B.Cu")
+		(net "FMC_LA24_P")
 	)
 	(via
@@
 		(net "FMC_LA24_P")
 	)
-	(via
-		(at 98.176 80.741)
-		(size 0.6)
-		(drill 0.3)
-		(layers "F.Cu" "B.Cu")
+	(segment
+		(start 97.989186 94.227211)
+		(end 97.995564 94.233589)
+		(width 0.2)
+		(layer "In5.Cu")
 		(net "FMC_LA24_P")
 	)
 	(segment
-		(start 98.058894 94.172497)
-		(end 103.636396 99.749999)
+		(start 97.766001 81.150999)
+		(end 98.176 80.741)
 		(width 0.2)
 		(layer "In5.Cu")
@@
 	)
 	(segment
-		(start 97.766001 81.150999)
-		(end 97.766001 93.46539)
+		(start 98.430344 94.233589)
+		(end 98.637217 94.440462)
 		(width 0.2)
 		(layer "In5.Cu")
@@
 	)
 	(segment
-		(start 103.636396 99.749999)
-		(end 103.999999 99.749999)
+		(start 97.766001 93.688395)
+		(end 97.766001 81.150999)
 		(width 0.2)
 		(layer "In5.Cu")
@@
 	)
 	(segment
-		(start 98.176 80.741)
-		(end 97.766001 81.150999)
+		(start 98.844092 95.082117)
+		(end 98.863499 95.101524)
 		(width 0.2)
 		(layer "In5.Cu")
 		(net "FMC_LA24_P")
 	)
+	(segment
+		(start 98.863499 95.101524)
+		(end 103.226988 99.465013)
+		(width 0.2)
+		(layer "In5.Cu")
+		(net "FMC_LA24_P")
+	)
+	(segment
+		(start 98.637218 94.875244)
+		(end 98.844092 95.082117)
+		(width 0.2)
+		(layer "In5.Cu")
+		(net "FMC_LA24_P")
+	)
 	(arc
-		(start 98.058894 94.172497)
-		(mid 97.842121 93.848074)
-		(end 97.766001 93.46539)
+		(start 98.637218 94.657854)
+		(mid 98.592195 94.766549)
+		(end 98.637218 94.875244)
+		(width 0.2)
+		(layer "In5.Cu")
+		(net "FMC_LA24_P")
+	)
+	(arc
+		(start 98.212954 94.233589)
+		(mid 98.321649 94.188566)
+		(end 98.430344 94.233589)
+		(width 0.2)
+		(layer "In5.Cu")
+		(net "FMC_LA24_P")
+	)
+	(arc
+		(start 98.637217 94.440462)
+		(mid 98.682241 94.549159)
+		(end 98.637218 94.657854)
+		(width 0.2)
+		(layer "In5.Cu")
+		(net "FMC_LA24_P")
+	)
+	(arc
+		(start 97.989186 94.227211)
+		(mid 97.824005 93.98)
+		(end 97.766001 93.688395)
+		(width 0.2)
+		(layer "In5.Cu")
+		(net "FMC_LA24_P")
+	)
+	(arc
+		(start 97.995564 94.233589)
+		(mid 98.104259 94.278612)
+		(end 98.212954 94.233589)
 		(width 0.2)
 		(layer "In5.Cu")
@@
 	)
 	(segment
-		(start 97.315999 81.150999)
-		(end 97.315999 93.651785)
-		(width 0.2)
-		(layer "In5.Cu")
-		(net "FMC_LA24_N")
-	)
-	(segment
 		(start 96.906 80.741)
 		(end 97.315999 81.150999)
@@
 	)
 	(segment
-		(start 97.608892 94.358892)
-		(end 103.999999 100.749999)
+		(start 97.687974 94.562395)
+		(end 102.90879 99.783211)
 		(width 0.2)
 		(layer "In5.Cu")
 		(net "FMC_LA24_N")
 	)
+	(segment
+		(start 97.315999 81.150999)
+		(end 97.315999 93.664369)
+		(width 0.2)
+		(layer "In5.Cu")
+		(net "FMC_LA24_N")
+	)
 	(arc
-		(start 97.608892 94.358892)
-		(mid 97.392119 94.034469)
-		(end 97.315999 93.651785)
+		(start 97.315999 93.664369)
+		(mid 97.412672 94.150377)
+		(end 97.687974 94.562395)
 		(width 0.2)
 		(layer "In5.Cu")
@@
 	)
 	(segment
-		(start 144.847794 79.870705)
-		(end 144.663811 80.054688)
+		(start 142.520433 66.096466)
+		(end 142.981233 66.096466)
+		(width 0.4064)
+		(layer "F.Cu")
+		(net "Net-(U11-INA+)")
+	)
+	(segment
+		(start 142.520433 66.096466)
+		(end 141.893797 66.723102)
 		(width 0.3048)
 		(layer "F.Cu")
-		(net "Net-(U10-INA+)")
-	)
-	(segment
-		(start 145.285619 79.43288)
-		(end 144.847794 79.870705)
+		(net "Net-(U11-INA+)")
+	)
+	(arc
+		(start 141.893797 66.723102)
+		(mid 141.743286 66.948358)
+		(end 141.690433 67.214066)
 		(width 0.3048)
 		(layer "F.Cu")
-		(net "Net-(U10-INA+)")
-	)
-	(segment
-		(start 146.188167 79.059033)
-		(end 146.521433 78.725766)
+		(net "Net-(U11-INA+)")
+	)
+	(arc
+		(start 142.981233 66.096466)
+		(mid 143.571407 65.979073)
+		(end 144.071733 65.644766)
 		(width 0.4064)
 		(layer "F.Cu")
-		(net "Net-(U10-INA+)")
-	)
-	(segment
-		(start 145.289033 79.431466)
-		(end 145.285619 79.43288)
-		(width 0.2)
-		(layer "F.Cu")
-		(net "Net-(U10-INA+)")
-	)
-	(arc
-		(start 144.663811 80.054688)
-		(mid 144.512253 80.28151)
-		(end 144.459033 80.549066)
-		(width 0.3048)
-		(layer "F.Cu")
-		(net "Net-(U10-INA+)")
-	)
-	(arc
-		(start 145.285619 79.43288)
-		(mid 145.774074 79.33572)
-		(end 146.188167 79.059033)
-		(width 0.4064)
-		(layer "F.Cu")
-		(net "Net-(U10-INA+)")
+		(net "Net-(U11-INA+)")
 	)
 	(segment
@@
 		(net "Net-(U2-ZQ)")
 	)
+	(segment
+		(start 145.099033 80.549066)
+		(end 145.430933 80.549066)
+		(width 0.4064)
+		(layer "F.Cu")
+		(net "Net-(U10-INB-)")
+	)
+	(segment
+		(start 144.895669 81.04003)
+		(end 144.269033 81.666666)
+		(width 0.3048)
+		(layer "F.Cu")
+		(net "Net-(U10-INB-)")
+	)
+	(arc
+		(start 145.430933 80.549066)
+		(mid 146.021107 80.666459)
+		(end 146.521433 81.000766)
+		(width 0.4064)
+		(layer "F.Cu")
+		(net "Net-(U10-INB-)")
+	)
+	(arc
+		(start 145.099033 80.549066)
+		(mid 145.04618 80.814774)
+		(end 144.895669 81.04003)
+		(width 0.3048)
+		(layer "F.Cu")
+		(net "Net-(U10-INB-)")
+	)
+	(generated
+		(type tuning_pattern)
+		(name "Tuning Pattern")
+		(layer "In5.Cu")
+		(base_line
+			(pts
+				(xy 97.989186 94.227211) (xy 97.995564 94.233589) (xy 98.863499 95.101524)
+			)
+		)
+		(base_line_coupled
+			(pts
+				(xy 98.073841 94.948262) (xy 98.071522 94.945943)
+			)
+		)
+		(corner_radius_percent 80)
+		(end
+			(xy 98.863499 95.101524)
+		)
+		(initial_side "left")
+		(is_time_domain no)
+		(last_diff_pair_gap 0.18)
+		(last_netname "FMC_LA24_P")
+		(last_status "tuned")
+		(last_track_width 0.2)
+		(last_tuning_length -1.9e-05)
+		(max_amplitude 1)
+		(min_amplitude 0.2)
+		(min_spacing 0.6)
+		(origin
+			(xy 97.989186 94.227211)
+		)
+		(override_custom_rules no)
+		(rounded yes)
+		(single_sided no)
+		(target_delay 1000000)
+		(target_delay_max 1000000)
+		(target_delay_min 0)
+		(target_length 1000000)
+		(target_length_max 1000000)
+		(target_length_min 0)
+		(target_skew 0)
+		(target_skew_max 0.1)
+		(target_skew_min -0.1)
+		(tuning_mode "diff_pair_skew")
+		(members "03557eca-0ecb-49e5-b31b-f3fac5f75b1e" "236e7baf-d1fb-4be6-9b92-4635a446c849"
+			"323f29a3-625e-47ce-8cb6-f09aa5ed5ef7" "366c705b-d9e0-4ae2-9fdf-9dd111722186"
+			"3b4612fb-1d7b-43d7-a969-fc3ae77bb578" "783180ad-d889-46bf-b6d1-83f36f6f0747"
+			"c5a39420-5e1d-4fd6-92d9-a7892076ad3f" "d69c0aa5-db66-4351-b302-f11c2b9d3726"
+		)
+	)
 	(embedded_fonts no)
