File: KiCad/uranus-fpga-board/uranus-fpga-board.kicad_pcb (KiCad board)
At the start: 8 copper layers, 100 x 100 mm, 73 parts, among them J1 ASP-134486-01, J2 1040100018, J3 TYPE-C-31-M-12, Q1 2N7002, U1 XC7K325T, U10 TLV6700DDCR, U11 TLV6700DDCR, U12 TMUX1108PW, U13 TLV6700DDCR, U15 FT232HL-REEL, U16 93LC56BT, U17 USBLC6-2SC6, U18 TPS564201DDCR, U19 TMUX1108PWR, U2 NT5CB64M16GP-FL, U3 NT5CB64M16GP-FL, U4 NT5CB64M16GP-FL, U5 NT5CB64M16GP-FL, U6 TPS2553DBVR, U7 SY6288F1ABC, U8 SY6874DBC, U9 TLV6700DDCR, Y1 SX7DF200.000B20F30DNN, Y2 3225-12-20-10-10/4B

Commit message: I finally did it
Parts:
- added J4: TYPE-C-31-M-12, Connector_USB:USB_C_Receptacle_HRO_TYPE-C-31-M-12, F.Cu at (58.6, 97.8)
- J2: footprint Connector_PinHeader_1.27mm:PinHeader_2x25_P1.27mm_Vertical_SMD -> Connector_IDC:IDC-Header_2x25_P2.54mm_Vertical_SMD; moved to B.Cu
- J3: value TYPE-C-31-M-12 -> IDC 2x8; footprint Connector_USB:USB_C_Receptacle_HRO_TYPE-C-31-M-12 -> Connector_IDC:IDC-Header_2x08_P2.54mm_Vertical_SMD
- R13: value 1.8 kΩ -> 10 kΩ; footprint Resistor_SMD:R_0402_1005Metric -> Resistor_SMD:R_0201_0603Metric
- R15: value 200 kΩ -> 1.8 kΩ
- R16: value 7.5 kΩ -> 10 kΩ
- R17: value 10 kΩ -> 200 kΩ; footprint Resistor_SMD:R_0201_0603Metric -> Resistor_SMD:R_0402_1005Metric
- R18: value 57.6 kΩ -> 7.5 kΩ; footprint Resistor_SMD:R_0402_1005Metric -> Resistor_SMD:R_0201_0603Metric
- R19, R22: value 499 Ω -> 57.6 kΩ; footprint Resistor_SMD:R_0201_0603Metric -> Resistor_SMD:R_0402_1005Metric
- R20: value 7.68 kΩ -> 57.6 kΩ
- R23: value 7.68 kΩ -> 41.2 kΩ
- R24: value 57.6 kΩ -> 27.4 kΩ
- R25: value 499 Ω -> 21.5 kΩ; footprint Resistor_SMD:R_0201_0603Metric -> Resistor_SMD:R_0402_1005Metric
- R26: value 7.68 kΩ -> 200 kΩ; footprint Resistor_SMD:R_0402_1005Metric -> Resistor_SMD:R_0201_0603Metric
- R27: value 10 kΩ -> 200 kΩ
- R28: value 499 Ω -> 200 kΩ
- R29: value 7.68 kΩ -> 15.8 kΩ
- R30: value 15.8 kΩ -> 499 Ω; footprint Resistor_SMD:R_0402_1005Metric -> Resistor_SMD:R_0201_0603Metric
- R31: value 21.5 kΩ -> 7.68 kΩ
- R32: value 27.4 kΩ -> 499 Ω; footprint Resistor_SMD:R_0402_1005Metric -> Resistor_SMD:R_0201_0603Metric
- R33: value 41.2 kΩ -> 7.68 kΩ
- R34: value 57.6 kΩ -> 499 Ω; footprint Resistor_SMD:R_0402_1005Metric -> Resistor_SMD:R_0201_0603Metric
- R35, R37: value 200 kΩ -> 7.68 kΩ; footprint Resistor_SMD:R_0201_0603Metric -> Resistor_SMD:R_0402_1005Metric
- R36: value 200 kΩ -> 499 Ω
- R41: value 52.3 kΩ -> 8.98 kΩ; footprint Resistor_SMD:R_0402_1005Metric -> Resistor_SMD:R_0603_1608Metric
- R42: value 30.9 kΩ -> 200 kΩ; footprint Resistor_SMD:R_0402_1005Metric -> Resistor_SMD:R_0201_0603Metric
- R43: value 22.1 kΩ -> 200 kΩ; footprint Resistor_SMD:R_0402_1005Metric -> Resistor_SMD:R_0201_0603Metric
- R44: value 13 kΩ -> 200 kΩ; footprint Resistor_SMD:R_0402_1005Metric -> Resistor_SMD:R_0201_0603Metric
- R45: value 8.98 kΩ -> 13 kΩ; footprint Resistor_SMD:R_0603_1608Metric -> Resistor_SMD:R_0402_1005Metric
- R46: value 200 kΩ -> 22.1 kΩ; footprint Resistor_SMD:R_0201_0603Metric -> Resistor_SMD:R_0402_1005Metric
- R47: value 200 kΩ -> 30.9 kΩ; footprint Resistor_SMD:R_0201_0603Metric -> Resistor_SMD:R_0402_1005Metric
- R48: value 200 kΩ -> 52.3 kΩ; footprint Resistor_SMD:R_0201_0603Metric -> Resistor_SMD:R_0402_1005Metric
- U1: value XC7K325T -> XC7K325T-3FFG900E; footprint XC7K325T-3FFG900E:FFG900XC7K325T_AMD -> Package_BGA:Xilinx_FFG900_FFG901
- U12: value TMUX1108PW -> TLV6700DDCR; footprint Package_SO:TSSOP-16_4.4x5mm_P0.65mm -> Package_TO_SOT_SMD:SOT-23-6
- U19: value TMUX1108PWR -> TMUX1108
- U6: value TPS2553DBVR -> SY6874DBC; footprint Package_TO_SOT_SMD:SOT-23-6 -> Package_DFN_QFN:DFN-10-1EP_3x3mm_P0.5mm_EP1.75x2.7mm
- U7: value SY6288F1ABC -> TPS2553DBVR
- U8: value SY6874DBC -> SY6288F1ABC; footprint Package_DFN_QFN:DFN-10-1EP_3x3mm_P0.5mm_EP1.75x2.7mm -> Package_TO_SOT_SMD:SOT-23-6
- U9: value TLV6700DDCR -> TMUX1108; footprint Package_TO_SOT_SMD:SOT-23-6 -> Package_SO:TSSOP-16_4.4x5mm_P0.65mm
- moved R1 153.3 mm to (228.4, 122.8)
- moved R2 153.3 mm to (228.4, 124.8)
- moved R3 153.3 mm to (228.4, 126.8)
- moved R42 151.6 mm to (210.5, 132.8)
- moved R43 151.6 mm to (210.5, 134.5)
- moved R44 151.6 mm to (210.5, 136.3)
- moved R10 149.2 mm to (228.1, 141.3)
- moved R11 149.2 mm to (228.1, 143.3)
- moved R12 149.2 mm to (228.1, 145.3)
- moved R41 146.0 mm to (204.5, 135.3)
- moved L1 142.2 mm to (205.9, 131.2)
- moved R38 142.2 mm to (210.5, 129.3)
- moved R39 142.2 mm to (201.1, 129.4)
- moved R40 142.2 mm to (210.5, 131.0)
- moved U18 142.2 mm to (211.3, 124.2)
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Connections:
- net DDR_A0 renamed /RAM/A0
- net DDR_A1 renamed /RAM/A1
- net DDR_A10 renamed /RAM/A10
- net DDR_A11 renamed /RAM/A11
- net DDR_A12 renamed /RAM/A12
- net DDR_A2 renamed /RAM/A2
- net DDR_A3 renamed /RAM/A3
- net DDR_A4 renamed /RAM/A4
- net DDR_A5 renamed /RAM/A5
- net DDR_A6 renamed /RAM/A6
- net DDR_A7 renamed /RAM/A7
- net DDR_A8 renamed /RAM/A8
- net DDR_A9 renamed /RAM/A9
- net DDR_BA0 renamed /RAM/BA0
- net DDR_BA1 renamed /RAM/BA1
- net DDR_BA2 renamed /RAM/BA2
- net DDR_CKE renamed /FPGA/CKE
- net DDR_CK_N renamed /RAM/CK_N
- net DDR_CK_P renamed /RAM/CK_P
- net DDR_CLK_N renamed /FPGA/IO Banks/32 33 34/CLK_N
- net DDR_CLK_P renamed /FPGA/IO Banks/32 33 34/CLK_P
- net DDR_DM0 renamed /FPGA/L0.DM
- net DDR_DM1 renamed /FPGA/H0.DM
- net DDR_DM2 renamed /FPGA/L1.DM
- net DDR_DM3 renamed /FPGA/H1.DM
- net DDR_DM4 renamed /FPGA/L2.DM
- net DDR_DM5 renamed /FPGA/H2.DM
- net DDR_DQ00 renamed /FPGA/L0.DQ0
- net DDR_DQ01 renamed /FPGA/L0.DQ1
- net DDR_DQ02 renamed /FPGA/L0.DQ2
- net DDR_DQ03 renamed /FPGA/L0.DQ3
- net DDR_DQ04 renamed /FPGA/L0.DQ4
- net DDR_DQ05 renamed /FPGA/L0.DQ5
- net DDR_DQ06 renamed /FPGA/L0.DQ6
- net DDR_DQ07 renamed /FPGA/L0.DQ7
- net DDR_DQ08 renamed /FPGA/H0.DQ0
- net DDR_DQ09 renamed /FPGA/H0.DQ1
- net DDR_DQ10 renamed /FPGA/H0.DQ2
- net DDR_DQ11 renamed /FPGA/H0.DQ3
- net DDR_DQ12 renamed /FPGA/H0.DQ4
- net DDR_DQ13 renamed /FPGA/H0.DQ5
- net DDR_DQ14 renamed /FPGA/H0.DQ6
- net DDR_DQ15 renamed /FPGA/H0.DQ7
- net DDR_DQ16 renamed /FPGA/L1.DQ0
- net DDR_DQ17 renamed /FPGA/L1.DQ1
- net DDR_DQ18 renamed /FPGA/L1.DQ2
- net DDR_DQ19 renamed /FPGA/L1.DQ3
- net DDR_DQ20 renamed /FPGA/L1.DQ4
- net DDR_DQ21 renamed /FPGA/L1.DQ5
- net DDR_DQ22 renamed /FPGA/L1.DQ6
- net DDR_DQ23 renamed /FPGA/L1.DQ7
- net DDR_DQ24 renamed /FPGA/H1.DQ0
- net DDR_DQ25 renamed /FPGA/H1.DQ1
- net DDR_DQ26 renamed /FPGA/H1.DQ2
- net DDR_DQ27 renamed /FPGA/H1.DQ3
- net DDR_DQ28 renamed /FPGA/H1.DQ4
- net DDR_DQ29 renamed /FPGA/H1.DQ5
- net DDR_DQ30 renamed /FPGA/H1.DQ6
- net DDR_DQ31 renamed /FPGA/H1.DQ7
- net DDR_DQ32 renamed /FPGA/L2.DQ0
- net DDR_DQ33 renamed /FPGA/L2.DQ1
- net DDR_DQ34 renamed /FPGA/L2.DQ2
- net DDR_DQ35 renamed /FPGA/L2.DQ3
- net DDR_DQ36 renamed /FPGA/L2.DQ4
- net DDR_DQ37 renamed /FPGA/L2.DQ5
- net DDR_DQ38 renamed /FPGA/L2.DQ6
- net DDR_DQ39 renamed /FPGA/L2.DQ7
- net DDR_DQ40 renamed /FPGA/H2.DQ0
- net DDR_DQ41 renamed /FPGA/H2.DQ1
- net DDR_DQ42 renamed /FPGA/H2.DQ2
- net DDR_DQ43 renamed /FPGA/H2.DQ3
- net DDR_DQ44 renamed /FPGA/H2.DQ4
- net DDR_DQ45 renamed /FPGA/H2.DQ5
- net DDR_DQ46 renamed /FPGA/H2.DQ6
- net DDR_DQ47 renamed /FPGA/H2.DQ7
- net DDR_DQS_N0 renamed /FPGA/L0.DQS_N
- net DDR_DQS_N1 renamed /FPGA/H0.DQS_N
- net DDR_DQS_N2 renamed /FPGA/L1.DQS_N
- net DDR_DQS_N3 renamed /FPGA/H1.DQS_N
- net DDR_DQS_N4 renamed /FPGA/L2.DQS_N
- net DDR_DQS_N5 renamed /FPGA/H2.DQS_N
- net DDR_DQS_P0 renamed /FPGA/L0.DQS_P
- net DDR_DQS_P1 renamed /FPGA/H0.DQS_P
- net DDR_DQS_P2 renamed /FPGA/L1.DQS_P
- net DDR_DQS_P3 renamed /FPGA/H1.DQS_P
- net DDR_DQS_P4 renamed /FPGA/L2.DQS_P
- net DDR_DQS_P5 renamed /FPGA/H2.DQS_P
- net DDR_ODT renamed /FPGA/ODT
- net DDR_REF_N renamed /FPGA/IO Banks/32 33 34/REF_N
- net DDR_REF_P renamed /FPGA/IO Banks/32 33 34/REF_P
- net FMC_DP0_C2M_N renamed /FMC/DP0_C2M_N
- net FMC_DP0_C2M_P renamed /FMC/DP0_C2M_P
- net FMC_DP0_M2C_N renamed /FMC/DP0_M2C_N
- net FMC_DP0_M2C_P renamed /FMC/DP0_M2C_P
- net FMC_LA00_CC_N renamed /FMC/LA00_CC_N
- net FMC_LA00_CC_P renamed /FMC/LA00_CC_P
- net FMC_LA01_N renamed /FMC/LA01_N
- net FMC_LA01_P renamed /FMC/LA01_P
- net FMC_LA02_N renamed /FMC/LA02_N
- net FMC_LA02_P renamed /FMC/LA02_P
- net FMC_LA03_N renamed /FMC/LA03_N
- net FMC_LA03_P renamed /FMC/LA03_P
- net FMC_LA04_N renamed /FMC/LA04_N
- net FMC_LA04_P renamed /FMC/LA04_P
- net FMC_LA05_N renamed /FMC/LA05_N
- net FMC_LA05_P renamed /FMC/LA05_P
- net FMC_LA06_N renamed /FMC/LA06_N
- net FMC_LA06_P renamed /FMC/LA06_P
- net FMC_LA07_N renamed /FMC/LA07_N
- net FMC_LA07_P renamed /FMC/LA07_P
- net FMC_LA08_N renamed /FMC/LA08_N
- net FMC_LA08_P renamed /FMC/LA08_P
- net FMC_LA09_N renamed /FMC/LA09_N
- net FMC_LA09_P renamed /FMC/LA09_P
- net FMC_LA10_N renamed /FMC/LA10_N
- net FMC_LA10_P renamed /FMC/LA10_P
- net FMC_LA11_N renamed /FMC/LA11_N
- net FMC_LA11_P renamed /FMC/LA11_P
- net FMC_LA12_N renamed /FMC/LA12_N
- net FMC_LA12_P renamed /FMC/LA12_P
- net FMC_LA13_N renamed /FMC/LA13_N
- net FMC_LA13_P renamed /FMC/LA13_P
- net FMC_LA14_N renamed /FMC/LA14_N
- net FMC_LA14_P renamed /FMC/LA14_P
- net FMC_LA15_N renamed /FMC/LA15_N
- net FMC_LA15_P renamed /FMC/LA15_P
- net FMC_LA16_N renamed /FMC/LA16_N
- net FMC_LA16_P renamed /FMC/LA16_P
- net FMC_LA17_CC_N renamed /FMC/LA17_CC_N
- net FMC_LA17_CC_P renamed /FMC/LA17_CC_P
- net FMC_LA18_CC_N renamed /FMC/LA18_CC_N
- net FMC_LA18_CC_P renamed /FMC/LA18_CC_P
- net FMC_LA19_N renamed /FMC/LA19_N
- net FMC_LA19_P renamed /FMC/LA19_P
- net FMC_LA20_N renamed /FMC/LA20_N
- net FMC_LA20_P renamed /FMC/LA20_P
- net FMC_LA21_N renamed /FMC/LA21_N
- net FMC_LA21_P renamed /FMC/LA21_P
- net FMC_LA22_N renamed /FMC/LA22_N
- net FMC_LA22_P renamed /FMC/LA22_P
- net FMC_LA23_N renamed /FMC/LA23_N
- net FMC_LA23_P renamed /FMC/LA23_P
- net FMC_LA24_N renamed /FMC/LA24_N
- net FMC_LA24_P renamed /FMC/LA24_P
- net FMC_LA25_N renamed /FMC/LA25_N
- net FMC_LA25_P renamed /FMC/LA25_P
- net FMC_LA26_N renamed /FMC/LA26_N
- net FMC_LA26_P renamed /FMC/LA26_P
- net FMC_LA27_N renamed /FMC/LA27_N
- net FMC_LA27_P renamed /FMC/LA27_P
- net FMC_LA28_N renamed /FMC/LA28_N
- net FMC_LA28_P renamed /FMC/LA28_P
- net FMC_LA29_N renamed /FMC/LA29_N
- net FMC_LA29_P renamed /FMC/LA29_P
- net FMC_LA30_N renamed /FMC/LA30_N
- net FMC_LA30_P renamed /FMC/LA30_P
- net FMC_LA31_N renamed /FMC/LA31_N
- net FMC_LA31_P renamed /FMC/LA31_P
- net FMC_LA32_N renamed /FMC/LA32_N
- net FMC_LA32_P renamed /FMC/LA32_P
- net FMC_LA33_N renamed /FMC/LA33_N
- net FMC_LA33_P renamed /FMC/LA33_P
- net FMC_SCL renamed /FMC/SCL
- net FMC_SDA renamed /FMC/SDA
- net FMC_TCK renamed /FMC/TCK
- net FMC_TDI renamed /FMC/TDI
- net FMC_TDO renamed /FMC/TDO
- net FMC_TMS renamed /FMC/TMS
- net FMC_TRST_L renamed /FMC/~{TRST}
- net J2_CLK0 renamed /FPGA/IDC_B13_CLK
- net J2_CLK1 renamed /FPGA/IDC_B14_CLK
- net J2_DB0 renamed /FPGA/J2_B13.D0
- net J2_DB1 renamed /FPGA/J2_B13.D1
- net J2_DB10 renamed /FPGA/J2_B13.D10
- net J2_DB11 renamed /FPGA/J2_B13.D11
- net J2_DB12 renamed /FPGA/J2_B13.D12
- net J2_DB13 renamed /FPGA/J2_B13.D13
- net J2_DB14 renamed /FPGA/J2_B13.D14
- net J2_DB15 renamed /FPGA/J2_B13.D15
- net J2_DB16 renamed /FPGA/J2_B15.D0
- net J2_DB17 renamed /FPGA/J2_B15.D1
- net J2_DB18 renamed /FPGA/J2_B15.D2
- net J2_DB19 renamed /FPGA/J2_B15.D3
- net J2_DB2 renamed /FPGA/J2_B13.D2
- net J2_DB20 renamed /FPGA/J2_B15.D4
- net J2_DB21 renamed /FPGA/J2_B15.D5
- net J2_DB22 renamed /FPGA/J2_B15.D6
- net J2_DB23 renamed /FPGA/J2_B15.D7
- net J2_DB24 renamed /FPGA/J2_B15.D8
- net J2_DB25 renamed /FPGA/J2_B15.D9
- net J2_DB26 renamed /FPGA/J2_B15.D10
- net J2_DB27 renamed /FPGA/J2_B15.D11
- net J2_DB28 renamed /FPGA/J2_B15.D12
- net J2_DB29 renamed /FPGA/J2_B15.D13
- net J2_DB3 renamed /FPGA/J2_B13.D3
- net J2_DB30 renamed /FPGA/J2_B15.D14
- net J2_DB31 renamed /FPGA/J2_B15.D15
- net J2_DB4 renamed /FPGA/J2_B13.D4
- net J2_DB5 renamed /FPGA/J2_B13.D5
- net J2_DB6 renamed /FPGA/J2_B13.D6
- net J2_DB7 renamed /FPGA/J2_B13.D7
- net J2_DB8 renamed /FPGA/J2_B13.D8
- net J2_DB9 renamed /FPGA/J2_B13.D9
- net J2_WRT0 renamed /FPGA/IDC_B13_WRT
- net J2_WRT1 renamed /FPGA/IDC_B14_WRT
- net Net-(U18-VFB) renamed /Power/VADJ/VFB
- net U2_VREF renamed Net-(U2-VREFCA)
- net U3_VREF renamed Net-(U3-VREFCA)
- net U4_VREF renamed Net-(U4-VREFCA)
- net U5_VREF renamed Net-(U5-VREFCA)
- net VADJ_REG_EN renamed /FMC/REG_EN
- net ~{DDR_CAS} renamed /FPGA/~{CAS}
- net ~{DDR_CS} renamed /FPGA/~{CS}
- net ~{DDR_RAS} renamed /FPGA/~{RAS}
- net ~{DDR_WE} renamed /FPGA/~{WE}
- J1 pad A01: unconnected-(J1-PadA01) -> (no net)
- J1 pad A02: unconnected-(J1-PadA02) -> (no net)
- J1 pad A03: unconnected-(J1-PadA03) -> (no net)
- J1 pad A04: unconnected-(J1-PadA04) -> (no net)
- J1 pad A05: unconnected-(J1-PadA05) -> (no net)
- J1 pad A06: unconnected-(J1-PadA06) -> (no net)
- J1 pad A07: unconnected-(J1-PadA07) -> (no net)
- J1 pad A08: unconnected-(J1-PadA08) -> (no net)
- J1 pad A09: unconnected-(J1-PadA09) -> (no net)
- J1 pad A10: unconnected-(J1-PadA10) -> (no net)
- J1 pad A11: unconnected-(J1-PadA11) -> (no net)
- J1 pad A12: unconnected-(J1-PadA12) -> (no net)
- J1 pad A13: unconnected-(J1-PadA13) -> (no net)
- J1 pad A14: unconnected-(J1-PadA14) -> (no net)
- J1 pad A15: unconnected-(J1-PadA15) -> (no net)
- J1 pad A16: unconnected-(J1-PadA16) -> (no net)
- J1 pad A17: unconnected-(J1-PadA17) -> (no net)
- J1 pad A18: unconnected-(J1-PadA18) -> (no net)
- J1 pad A19: unconnected-(J1-PadA19) -> (no net)
- J1 pad A20: unconnected-(J1-PadA20) -> (no net)
- J1 pad A21: unconnected-(J1-PadA21) -> (no net)
- J1 pad A22: unconnected-(J1-PadA22) -> (no net)
- J1 pad A23: unconnected-(J1-PadA23) -> (no net)
- J1 pad A24: unconnected-(J1-PadA24) -> (no net)
- J1 pad A25: unconnected-(J1-PadA25) -> (no net)
- J1 pad A26: unconnected-(J1-PadA26) -> (no net)
- J1 pad A27: unconnected-(J1-PadA27) -> (no net)
- J1 pad A28: unconnected-(J1-PadA28) -> (no net)
- J1 pad A29: unconnected-(J1-PadA29) -> (no net)
- J1 pad A30: unconnected-(J1-PadA30) -> (no net)
- J1 pad A31: unconnected-(J1-PadA31) -> (no net)
- J1 pad A32: unconnected-(J1-PadA32) -> (no net)
- J1 pad A33: unconnected-(J1-PadA33) -> (no net)
- J1 pad A34: unconnected-(J1-PadA34) -> (no net)
- J1 pad A35: unconnected-(J1-PadA35) -> (no net)
- J1 pad A36: unconnected-(J1-PadA36) -> (no net)
- J1 pad A37: unconnected-(J1-PadA37) -> (no net)
- J1 pad A38: unconnected-(J1-PadA38) -> (no net)
- J1 pad A39: unconnected-(J1-PadA39) -> (no net)
- J1 pad A40: unconnected-(J1-PadA40) -> (no net)
- J1 pad B01: unconnected-(J1-PadB01) -> (no net)
- J1 pad B02: unconnected-(J1-PadB02) -> (no net)
- J1 pad B03: unconnected-(J1-PadB03) -> (no net)
- J1 pad B04: unconnected-(J1-PadB04) -> (no net)
- J1 pad B05: unconnected-(J1-PadB05) -> (no net)
- J1 pad B06: unconnected-(J1-PadB06) -> (no net)
- J1 pad B07: unconnected-(J1-PadB07) -> (no net)
- J1 pad B08: unconnected-(J1-PadB08) -> (no net)
- J1 pad B09: unconnected-(J1-PadB09) -> (no net)
- J1 pad B10: unconnected-(J1-PadB10) -> (no net)
- J1 pad B11: unconnected-(J1-PadB11) -> (no net)
- J1 pad B12: unconnected-(J1-PadB12) -> (no net)
- J1 pad B13: unconnected-(J1-PadB13) -> (no net)
- J1 pad B14: unconnected-(J1-PadB14) -> (no net)
- J1 pad B15: unconnected-(J1-PadB15) -> (no net)
- J1 pad B16: unconnected-(J1-PadB16) -> (no net)
- J1 pad B17: unconnected-(J1-PadB17) -> (no net)
- J1 pad B18: unconnected-(J1-PadB18) -> (no net)
- J1 pad B19: unconnected-(J1-PadB19) -> (no net)
- J1 pad B20: unconnected-(J1-PadB20) -> (no net)
- J1 pad B21: unconnected-(J1-PadB21) -> (no net)
- J1 pad B22: unconnected-(J1-PadB22) -> (no net)
- J1 pad B23: unconnected-(J1-PadB23) -> (no net)
- J1 pad B24: unconnected-(J1-PadB24) -> (no net)
- J1 pad B25: unconnected-(J1-PadB25) -> (no net)
- J1 pad B26: unconnected-(J1-PadB26) -> (no net)
- J1 pad B27: unconnected-(J1-PadB27) -> (no net)
- J1 pad B28: unconnected-(J1-PadB28) -> (no net)
- J1 pad B29: unconnected-(J1-PadB29) -> (no net)
- J1 pad B30: unconnected-(J1-PadB30) -> (no net)
- J1 pad B31: unconnected-(J1-PadB31) -> (no net)
- J1 pad B32: unconnected-(J1-PadB32) -> (no net)
- J1 pad B33: unconnected-(J1-PadB33) -> (no net)
- J1 pad B34: unconnected-(J1-PadB34) -> (no net)
- J1 pad B35: unconnected-(J1-PadB35) -> (no net)
- J1 pad B36: unconnected-(J1-PadB36) -> (no net)
- J1 pad B37: unconnected-(J1-PadB37) -> (no net)
- J1 pad B38: unconnected-(J1-PadB38) -> (no net)
- J1 pad B39: unconnected-(J1-PadB39) -> (no net)
- J1 pad B40: unconnected-(J1-PadB40) -> (no net)
- J1 pad C35: +12V0_P -> +12V0
- J1 pad C37: +12V0_P -> +12V0
- J1 pad D01: FMC_PG_C2M -> /FMC/PG
- J1 pad D04: FMC_GPTCLK0_M2C_P -> /FMC/GTXCLK0_P
- J1 pad D05: FMC_GBTCLK0_M2C_N -> /FMC/GTXCLK0_N
- J1 pad E01: unconnected-(J1-PadE01) -> (no net)
- J1 pad E02: unconnected-(J1-PadE02) -> (no net)
- J1 pad E03: unconnected-(J1-PadE03) -> (no net)
- J1 pad E04: unconnected-(J1-PadE04) -> (no net)
- J1 pad E05: unconnected-(J1-PadE05) -> (no net)
- J1 pad E06: unconnected-(J1-PadE06) -> (no net)
- J1 pad E07: unconnected-(J1-PadE07) -> (no net)
- J1 pad E08: unconnected-(J1-PadE08) -> (no net)
- J1 pad E09: unconnected-(J1-PadE09) -> (no net)
- J1 pad E10: unconnected-(J1-PadE10) -> (no net)
- J1 pad E11: unconnected-(J1-PadE11) -> (no net)
- J1 pad E12: unconnected-(J1-PadE12) -> (no net)
- J1 pad E13: unconnected-(J1-PadE13) -> (no net)
- J1 pad E14: unconnected-(J1-PadE14) -> (no net)
- J1 pad E15: unconnected-(J1-PadE15) -> (no net)
- J1 pad E16: unconnected-(J1-PadE16) -> (no net)
- J1 pad E17: unconnected-(J1-PadE17) -> (no net)
- J1 pad E18: unconnected-(J1-PadE18) -> (no net)
- J1 pad E19: unconnected-(J1-PadE19) -> (no net)
- J1 pad E20: unconnected-(J1-PadE20) -> (no net)
- J1 pad E21: unconnected-(J1-PadE21) -> (no net)
- J1 pad E22: unconnected-(J1-PadE22) -> (no net)
- J1 pad E23: unconnected-(J1-PadE23) -> (no net)
- J1 pad E24: unconnected-(J1-PadE24) -> (no net)
- J1 pad E25: unconnected-(J1-PadE25) -> (no net)
- J1 pad E26: unconnected-(J1-PadE26) -> (no net)
- J1 pad E27: unconnected-(J1-PadE27) -> (no net)
- J1 pad E28: unconnected-(J1-PadE28) -> (no net)
- J1 pad E29: unconnected-(J1-PadE29) -> (no net)
- J1 pad E30: unconnected-(J1-PadE30) -> (no net)
- J1 pad E31: unconnected-(J1-PadE31) -> (no net)
- J1 pad E32: unconnected-(J1-PadE32) -> (no net)
- J1 pad E33: unconnected-(J1-PadE33) -> (no net)
- J1 pad E34: unconnected-(J1-PadE34) -> (no net)
- J1 pad E35: unconnected-(J1-PadE35) -> (no net)
- J1 pad E36: unconnected-(J1-PadE36) -> (no net)
- J1 pad E37: unconnected-(J1-PadE37) -> (no net)
- J1 pad E38: unconnected-(J1-PadE38) -> (no net)
- J1 pad E39: unconnected-(J1-PadE39) -> (no net)
- J1 pad E40: unconnected-(J1-PadE40) -> (no net)
- J1 pad F01: unconnected-(J1-PadF01) -> (no net)
- J1 pad F02: unconnected-(J1-PadF02) -> (no net)
- J1 pad F03: unconnected-(J1-PadF03) -> (no net)
- J1 pad F04: unconnected-(J1-PadF04) -> (no net)
- J1 pad F05: unconnected-(J1-PadF05) -> (no net)
- J1 pad F06: unconnected-(J1-PadF06) -> (no net)
- J1 pad F07: unconnected-(J1-PadF07) -> (no net)
- J1 pad F08: unconnected-(J1-PadF08) -> (no net)
- J1 pad F09: unconnected-(J1-PadF09) -> (no net)
- J1 pad F10: unconnected-(J1-PadF10) -> (no net)
- J1 pad F11: unconnected-(J1-PadF11) -> (no net)
- J1 pad F12: unconnected-(J1-PadF12) -> (no net)
- J1 pad F13: unconnected-(J1-PadF13) -> (no net)
- J1 pad F14: unconnected-(J1-PadF14) -> (no net)
- J1 pad F15: unconnected-(J1-PadF15) -> (no net)
- J1 pad F16: unconnected-(J1-PadF16) -> (no net)
- J1 pad F17: unconnected-(J1-PadF17) -> (no net)
- J1 pad F18: unconnected-(J1-PadF18) -> (no net)
- J1 pad F19: unconnected-(J1-PadF19) -> (no net)
- J1 pad F20: unconnected-(J1-PadF20) -> (no net)
- J1 pad F21: unconnected-(J1-PadF21) -> (no net)
- J1 pad F22: unconnected-(J1-PadF22) -> (no net)
- J1 pad F23: unconnected-(J1-PadF23) -> (no net)
- J1 pad F24: unconnected-(J1-PadF24) -> (no net)
- J1 pad F25: unconnected-(J1-PadF25) -> (no net)
- J1 pad F26: unconnected-(J1-PadF26) -> (no net)
- J1 pad F27: unconnected-(J1-PadF27) -> (no net)
- J1 pad F28: unconnected-(J1-PadF28) -> (no net)
- J1 pad F29: unconnected-(J1-PadF29) -> (no net)
- J1 pad F30: unconnected-(J1-PadF30) -> (no net)
- J1 pad F31: unconnected-(J1-PadF31) -> (no net)
- J1 pad F32: unconnected-(J1-PadF32) -> (no net)
- J1 pad F33: unconnected-(J1-PadF33) -> (no net)
- J1 pad F34: unconnected-(J1-PadF34) -> (no net)
- J1 pad F35: unconnected-(J1-PadF35) -> (no net)
- J1 pad F36: unconnected-(J1-PadF36) -> (no net)
- J1 pad F37: unconnected-(J1-PadF37) -> (no net)
- J1 pad F38: unconnected-(J1-PadF38) -> (no net)
- J1 pad F39: unconnected-(J1-PadF39) -> (no net)
- J1 pad F40: unconnected-(J1-PadF40) -> (no net)
- J1 pad G02: FMC_CLK1_M2C_P -> /FMC/CLK1_P
- J1 pad G03: FMC_CLK1_M2C_N -> /FMC/CLK1_N
- J1 pad H02: ~{FMC_PRSNT_M2C} -> /FMC/Power Management/~{PRSNT}
- J1 pad H04: FMC_CLK0_M2C_P -> /FMC/CLK0_P
- J1 pad H05: FMC_CLK0_M2C_N -> /FMC/CLK0_N
- J1 pad J01: unconnected-(J1-PadJ01) -> (no net)
- J1 pad J02: unconnected-(J1-PadJ02) -> (no net)
- J1 pad J03: unconnected-(J1-PadJ03) -> (no net)
- J1 pad J04: unconnected-(J1-PadJ04) -> (no net)
- J1 pad J05: unconnected-(J1-PadJ05) -> (no net)
- J1 pad J06: unconnected-(J1-PadJ06) -> (no net)
- J1 pad J07: unconnected-(J1-PadJ07) -> (no net)
- J1 pad J08: unconnected-(J1-PadJ08) -> (no net)
- J1 pad J09: unconnected-(J1-PadJ09) -> (no net)
- J1 pad J10: unconnected-(J1-PadJ10) -> (no net)
- J1 pad J11: unconnected-(J1-PadJ11) -> (no net)
- J1 pad J12: unconnected-(J1-PadJ12) -> (no net)
- J1 pad J13: unconnected-(J1-PadJ13) -> (no net)
- J1 pad J14: unconnected-(J1-PadJ14) -> (no net)
- J1 pad J15: unconnected-(J1-PadJ15) -> (no net)
- J1 pad J16: unconnected-(J1-PadJ16) -> (no net)
- J1 pad J17: unconnected-(J1-PadJ17) -> (no net)
- J1 pad J18: unconnected-(J1-PadJ18) -> (no net)
- J1 pad J19: unconnected-(J1-PadJ19) -> (no net)
- J1 pad J20: unconnected-(J1-PadJ20) -> (no net)
- J1 pad J21: unconnected-(J1-PadJ21) -> (no net)
- J1 pad J22: unconnected-(J1-PadJ22) -> (no net)
- J1 pad J23: unconnected-(J1-PadJ23) -> (no net)
- J1 pad J24: unconnected-(J1-PadJ24) -> (no net)
- J1 pad J25: unconnected-(J1-PadJ25) -> (no net)
- J1 pad J26: unconnected-(J1-PadJ26) -> (no net)
- J1 pad J27: unconnected-(J1-PadJ27) -> (no net)
- J1 pad J28: unconnected-(J1-PadJ28) -> (no net)
- J1 pad J29: unconnected-(J1-PadJ29) -> (no net)
- J1 pad J30: unconnected-(J1-PadJ30) -> (no net)
- J1 pad J31: unconnected-(J1-PadJ31) -> (no net)
- J1 pad J32: unconnected-(J1-PadJ32) -> (no net)
- J1 pad J33: unconnected-(J1-PadJ33) -> (no net)
- J1 pad J34: unconnected-(J1-PadJ34) -> (no net)
- J1 pad J35: unconnected-(J1-PadJ35) -> (no net)
- J1 pad J36: unconnected-(J1-PadJ36) -> (no net)
- J1 pad J37: unconnected-(J1-PadJ37) -> (no net)
- J1 pad J38: unconnected-(J1-PadJ38) -> (no net)
- J1 pad J39: unconnected-(J1-PadJ39) -> (no net)
- J1 pad J40: unconnected-(J1-PadJ40) -> (no net)
- J1 pad K01: unconnected-(J1-PadK01) -> (no net)
- J1 pad K02: unconnected-(J1-PadK02) -> (no net)
- J1 pad K03: unconnected-(J1-PadK03) -> (no net)
- J1 pad K04: unconnected-(J1-PadK04) -> (no net)
- J1 pad K05: unconnected-(J1-PadK05) -> (no net)
- J1 pad K06: unconnected-(J1-PadK06) -> (no net)
- J1 pad K07: unconnected-(J1-PadK07) -> (no net)
- J1 pad K08: unconnected-(J1-PadK08) -> (no net)
- J1 pad K09: unconnected-(J1-PadK09) -> (no net)
- J1 pad K10: unconnected-(J1-PadK10) -> (no net)
- J1 pad K11: unconnected-(J1-PadK11) -> (no net)
- J1 pad K12: unconnected-(J1-PadK12) -> (no net)
- J1 pad K13: unconnected-(J1-PadK13) -> (no net)
- J1 pad K14: unconnected-(J1-PadK14) -> (no net)
- J1 pad K15: unconnected-(J1-PadK15) -> (no net)
- J1 pad K16: unconnected-(J1-PadK16) -> (no net)
- J1 pad K17: unconnected-(J1-PadK17) -> (no net)
- J1 pad K18: unconnected-(J1-PadK18) -> (no net)
- J1 pad K19: unconnected-(J1-PadK19) -> (no net)
- J1 pad K20: unconnected-(J1-PadK20) -> (no net)
- J1 pad K21: unconnected-(J1-PadK21) -> (no net)
- J1 pad K22: unconnected-(J1-PadK22) -> (no net)
- J1 pad K23: unconnected-(J1-PadK23) -> (no net)
- J1 pad K24: unconnected-(J1-PadK24) -> (no net)
- J1 pad K25: unconnected-(J1-PadK25) -> (no net)
- J1 pad K26: unconnected-(J1-PadK26) -> (no net)
- J1 pad K27: unconnected-(J1-PadK27) -> (no net)
- J1 pad K28: unconnected-(J1-PadK28) -> (no net)
- J1 pad K29: unconnected-(J1-PadK29) -> (no net)
- J1 pad K30: unconnected-(J1-PadK30) -> (no net)
- J1 pad K31: unconnected-(J1-PadK31) -> (no net)
- J1 pad K32: unconnected-(J1-PadK32) -> (no net)
- J1 pad K33: unconnected-(J1-PadK33) -> (no net)
- J1 pad K34: unconnected-(J1-PadK34) -> (no net)
- J1 pad K35: unconnected-(J1-PadK35) -> (no net)
- J1 pad K36: unconnected-(J1-PadK36) -> (no net)
- J1 pad K37: unconnected-(J1-PadK37) -> (no net)
- J1 pad K38: unconnected-(J1-PadK38) -> (no net)
- J1 pad K39: unconnected-(J1-PadK39) -> (no net)
- J1 pad K40: unconnected-(J1-PadK40) -> (no net)
- Q1 pad 1: ~{FMC_PRSNT_M2C} -> /FMC/Power Management/~{PRSNT}
- Q1 pad 3: FMC_PRSNT -> /FMC/Power Management/PRSNT
- R12 pad 1: GND -> Net-(U5-ZQ)
- R12 pad 2: Net-(U5-ZQ) -> GND
- R13 pad 1: GND -> +3V3
- R13 pad 2: Net-(U7-ISET) -> /FMC/Power Management/~{PRSNT}
- R14 pad 1: +3V3 -> +3V3_P
- R14 pad 2: FMC_PRSNT -> /FMC/PG
- R15 pad 1: Net-(U6-ILIM) -> Net-(U8-ILIM)
- R16 pad 1: GND -> +3V3
- R16 pad 2: Net-(U8-ILIM) -> /FMC/Power Management/PRSNT
- R17 pad 1: +3V3_P -> Net-(U7-ILIM)
- R17 pad 2: FMC_PG_C2M -> GND
- R18 pad 1: +3V3AUX -> Net-(U6-ILIM)
- R18 pad 2: Net-(U9-INA+) -> GND
- R19 pad 1: Net-(U9-INA+) -> /FMC/Power Management/Window Comparator +3V3AUX/IN
- R19 pad 2: Net-(U9-INB-) -> +3V3AUX
- R20 pad 1: Net-(U9-INB-) -> /FMC/Power Management/Window Comparator +3V3_P/IN
- R20 pad 2: GND -> +3V3_P
- R21 pad 1: +12V0_P -> /FMC/Power Management/Window Comparator +12V0_P/IN
- R21 pad 2: Net-(U10-INA+) -> +12V0_P
- R22 pad 1: Net-(U10-INA+) -> Net-(U9-S6)
- R22 pad 2: Net-(U10-INB-) -> VADJ
- R23 pad 1: Net-(U10-INB-) -> Net-(U9-S5)
- R23 pad 2: GND -> VADJ
- R24 pad 1: +3V3_P -> Net-(U9-S4)
- R24 pad 2: Net-(U11-INA+) -> VADJ
- R25 pad 1: Net-(U11-INA+) -> Net-(U9-S3)
- R25 pad 2: Net-(U11-INB-) -> VADJ
- R26 pad 1: Net-(U11-INB-) -> GND
- R26 pad 2: GND -> /FMC/SEL_A0
- R27 pad 1: +3V3 -> GND
- R27 pad 2: ~{FMC_PRSNT_M2C} -> /FMC/SEL_A1
- R28 pad 1: Net-(U12-D) -> GND
- R28 pad 2: Net-(U13-INB-) -> /FMC/SEL_A2
- R29 pad 1: Net-(U13-INB-) -> Net-(U9-S2)
- R29 pad 2: GND -> VADJ
- R3 pad 1: GND -> Net-(U2-ZQ)
- R3 pad 2: Net-(U2-ZQ) -> GND
- R30 pad 1: VADJ -> /FMC/Power Management/Window Comparator +3V3AUX/IN
- R30 pad 2: Net-(U12-S2) -> Net-(U10-INB-)
- R31 pad 1: VADJ -> Net-(U10-INB-)
- R31 pad 2: Net-(U12-S3) -> GND
- R32 pad 1: VADJ -> /FMC/Power Management/Window Comparator +12V0_P/IN
- R32 pad 2: Net-(U12-S4) -> Net-(U11-INB-)
- R33 pad 1: VADJ -> Net-(U11-INB-)
- R33 pad 2: Net-(U12-S5) -> GND
- R34 pad 1: VADJ -> /FMC/Power Management/Window Comparator +3V3_P/IN
- R34 pad 2: Net-(U12-S6) -> Net-(U12-INB-)
- R35 pad 1: VADJ_SEL_A0 -> Net-(U12-INB-)
- R36 pad 1: GND -> /FMC/Power Management/Window Comparator VADJ/IN
- R36 pad 2: VADJ_SEL_A1 -> Net-(U13-INB-)
- R37 pad 1: GND -> Net-(U13-INB-)
- R37 pad 2: VADJ_SEL_A2 -> GND
- R39 pad 1: GND -> VADJ
- R39 pad 2: VADJ -> GND
- R41 pad 1: Net-(U19-S2) -> /Power/VADJ/MUX_3V3
- R42 pad 1: Net-(U19-S3) -> /FMC/SEL_A0
- R43 pad 1: Net-(U19-S4) -> /FMC/SEL_A1
- R44 pad 1: Net-(U19-S5) -> /FMC/SEL_A2
- R45 pad 1: Net-(U19-S6) -> /Power/VADJ/MUX_2V5
- R46 pad 1: VADJ_SEL_A0 -> /Power/VADJ/MUX_1V8
- R47 pad 1: GND -> /Power/VADJ/MUX_1V5
- R47 pad 2: VADJ_SEL_A1 -> GND
- R48 pad 1: GND -> /Power/VADJ/MUX_1V2
- R48 pad 2: VADJ_SEL_A2 -> GND
- R6 pad 1: GND -> Net-(U3-ZQ)
- R6 pad 2: Net-(U3-ZQ) -> GND
- R9 pad 1: GND -> Net-(U4-ZQ)
- R9 pad 2: Net-(U4-ZQ) -> GND
- U1 pad AA15: DDR_DQ56 -> /FPGA/L3.DQ0
- U1 pad AA16: DDR_DQ61 -> /FPGA/L3.DQ5
- U1 pad AA17: DDR_DQ60 -> /FPGA/L3.DQ4
- U1 pad AA18: DDR_DM6 -> /FPGA/H3.DM
- U1 pad AB15: DDR_DQ57 -> /FPGA/L3.DQ1
- U1 pad AB17: DDR_DQ55 -> /FPGA/H3.DQ7
- U1 pad AB18: DDR_DQ52 -> /FPGA/H3.DQ4
- U1 pad AB19: DDR_DQ53 -> /FPGA/H3.DQ5
- U1 pad AC14: DDR_DQ58 -> /FPGA/L3.DQ2
- U1 pad AC15: DDR_DQS_N7 -> /FPGA/L3.DQS_N
- U1 pad AC16: DDR_DQS_P7 -> /FPGA/L3.DQS_P
- U1 pad AC19: DDR_DQ54 -> /FPGA/H3.DQ6
- U1 pad AD11: unconnected-(U1E-IO_L12N_T1_MRCC_33-PadAD11) -> /FPGA/~{RESET}
- U1 pad AD14: DDR_DQ59 -> /FPGA/L3.DQ3
- U1 pad AD16: DDR_DQ51 -> /FPGA/H3.DQ3
- U1 pad AD17: DDR_DQ50 -> /FPGA/H3.DQ2
- U1 pad AD18: DDR_DQ48 -> /FPGA/H3.DQ0
- U1 pad AE15: DDR_DM7 -> /FPGA/L3.DM
- U1 pad AE18: DDR_DQ49 -> /FPGA/H3.DQ1
- U1 pad AG5: DDR_RESET -> unconnected-(U1J-IO_L12N_T1_MRCC_34-PadAG5)
- U1 pad B25: unconnected-(U1E-IO_L12N_T1_MRCC_16-PadB25) -> /FMC/CLK0_N
- U1 pad B3: GND -> unconnected-(U1O-MGTAVTT-PadB3)
- U1 pad B7: GND -> unconnected-(U1O-MGTAVCC-PadB7)
- U1 pad C25: unconnected-(U1E-IO_L12P_T1_MRCC_16-PadC25) -> /FMC/CLK0_P
- U1 pad C5: GND -> unconnected-(U1O-MGTAVTT-PadC5)
- U1 pad C7: FMC_MGTREFCLK0_N -> /FMC/GTXCLK0_N
- U1 pad C8: FMC_MGTREFCLK0_P -> /FMC/GTXCLK0_P
- U1 pad D28: unconnected-(U1E-IO_L14N_T2_SRCC_16-PadD28) -> /FMC/CLK1_N
- U1 pad D3: GND -> unconnected-(U1O-MGTAVTT-PadD3)
- U1 pad D7: GND -> unconnected-(U1O-MGTAVCC-PadD7)
- U1 pad E28: unconnected-(U1E-IO_L14P_T2_SRCC_16-PadE28) -> /FMC/CLK1_P
- U1 pad E5: GND -> unconnected-(U1O-MGTAVTT-PadE5)
- U1 pad F3: GND -> unconnected-(U1O-MGTAVTT-PadF3)
- U1 pad F7: GND -> unconnected-(U1O-MGTAVCC-PadF7)
- U1 pad G5: GND -> unconnected-(U1O-MGTAVTT-PadG5)
- U1 pad H3: GND -> unconnected-(U1O-MGTAVTT-PadH3)
- U1 pad H7: GND -> unconnected-(U1O-MGTAVCC-PadH7)
- U1 pad J25: unconnected-(U1I-VCCO_15-PadJ25) -> +3V3
- U1 pad J5: GND -> unconnected-(U1O-MGTAVTT-PadJ5)
- U1 pad K22: unconnected-(U1I-VCCO_15-PadK22) -> +3V3
- U1 pad K3: GND -> unconnected-(U1O-MGTAVTT-PadK3)
- U1 pad K7: GND -> unconnected-(U1O-MGTAVCC-PadK7)
- U1 pad L29: unconnected-(U1I-VCCO_15-PadL29) -> +3V3
- U1 pad L5: GND -> unconnected-(U1O-MGTAVTT-PadL5)
- U1 pad M26: unconnected-(U1I-VCCO_15-PadM26) -> +3V3
- U1 pad M3: GND -> unconnected-(U1O-MGTAVTT-PadM3)
- U1 pad M7: GND -> unconnected-(U1O-MGTAVCC-PadM7)
- U1 pad N23: unconnected-(U1I-VCCO_15-PadN23) -> +3V3
- U1 pad N5: GND -> unconnected-(U1O-MGTAVTT-PadN5)
- U1 pad P20: unconnected-(U1I-VCCO_15-PadP20) -> +3V3
- U1 pad P3: GND -> unconnected-(U1O-MGTAVTT-PadP3)
- U1 pad P7: GND -> unconnected-(U1O-MGTAVCC-PadP7)
- U1 pad R5: GND -> unconnected-(U1O-MGTAVTT-PadR5)
- U1 pad T3: GND -> unconnected-(U1O-MGTAVTT-PadT3)
- U1 pad T7: GND -> unconnected-(U1O-MGTVCCAUX-PadT7)
- U1 pad U5: GND -> unconnected-(U1O-MGTAVTT-PadU5)
- U1 pad V11: +1V8 -> +2V0
- U1 pad V15: +1V8 -> Net-(U1P-VCCAUX-PadV15)
- U1 pad V3: GND -> unconnected-(U1O-MGTAVTT-PadV3)
- U1 pad V7: GND -> unconnected-(U1O-MGTVCCAUX-PadV7)
- U1 pad W10: +1V8 -> +2V0
- U1 pad W12: +1V8 -> +2V0
- U1 pad W14: +1V8 -> Net-(U1P-VCCAUX-PadV15)
- U1 pad W5: GND -> unconnected-(U1O-MGTAVTT-PadW5)
- U1 pad W7: GND -> unconnected-(U1O-MGTAVTTRCAL_115-PadW7)
- U1 pad Y15: DDR_DQ63 -> /FPGA/L3.DQ7
- U1 pad Y16: DDR_DQ62 -> /FPGA/L3.DQ6
- U1 pad Y18: DDR_DQS_N6 -> /FPGA/H3.DQS_N
- U1 pad Y19: DDR_DQS_P6 -> /FPGA/H3.DQS_P
- U10 pad 1: FMC_PG_C2M -> /FMC/PG
- U10 pad 3: Net-(U10-INA+) -> /FMC/Power Management/Window Comparator +3V3AUX/IN
- U10 pad 6: FMC_PG_C2M -> /FMC/PG
- U11 pad 1: FMC_PG_C2M -> /FMC/PG
- U11 pad 3: Net-(U11-INA+) -> /FMC/Power Management/Window Comparator +12V0_P/IN
- U11 pad 6: FMC_PG_C2M -> /FMC/PG
- U12 pad 1: VADJ_SEL_A0 -> /FMC/PG
- U12 pad 2: +5V0 -> GND
- U12 pad 3: GND -> /FMC/Power Management/Window Comparator +3V3_P/IN
- U12 pad 4: unconnected-(U12-S1-Pad4) -> Net-(U12-INB-)
- U12 pad 5: Net-(U12-S2) -> +3V3
- U12 pad 6: Net-(U12-S3) -> /FMC/PG
- U13 pad 1: FMC_PG_C2M -> /FMC/PG
- U13 pad 3: Net-(U12-D) -> /FMC/Power Management/Window Comparator VADJ/IN
- U13 pad 6: FMC_PG_C2M -> /FMC/PG
- U19 pad 1: VADJ_SEL_A0 -> /FMC/SEL_A0
- U19 pad 11: Net-(U19-S6) -> /Power/VADJ/MUX_3V3
- U19 pad 12: Net-(U19-S5) -> /Power/VADJ/MUX_2V5
- U19 pad 15: VADJ_SEL_A2 -> /FMC/SEL_A2
- U19 pad 16: VADJ_SEL_A1 -> /FMC/SEL_A1
- U19 pad 5: Net-(U19-S2) -> /Power/VADJ/MUX_1V2
- U19 pad 6: Net-(U19-S3) -> /Power/VADJ/MUX_1V5
- U19 pad 7: Net-(U19-S4) -> /Power/VADJ/MUX_1V8
- U2 pad T2: DDR_RESET -> /FPGA/~{RESET}
- U3 pad T2: DDR_RESET -> /FPGA/~{RESET}
- U4 pad T2: DDR_RESET -> /FPGA/~{RESET}
- U5 pad A2: DDR_DQ61 -> /FPGA/H3.DQ5
- U5 pad A3: DDR_DQ63 -> /FPGA/H3.DQ7
- U5 pad A7: DDR_DQ60 -> /FPGA/H3.DQ4
- U5 pad B7: DDR_DQS_N7 -> /FPGA/H3.DQS_N
- U5 pad B8: DDR_DQ62 -> /FPGA/H3.DQ6
- U5 pad C2: DDR_DQ59 -> /FPGA/H3.DQ3
- U5 pad C3: DDR_DQ57 -> /FPGA/H3.DQ1
- U5 pad C7: DDR_DQS_P7 -> /FPGA/H3.DQS_P
- U5 pad C8: DDR_DQ58 -> /FPGA/H3.DQ2
- U5 pad D3: DDR_DM7 -> /FPGA/H3.DM
- U5 pad D7: DDR_DQ56 -> /FPGA/H3.DQ0
- U5 pad E3: DDR_DQ48 -> /FPGA/L3.DQ0
- U5 pad E7: DDR_DM6 -> /FPGA/L3.DM
- U5 pad F2: DDR_DQ50 -> /FPGA/L3.DQ2
- U5 pad F3: DDR_DQS_P6 -> /FPGA/L3.DQS_P
- U5 pad F7: DDR_DQ49 -> /FPGA/L3.DQ1
- U5 pad F8: DDR_DQ51 -> /FPGA/L3.DQ3
- U5 pad G2: DDR_DQ54 -> /FPGA/L3.DQ6
- U5 pad G3: DDR_DQS_N6 -> /FPGA/L3.DQS_N
- U5 pad H3: DDR_DQ52 -> /FPGA/L3.DQ4
- U5 pad H7: DDR_DQ55 -> /FPGA/L3.DQ7
- U5 pad H8: DDR_DQ53 -> /FPGA/L3.DQ5
- U5 pad T2: DDR_RESET -> /FPGA/~{RESET}
- U6 pad 1: +3V3 -> +12V0
- U6 pad 2: GND -> /FMC/Power Management/PRSNT
- U6 pad 3: +3V3 -> /FMC/Power Management/PRSNT
- U6 pad 6: +3V3AUX -> Net-(U6-SST)
- U7 pad 1: +3V3_P -> +3V3
- U7 pad 3: unconnected-(U7-OCB-Pad3) -> +3V3
- U7 pad 4: FMC_PRSNT -> unconnected-(U7-~{FAULT}-Pad4)
- U7 pad 5: Net-(U7-ISET) -> Net-(U7-ILIM)
- U7 pad 6: +3V3 -> +3V3AUX
- U8 pad 1: +12V0 -> +3V3_P
- U8 pad 2: +12V0 -> GND
- U8 pad 3: +12V0 -> unconnected-(U8-~{OCB}-Pad3)
- U8 pad 4: unconnected-(U8-VCP-Pad4) -> /FMC/Power Management/PRSNT
- U8 pad 6: Net-(U8-SST) -> +3V3
- U9 pad 1: FMC_PG_C2M -> /FMC/SEL_A0
- U9 pad 2: GND -> +5V0
- U9 pad 3: Net-(U9-INA+) -> GND
- U9 pad 4: Net-(U9-INB-) -> unconnected-(U9-S1-Pad4)
- U9 pad 5: +3V3 -> Net-(U9-S2)
- U9 pad 6: FMC_PG_C2M -> Net-(U9-S3)
Routing:
- net /FMC/LA29_N: track 0.00 -> 29.5 mm, vias 0 -> 2
- net /FMC/LA29_P: track 0.00 -> 29.4 mm, vias 0 -> 2
- net /FMC/LA21_P: track 0.00 -> 28.5 mm, vias 0 -> 2
- net /FMC/LA21_N: track 0.00 -> 28.4 mm, vias 0 -> 2
- net /FMC/LA25_P: track 0.00 -> 28.0 mm, vias 0 -> 2
- net /FMC/LA25_N: track 0.00 -> 28.0 mm, vias 0 -> 2
- net /FMC/LA24_N: track 21.5 -> 28.1 mm
- net /FMC/LA24_P: track 21.4 -> 27.1 mm
- net Net-(U11-INB-): track 3.37 -> 0.00 mm
- net Net-(U11-INA+): track 3.09 -> 0.00 mm
- net Net-(U10-INB-): track 2.96 -> 0.00 mm
- net Net-(U10-INA+): track 2.90 -> 0.00 mm
- net GND: track 0.00 -> 1.80 mm, vias 0 -> 15
- net VADJ: vias 0 -> 2
- net Net-(U2-ZQ): vias 1 -> 0
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Other:
- board text added: "1"
- board text added: "30"
- board text added: "A"
- board text added: "AK"
