File: KiCad/uranus-fpga-board/uranus-fpga-board.kicad_sch (KiCad schematic)
At the start: 0 parts

Commit message: big things happening in JOURNAL
Other:
- sheet High Speed IO renamed FMC
- added sheet IDC (idc.kicad_sch)
- sheet FMC: file highspeed.kicad_sch -> fmc.kicad_sch
- sheet Misc Peripherals: file peripherals.kicad_sch -> misc.kicad_sch
Changed lines of the file:
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@@
 	)
 	(sheet
-		(at 134.62 134.62)
-		(size 114.3 113.03)
-		(exclude_from_sim no)
-		(in_bom yes)
-		(on_board yes)
-		(dnp no)
-		(fields_autoplaced yes)
-		(stroke
-			(width 0.1524)
-			(type solid)
-		)
-		(fill
-			(color 0 0 0 0)
-		)
-		(property "Sheetname" "Power"
-			(at 134.62 133.9084 0)
-			(show_name no)
-			(do_not_autoplace no)
-			(effects
-				(font
-					(size 1.27 1.27)
-				)
-				(justify left bottom)
-			)
-		)
-		(property "Sheetfile" "power.kicad_sch"
-			(at 134.62 248.2346 0)
-			(show_name no)
-			(do_not_autoplace no)
-			(effects
-				(font
-					(size 1.27 1.27)
-				)
-				(justify left top)
-			)
-		)
-		(instances
-			(project "uranus-fpga-board"
-				(path "/11d4e4d4-71ba-48aa-ae73-e6b6dc32b11b"
-					(page "6")
+		(at 15.24 134.62)
+		(size 114.3 114.3)
+		(exclude_from_sim no)
+		(in_bom yes)
+		(on_board yes)
+		(dnp no)
+		(fields_autoplaced yes)
+		(stroke
+			(width 0.1524)
+			(type solid)
+		)
+		(fill
+			(color 0 0 0 0)
+		)
+		(property "Sheetname" "IDC"
+			(at 15.24 133.9084 0)
+			(show_name no)
+			(do_not_autoplace no)
+			(effects
+				(font
+					(size 1.27 1.27)
+				)
+				(justify left bottom)
+			)
+		)
+		(property "Sheetfile" "idc.kicad_sch"
+			(at 15.24 249.5046 0)
+			(show_name no)
+			(do_not_autoplace no)
+			(effects
+				(font
+					(size 1.27 1.27)
+				)
+				(justify left top)
+			)
+		)
+		(instances
+			(project "uranus-fpga-board"
+				(path "/11d4e4d4-71ba-48aa-ae73-e6b6dc32b11b"
+					(page "5")
 				)
 			)
@@
 	)
 	(sheet
+		(at 254 134.62)
+		(size 114.3 114.3)
+		(exclude_from_sim no)
+		(in_bom yes)
+		(on_board yes)
+		(dnp no)
+		(fields_autoplaced yes)
+		(stroke
+			(width 0.1524)
+			(type solid)
+		)
+		(fill
+			(color 0 0 0 0)
+		)
+		(property "Sheetname" "Power"
+			(at 254 133.9084 0)
+			(show_name no)
+			(do_not_autoplace no)
+			(effects
+				(font
+					(size 1.27 1.27)
+				)
+				(justify left bottom)
+			)
+		)
+		(property "Sheetfile" "power.kicad_sch"
+			(at 254 249.5046 0)
+			(show_name no)
+			(do_not_autoplace no)
+			(effects
+				(font
+					(size 1.27 1.27)
+				)
+				(justify left top)
+			)
+		)
+		(instances
+			(project "uranus-fpga-board"
+				(path "/11d4e4d4-71ba-48aa-ae73-e6b6dc32b11b"
+					(page "7")
+				)
+			)
+		)
+	)
+	(sheet
 		(at 254 15.24)
 		(size 114.3 114.3)
@@
 			(color 0 0 0 0)
 		)
-		(property "Sheetname" "High Speed IO"
+		(property "Sheetname" "FMC"
 			(at 254 14.5284 0)
 			(show_name no)
@@
 			)
 		)
-		(property "Sheetfile" "highspeed.kicad_sch"
+		(property "Sheetfile" "fmc.kicad_sch"
 			(at 254 130.1246 0)
 			(show_name no)
@@
 	)
 	(sheet
-		(at 15.24 134.62)
+		(at 134.62 134.62)
 		(size 114.3 114.3)
 		(exclude_from_sim no)
@@
 		)
 		(property "Sheetname" "Misc Peripherals"
-			(at 15.24 133.9084 0)
-			(show_name no)
-			(do_not_autoplace no)
-			(effects
-				(font
-					(size 1.27 1.27)
-				)
-				(justify left bottom)
-			)
-		)
-		(property "Sheetfile" "peripherals.kicad_sch"
-			(at 15.24 249.5046 0)
-			(show_name no)
-			(do_not_autoplace no)
-			(effects
-				(font
-					(size 1.27 1.27)
-				)
-				(justify left top)
-			)
-		)
-		(instances
-			(project "uranus-fpga-board"
-				(path "/11d4e4d4-71ba-48aa-ae73-e6b6dc32b11b"
-					(page "5")
-				)
-			)
+			(at 134.62 133.9084 0)
+			(show_name no)
+			(do_not_autoplace no)
+			(effects
+				(font
+					(size 1.27 1.27)
+				)
+				(justify left bottom)
+			)
+		)
+		(property "Sheetfile" "misc.kicad_sch"
+			(at 134.62 249.5046 0)
+			(show_name no)
+			(do_not_autoplace no)
+			(effects
+				(font
+					(size 1.27 1.27)
+				)
+				(justify left top)
+			)
+		)
+		(instances
+			(project "uranus-fpga-board"
+				(path "/11d4e4d4-71ba-48aa-ae73-e6b6dc32b11b"
+					(page "6")
+				)
+			)

Commit message: big things happening in schematic quality
Other:
- sheet FMC ports: added {VADJ_CTRL}; removed none
- sheet FPGA ports: added B13{IDC_DB}, B14{IDC_DB}, H0{RAM_DB}, H1{RAM_DB}, H2{RAM_DB}, H3{RAM_DB}, L0{RAM_DB}, L1{RAM_DB}, L2{RAM_DB}, L3{RAM_DB}, {RAM_A}, {RAM_CLK}, {RAM_CTRL}, {VADJ_CTRL}; removed none
- sheet IDC ports: added B13{IDC_DB}, B14{IDC_DB}; removed none
- sheet Power ports: added {VADJ_CTRL}; removed none
- sheet RAM ports: added H0{RAM_DB}, H1{RAM_DB}, H2{RAM_DB}, H3{RAM_DB}, L0{RAM_DB}, L1{RAM_DB}, L2{RAM_DB}, L3{RAM_DB}, {RAM_A}, {RAM_CLK}, {RAM_CTRL}; removed none

Commit message: Big things have mostly happened in schematic quality
Other:
- sheet FMC ports: added {FMC_CLK}, {FMC_DB_B16}, {FMC_DB_B17}, {FMC_DB_B18}, {FMC_GTXCLK}, {FMC_GTXDB}, {FMC_I2C}, {FMC_JTAG}; removed none
- sheet FPGA ports: added IDC_B13_CLK, IDC_B13_WRT, IDC_B14_CLK, IDC_B14_WRT, {FMC_CLK}, {FMC_DB_B16}, {FMC_DB_B17}, {FMC_DB_B18}, {FMC_GTXCLK}, {FMC_GTXDB}, {FMC_I2C}, {FMC_JTAG}; removed none
- sheet IDC ports: added IDC_B13_CLK, IDC_B13_WRT, IDC_B14_CLK, IDC_B14_WRT; removed none

Commit message: I finally did it
Other:
- sheet FMC ports: added {I2C}; removed {FMC_I2C}
- sheet FPGA ports: added J2_B13{DB}, J2_B15{DB}, {I2C}; removed B13{IDC_DB}, B14{IDC_DB}, {FMC_I2C}
- sheet IDC ports: added J2_B13{DB}, J2_B15{DB}; removed B13{IDC_DB}, B14{IDC_DB}
Changed lines of the file:
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@@
 	)
 	(junction
-		(at 172.72 125.73)
+		(at 172.72 156.21)
 		(diameter 0)
 		(color 0 0 0 0)
@@
 	(bus
 		(pts
-			(xy 172.72 125.73) (xy 170.18 125.73)
+			(xy 172.72 156.21) (xy 170.18 156.21)
 		)
 		(stroke
@@
 	(bus
 		(pts
-			(xy 172.72 125.73) (xy 186.69 125.73)
+			(xy 172.72 156.21) (xy 186.69 156.21)
 		)
 		(stroke
@@
 	(bus
 		(pts
-			(xy 172.72 85.09) (xy 172.72 125.73)
+			(xy 172.72 85.09) (xy 172.72 156.21)
 		)
 		(stroke
@@
 		)
 		(property "Sheetname" "IDC"
-			(at 52.324 57.15 0)
-			(show_name no)
-			(do_not_autoplace no)
-			(effects
-				(font
-					(size 1.27 1.27)
-				)
-				(justify left bottom)
+			(at 57.15 56.642 0)
+			(show_name no)
+			(do_not_autoplace no)
+			(effects
+				(font
+					(size 1.27 1.27)
+				)
 			)
 		)
@@
 			)
 		)
-		(pin "B13{IDC_DB}" bidirectional
+		(pin "J2_B13{DB}" bidirectional
 			(at 88.9 27.94 0)
 			(effects
@@
 			)
 		)
-		(pin "B14{IDC_DB}" bidirectional
+		(pin "J2_B15{DB}" bidirectional
 			(at 88.9 38.1 0)
 			(effects
@@
 			(project "uranus-fpga-board"
 				(path "/11d4e4d4-71ba-48aa-ae73-e6b6dc32b11b"
-					(page "5")
+					(page "25")
 				)
 			)
@@
 		)
 		(property "Sheetname" "FMC"
-			(at 134.874 154.94 0)
-			(show_name no)
-			(do_not_autoplace no)
-			(effects
-				(font
-					(size 1.27 1.27)
-				)
-				(justify left bottom)
+			(at 138.43 152.908 0)
+			(show_name no)
+			(do_not_autoplace no)
+			(effects
+				(font
+					(size 1.27 1.27)
+				)
 			)
 		)
@@
 		)
 		(pin "{VADJ_CTRL}" input
-			(at 170.18 125.73 0)
-			(effects
-				(font
-					(size 1.27 1.27)
-				)
-				(justify right)
-			)
-		)
-		(pin "{FMC_DB_B16}" bidirectional
+			(at 170.18 156.21 0)
+			(effects
+				(font
+					(size 1.27 1.27)
+				)
+				(justify right)
+			)
+		)
+		(pin "{FMC_DB_B16}" output
 			(at 125.73 120.65 90)
 			(effects
@@
 			)
 		)
-		(pin "{FMC_DB_B17}" bidirectional
+		(pin "{FMC_DB_B17}" output
 			(at 128.27 120.65 90)
 			(effects
@@
 			)
 		)
-		(pin "{FMC_DB_B18}" bidirectional
+		(pin "{FMC_DB_B18}" output
 			(at 130.81 120.65 90)
 			(effects
@@
 			)
 		)
-		(pin "{FMC_I2C}" bidirectional
+		(pin "{I2C}" bidirectional
 			(at 140.97 120.65 90)
 			(effects
@@
 			)
 		)
-		(pin "{FMC_JTAG}" bidirectional
+		(pin "{FMC_JTAG}" input
 			(at 144.78 120.65 90)
 			(effects
@@
 			(project "uranus-fpga-board"
 				(path "/11d4e4d4-71ba-48aa-ae73-e6b6dc32b11b"
-					(page "4")
+					(page "18")
 				)
 			)
@@
 		)
 		(property "Sheetname" "RAM"
-			(at 213.868 60.198 0)
-			(show_name no)
-			(do_not_autoplace no)
-			(effects
-				(font
-					(size 1.27 1.27)
-				)
-				(justify left bottom)
+			(at 215.9 57.912 0)
+			(show_name no)
+			(do_not_autoplace no)
+			(effects
+				(font
+					(size 1.27 1.27)
+				)
 			)
 		)
@@
 			(project "uranus-fpga-board"
 				(path "/11d4e4d4-71ba-48aa-ae73-e6b6dc32b11b"
-					(page "3")
+					(page "13")
 				)
 			)
@@
 	(sheet
 		(at 30.48 121.92)
-		(size 54.61 50.8)
+		(size 53.34 50.8)
 		(exclude_from_sim no)
 		(in_bom yes)
@@
 		)
 		(property "Sheetname" "Misc Peripherals"
-			(at 48.006 147.828 0)
-			(show_name no)
-			(do_not_autoplace no)
-			(effects
-				(font
-					(size 1.27 1.27)
-				)
-				(justify left bottom)
+			(at 57.15 147.32 0)
+			(show_name no)
+			(do_not_autoplace no)
+			(effects
+				(font
+					(size 1.27 1.27)
+				)
 			)
 		)
@@
 			(project "uranus-fpga-board"
 				(path "/11d4e4d4-71ba-48aa-ae73-e6b6dc32b11b"
-					(page "6")
+					(page "26")
 				)
 			)
@@
 		)
 		(property "Sheetname" "FPGA"
-			(at 132.08 56.642 0)
-			(show_name no)
-			(do_not_autoplace no)
-			(effects
-				(font
-					(size 1.27 1.27)
-				)
-				(justify left bottom)
+			(at 137.16 56.642 0)
+			(show_name no)
+			(do_not_autoplace no)
+			(effects
+				(font
+					(size 1.27 1.27)
+				)
 			)
 		)
@@
 			)
 		)
-		(pin "B13{IDC_DB}" bidirectional
+		(pin "J2_B13{DB}" bidirectional
 			(at 105.41 27.94 180)
 			(effects
@@
 			)
 		)
-		(pin "B14{IDC_DB}" bidirectional
+		(pin "J2_B15{DB}" bidirectional
 			(at 105.41 38.1 180)
 			(effects
@@
 			)
 		)
-		(pin "{FMC_I2C}" bidirectional
+		(pin "{I2C}" bidirectional
 			(at 140.97 88.9 270)
 			(effects
@@
 		)
 		(pin "{VADJ_CTRL}" input
-			(at 186.69 125.73 180)
+			(at 186.69 156.21 180)
 			(effects
 				(font
@@
 			(project "uranus-fpga-board"
 				(path "/11d4e4d4-71ba-48aa-ae73-e6b6dc32b11b"
-					(page "7")
-				)
-			)
+					(page "27")
+				)
+			)
