File: KiCad/uranus-fpga-board/vadj_regulator.kicad_sch (KiCad schematic)
At the start: 21 parts, among them U18 TPS564201DDCR, U19 TMUX1108

Commit message: Big things have mostly happened in schematic quality
Parts:
- renumbered C86 to C27, C87 to C28, C88 to C29, C89 to C30, C90 to C31, C92 to C32, C93 to C33, R44 to R10, R43 to R11, R42 to R12, R41 to R13, R38 to R3, R39 to R4, R40 to R5, R45 to R6, R46 to R7, R47 to R8, R48 to R9, U18 to U6, U19 to U7

Commit message: I finally did it
Parts:
- renumbered C27 to C86, C28 to C87, C29 to C88, C30 to C89, C31 to C90, C32 to C91, C33 to C92, R3 to R38, R4 to R39, R5 to R40, R6 to R41, R7 to R42, R8 to R43, R9 to R44, R10 to R45, R11 to R46, R12 to R47, R13 to R48, U6 to U18, U7 to U19
