File: KiCad/uranus-fpga-board/window_comparator.kicad_sch (KiCad schematic)
At the start: 4 parts, among them U10 TLV6700DDCR

Commit message: Big things have mostly happened in schematic quality
Parts:
- renumbered C81 to C89, R22 to R41, R23 to R42, U10 to U17
Other:
- title: (none) -> Window Comparator
- moved on the sheet: C89

Commit message: I finally did it
Parts:
- renumbered C89 to C81, R41 to R30, R42 to R31, U17 to U10
Changed lines of the file:
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@@
 		(in_pos_files yes)
 		(dnp no)
-		(property "Reference" "U17"
+		(property "Reference" "U10"
 			(at 100.33 74.422 0)
 			(show_name no)
@@
 			(project "uranus-fpga-board"
 				(path "/11d4e4d4-71ba-48aa-ae73-e6b6dc32b11b/2757140f-486d-491c-90f5-6e7ccbeb0281/46a1c7eb-653d-4ea1-80bd-6d1b9830d8cd/6841b136-585d-4620-8c7f-346e962849dc"
-					(reference "U17")
+					(reference "U10")
 					(unit 1)
 				)
 				(path "/11d4e4d4-71ba-48aa-ae73-e6b6dc32b11b/2757140f-486d-491c-90f5-6e7ccbeb0281/46a1c7eb-653d-4ea1-80bd-6d1b9830d8cd/95b890cf-6890-4543-b4d6-b2ecad9816b0"
-					(reference "U20")
+					(reference "U13")
 					(unit 1)
 				)
 				(path "/11d4e4d4-71ba-48aa-ae73-e6b6dc32b11b/2757140f-486d-491c-90f5-6e7ccbeb0281/46a1c7eb-653d-4ea1-80bd-6d1b9830d8cd/bd59cc30-5e71-43c4-b6d6-9366f59ed92b"
-					(reference "U18")
+					(reference "U11")
 					(unit 1)
 				)
 				(path "/11d4e4d4-71ba-48aa-ae73-e6b6dc32b11b/2757140f-486d-491c-90f5-6e7ccbeb0281/46a1c7eb-653d-4ea1-80bd-6d1b9830d8cd/fb739f47-d8c4-40b2-98a1-6db3d4b23523"
-					(reference "U19")
+					(reference "U12")
 					(unit 1)
 				)
@@
 		(in_pos_files yes)
 		(dnp no)
-		(property "Reference" "#PWR0199"
+		(property "Reference" "#PWR0107"
 			(at 97.79 60.96 0)
 			(hide yes)
@@
 			(project "uranus-fpga-board"
 				(path "/11d4e4d4-71ba-48aa-ae73-e6b6dc32b11b/2757140f-486d-491c-90f5-6e7ccbeb0281/46a1c7eb-653d-4ea1-80bd-6d1b9830d8cd/6841b136-585d-4620-8c7f-346e962849dc"
-					(reference "#PWR0199")
+					(reference "#PWR0107")
 					(unit 1)
 				)
 				(path "/11d4e4d4-71ba-48aa-ae73-e6b6dc32b11b/2757140f-486d-491c-90f5-6e7ccbeb0281/46a1c7eb-653d-4ea1-80bd-6d1b9830d8cd/95b890cf-6890-4543-b4d6-b2ecad9816b0"
-					(reference "#PWR0208")
+					(reference "#PWR0116")
 					(unit 1)
 				)
 				(path "/11d4e4d4-71ba-48aa-ae73-e6b6dc32b11b/2757140f-486d-491c-90f5-6e7ccbeb0281/46a1c7eb-653d-4ea1-80bd-6d1b9830d8cd/bd59cc30-5e71-43c4-b6d6-9366f59ed92b"
-					(reference "#PWR0202")
+					(reference "#PWR0110")
 					(unit 1)
 				)
 				(path "/11d4e4d4-71ba-48aa-ae73-e6b6dc32b11b/2757140f-486d-491c-90f5-6e7ccbeb0281/46a1c7eb-653d-4ea1-80bd-6d1b9830d8cd/fb739f47-d8c4-40b2-98a1-6db3d4b23523"
-					(reference "#PWR0205")
+					(reference "#PWR0113")
 					(unit 1)
 				)
@@
 		(in_pos_files yes)
 		(dnp no)
-		(property "Reference" "#PWR0200"
+		(property "Reference" "#PWR0108"
 			(at 97.79 81.28 0)
 			(hide yes)
@@
 			(project "uranus-fpga-board"
 				(path "/11d4e4d4-71ba-48aa-ae73-e6b6dc32b11b/2757140f-486d-491c-90f5-6e7ccbeb0281/46a1c7eb-653d-4ea1-80bd-6d1b9830d8cd/6841b136-585d-4620-8c7f-346e962849dc"
-					(reference "#PWR0200")
+					(reference "#PWR0108")
 					(unit 1)
 				)
 				(path "/11d4e4d4-71ba-48aa-ae73-e6b6dc32b11b/2757140f-486d-491c-90f5-6e7ccbeb0281/46a1c7eb-653d-4ea1-80bd-6d1b9830d8cd/95b890cf-6890-4543-b4d6-b2ecad9816b0"
-					(reference "#PWR0209")
+					(reference "#PWR0117")
 					(unit 1)
 				)
 				(path "/11d4e4d4-71ba-48aa-ae73-e6b6dc32b11b/2757140f-486d-491c-90f5-6e7ccbeb0281/46a1c7eb-653d-4ea1-80bd-6d1b9830d8cd/bd59cc30-5e71-43c4-b6d6-9366f59ed92b"
-					(reference "#PWR0203")
+					(reference "#PWR0111")
 					(unit 1)
 				)
 				(path "/11d4e4d4-71ba-48aa-ae73-e6b6dc32b11b/2757140f-486d-491c-90f5-6e7ccbeb0281/46a1c7eb-653d-4ea1-80bd-6d1b9830d8cd/fb739f47-d8c4-40b2-98a1-6db3d4b23523"
-					(reference "#PWR0206")
+					(reference "#PWR0114")
 					(unit 1)
 				)
@@
 		(in_pos_files yes)
 		(dnp no)
-		(property "Reference" "R42"
+		(property "Reference" "R31"
 			(at 83.82 71.374 0)
 			(show_name no)
@@
 			(project "uranus-fpga-board"
 				(path "/11d4e4d4-71ba-48aa-ae73-e6b6dc32b11b/2757140f-486d-491c-90f5-6e7ccbeb0281/46a1c7eb-653d-4ea1-80bd-6d1b9830d8cd/6841b136-585d-4620-8c7f-346e962849dc"
-					(reference "R42")
+					(reference "R31")
 					(unit 1)
 				)
 				(path "/11d4e4d4-71ba-48aa-ae73-e6b6dc32b11b/2757140f-486d-491c-90f5-6e7ccbeb0281/46a1c7eb-653d-4ea1-80bd-6d1b9830d8cd/95b890cf-6890-4543-b4d6-b2ecad9816b0"
-					(reference "R48")
+					(reference "R37")
 					(unit 1)
 				)
 				(path "/11d4e4d4-71ba-48aa-ae73-e6b6dc32b11b/2757140f-486d-491c-90f5-6e7ccbeb0281/46a1c7eb-653d-4ea1-80bd-6d1b9830d8cd/bd59cc30-5e71-43c4-b6d6-9366f59ed92b"
-					(reference "R44")
+					(reference "R33")
 					(unit 1)
 				)
 				(path "/11d4e4d4-71ba-48aa-ae73-e6b6dc32b11b/2757140f-486d-491c-90f5-6e7ccbeb0281/46a1c7eb-653d-4ea1-80bd-6d1b9830d8cd/fb739f47-d8c4-40b2-98a1-6db3d4b23523"
-					(reference "R46")
+					(reference "R35")
 					(unit 1)
 				)
@@
 		(dnp no)
 		(fields_autoplaced yes)
-		(property "Reference" "#PWR0201"
+		(property "Reference" "#PWR0109"
 			(at 119.38 72.39 0)
 			(hide yes)
@@
 			(project "uranus-fpga-board"
 				(path "/11d4e4d4-71ba-48aa-ae73-e6b6dc32b11b/2757140f-486d-491c-90f5-6e7ccbeb0281/46a1c7eb-653d-4ea1-80bd-6d1b9830d8cd/6841b136-585d-4620-8c7f-346e962849dc"
-					(reference "#PWR0201")
+					(reference "#PWR0109")
 					(unit 1)
 				)
 				(path "/11d4e4d4-71ba-48aa-ae73-e6b6dc32b11b/2757140f-486d-491c-90f5-6e7ccbeb0281/46a1c7eb-653d-4ea1-80bd-6d1b9830d8cd/95b890cf-6890-4543-b4d6-b2ecad9816b0"
-					(reference "#PWR0210")
+					(reference "#PWR0118")
 					(unit 1)
 				)
 				(path "/11d4e4d4-71ba-48aa-ae73-e6b6dc32b11b/2757140f-486d-491c-90f5-6e7ccbeb0281/46a1c7eb-653d-4ea1-80bd-6d1b9830d8cd/bd59cc30-5e71-43c4-b6d6-9366f59ed92b"
-					(reference "#PWR0204")
+					(reference "#PWR0112")
 					(unit 1)
 				)
 				(path "/11d4e4d4-71ba-48aa-ae73-e6b6dc32b11b/2757140f-486d-491c-90f5-6e7ccbeb0281/46a1c7eb-653d-4ea1-80bd-6d1b9830d8cd/fb739f47-d8c4-40b2-98a1-6db3d4b23523"
-					(reference "#PWR0207")
+					(reference "#PWR0115")
 					(unit 1)
 				)
@@
 		(in_pos_files yes)
 		(dnp no)
-		(property "Reference" "C89"
+		(property "Reference" "C81"
 			(at 121.666 62.484 0)
 			(show_name no)
@@
 			(project "uranus-fpga-board"
 				(path "/11d4e4d4-71ba-48aa-ae73-e6b6dc32b11b/2757140f-486d-491c-90f5-6e7ccbeb0281/46a1c7eb-653d-4ea1-80bd-6d1b9830d8cd/6841b136-585d-4620-8c7f-346e962849dc"
-					(reference "C89")
+					(reference "C81")
 					(unit 1)
 				)
 				(path "/11d4e4d4-71ba-48aa-ae73-e6b6dc32b11b/2757140f-486d-491c-90f5-6e7ccbeb0281/46a1c7eb-653d-4ea1-80bd-6d1b9830d8cd/95b890cf-6890-4543-b4d6-b2ecad9816b0"
-					(reference "C92")
+					(reference "C84")
 					(unit 1)
 				)
 				(path "/11d4e4d4-71ba-48aa-ae73-e6b6dc32b11b/2757140f-486d-491c-90f5-6e7ccbeb0281/46a1c7eb-653d-4ea1-80bd-6d1b9830d8cd/bd59cc30-5e71-43c4-b6d6-9366f59ed92b"
-					(reference "C90")
+					(reference "C82")
 					(unit 1)
 				)
 				(path "/11d4e4d4-71ba-48aa-ae73-e6b6dc32b11b/2757140f-486d-491c-90f5-6e7ccbeb0281/46a1c7eb-653d-4ea1-80bd-6d1b9830d8cd/fb739f47-d8c4-40b2-98a1-6db3d4b23523"
-					(reference "C91")
+					(reference "C83")
 					(unit 1)
 				)
@@
 		(in_pos_files yes)
 		(dnp no)
-		(property "Reference" "R41"
+		(property "Reference" "R30"
 			(at 83.82 66.04 0)
 			(show_name no)
@@
 			(project "uranus-fpga-board"
 				(path "/11d4e4d4-71ba-48aa-ae73-e6b6dc32b11b/2757140f-486d-491c-90f5-6e7ccbeb0281/46a1c7eb-653d-4ea1-80bd-6d1b9830d8cd/6841b136-585d-4620-8c7f-346e962849dc"
-					(reference "R41")
+					(reference "R30")
 					(unit 1)
 				)
 				(path "/11d4e4d4-71ba-48aa-ae73-e6b6dc32b11b/2757140f-486d-491c-90f5-6e7ccbeb0281/46a1c7eb-653d-4ea1-80bd-6d1b9830d8cd/95b890cf-6890-4543-b4d6-b2ecad9816b0"
-					(reference "R47")
+					(reference "R36")
 					(unit 1)
 				)
 				(path "/11d4e4d4-71ba-48aa-ae73-e6b6dc32b11b/2757140f-486d-491c-90f5-6e7ccbeb0281/46a1c7eb-653d-4ea1-80bd-6d1b9830d8cd/bd59cc30-5e71-43c4-b6d6-9366f59ed92b"
-					(reference "R43")
+					(reference "R32")
 					(unit 1)
 				)
 				(path "/11d4e4d4-71ba-48aa-ae73-e6b6dc32b11b/2757140f-486d-491c-90f5-6e7ccbeb0281/46a1c7eb-653d-4ea1-80bd-6d1b9830d8cd/fb739f47-d8c4-40b2-98a1-6db3d4b23523"
-					(reference "R45")
-					(unit 1)
-				)
+					(reference "R34")
+					(unit 1)
+				)
